File: LEDs.sch (KiCad schematic (older format))
At the start: 9 parts, among them U2 PCA9532

Commit message: completing iteration with the LED's
Parts:
- D19, D20, D21, D22, D23, D24, D25, D26: footprint (none) -> LEDs:LED_D3.0mm
- U2: footprint (none) -> SMD_Packages:SOIC-24
Changed lines of the file:
@@
 F 0 "D19" H 4650 2900 50  0000 C CNN
 F 1 "LED_Q" H 4650 2700 50  0000 C CNN
-F 2 "" H 4650 2800 50  0000 C CNN
+F 2 "LEDs:LED_D3.0mm" H 4650 2800 50  0001 C CNN
 F 3 "" H 4650 2800 50  0000 C CNN
 	1    4650 2800
@@
 F 0 "D20" H 5150 2900 50  0000 C CNN
 F 1 "LED_W" H 5150 2700 50  0000 C CNN
-F 2 "" H 5150 2800 50  0000 C CNN
+F 2 "LEDs:LED_D3.0mm" H 5150 2800 50  0001 C CNN
 F 3 "" H 5150 2800 50  0000 C CNN
 	1    5150 2800
@@
 F 0 "D21" H 5750 2900 50  0000 C CNN
 F 1 "LED_E" H 5750 2700 50  0000 C CNN
-F 2 "" H 5750 2800 50  0000 C CNN
+F 2 "LEDs:LED_D3.0mm" H 5750 2800 50  0001 C CNN
 F 3 "" H 5750 2800 50  0000 C CNN
 	1    5750 2800
@@
 F 0 "D22" H 6250 2900 50  0000 C CNN
 F 1 "LED_R" H 6250 2700 50  0000 C CNN
-F 2 "" H 6250 2800 50  0000 C CNN
+F 2 "LEDs:LED_D3.0mm" H 6250 2800 50  0001 C CNN
 F 3 "" H 6250 2800 50  0000 C CNN
 	1    6250 2800
@@
 F 0 "D23" H 6700 2900 50  0000 C CNN
 F 1 "LED_T" H 6700 2700 50  0000 C CNN
-F 2 "" H 6700 2800 50  0000 C CNN
+F 2 "LEDs:LED_D3.0mm" H 6700 2800 50  0001 C CNN
 F 3 "" H 6700 2800 50  0000 C CNN
 	1    6700 2800
@@
 F 0 "D24" H 7150 2900 50  0000 C CNN
 F 1 "LED_Y" H 7150 2700 50  0000 C CNN
-F 2 "" H 7150 2800 50  0000 C CNN
+F 2 "LEDs:LED_D3.0mm" H 7150 2800 50  0001 C CNN
 F 3 "" H 7150 2800 50  0000 C CNN
 	1    7150 2800
@@
 F 0 "D25" H 7600 2900 50  0000 C CNN
 F 1 "LED_U" H 7600 2700 50  0000 C CNN
-F 2 "" H 7600 2800 50  0000 C CNN
+F 2 "LEDs:LED_D3.0mm" H 7600 2800 50  0001 C CNN
 F 3 "" H 7600 2800 50  0000 C CNN
 	1    7600 2800
@@
 F 0 "D26" H 8100 2900 50  0000 C CNN
 F 1 "LED_I" H 8100 2700 50  0000 C CNN
-F 2 "" H 8100 2800 50  0000 C CNN
+F 2 "LEDs:LED_D3.0mm" H 8100 2800 50  0001 C CNN
 F 3 "" H 8100 2800 50  0000 C CNN
 	1    8100 2800
@@
 F 0 "U2" V 2750 5250 60  0000 C CNN
 F 1 "PCA9532" V 2650 5250 60  0000 C CNN
-F 2 "" H 2700 4500 60  0001 C CNN
+F 2 "SMD_Packages:SOIC-24" H 2700 4500 60  0001 C CNN
 F 3 "" H 2700 4500 60  0001 C CNN
 	1    2700 4500

Commit message: updates
Parts:
- D19, D20, D21, D22, D23, D24, D25, D26: footprint LEDs:LED_D3.0mm -> (none)
- U2: footprint SMD_Packages:SOIC-24 -> (none)
Changed lines of the file:
@@
 F 0 "D19" H 4650 2900 50  0000 C CNN
 F 1 "LED_Q" H 4650 2700 50  0000 C CNN
-F 2 "LEDs:LED_D3.0mm" H 4650 2800 50  0001 C CNN
+F 2 "" H 4650 2800 50  0000 C CNN
 F 3 "" H 4650 2800 50  0000 C CNN
 	1    4650 2800
@@
 F 0 "D20" H 5150 2900 50  0000 C CNN
 F 1 "LED_W" H 5150 2700 50  0000 C CNN
-F 2 "LEDs:LED_D3.0mm" H 5150 2800 50  0001 C CNN
+F 2 "" H 5150 2800 50  0000 C CNN
 F 3 "" H 5150 2800 50  0000 C CNN
 	1    5150 2800
@@
 F 0 "D21" H 5750 2900 50  0000 C CNN
 F 1 "LED_E" H 5750 2700 50  0000 C CNN
-F 2 "LEDs:LED_D3.0mm" H 5750 2800 50  0001 C CNN
+F 2 "" H 5750 2800 50  0000 C CNN
 F 3 "" H 5750 2800 50  0000 C CNN
 	1    5750 2800
@@
 F 0 "D22" H 6250 2900 50  0000 C CNN
 F 1 "LED_R" H 6250 2700 50  0000 C CNN
-F 2 "LEDs:LED_D3.0mm" H 6250 2800 50  0001 C CNN
+F 2 "" H 6250 2800 50  0000 C CNN
 F 3 "" H 6250 2800 50  0000 C CNN
 	1    6250 2800
@@
 F 0 "D23" H 6700 2900 50  0000 C CNN
 F 1 "LED_T" H 6700 2700 50  0000 C CNN
-F 2 "LEDs:LED_D3.0mm" H 6700 2800 50  0001 C CNN
+F 2 "" H 6700 2800 50  0000 C CNN
 F 3 "" H 6700 2800 50  0000 C CNN
 	1    6700 2800
@@
 F 0 "D24" H 7150 2900 50  0000 C CNN
 F 1 "LED_Y" H 7150 2700 50  0000 C CNN
-F 2 "LEDs:LED_D3.0mm" H 7150 2800 50  0001 C CNN
+F 2 "" H 7150 2800 50  0000 C CNN
 F 3 "" H 7150 2800 50  0000 C CNN
 	1    7150 2800
@@
 F 0 "D25" H 7600 2900 50  0000 C CNN
 F 1 "LED_U" H 7600 2700 50  0000 C CNN
-F 2 "LEDs:LED_D3.0mm" H 7600 2800 50  0001 C CNN
+F 2 "" H 7600 2800 50  0000 C CNN
 F 3 "" H 7600 2800 50  0000 C CNN
 	1    7600 2800
@@
 F 0 "D26" H 8100 2900 50  0000 C CNN
 F 1 "LED_I" H 8100 2700 50  0000 C CNN
-F 2 "LEDs:LED_D3.0mm" H 8100 2800 50  0001 C CNN
+F 2 "" H 8100 2800 50  0000 C CNN
 F 3 "" H 8100 2800 50  0000 C CNN
 	1    8100 2800
@@
 F 0 "U2" V 2750 5250 60  0000 C CNN
 F 1 "PCA9532" V 2650 5250 60  0000 C CNN
-F 2 "SMD_Packages:SOIC-24" H 2700 4500 60  0001 C CNN
+F 2 "" H 2700 4500 60  0001 C CNN
 F 3 "" H 2700 4500 60  0001 C CNN
 	1    2700 4500
