File: Keys.sch (KiCad schematic (older format))
At the start: 36 parts, among them SW1 KEY_Q, SW10 KEY_G, SW11 KEY_Y, SW12 KEY_H, SW13 KEY_U, SW14 KEY_J, SW15 KEY_I, SW16 KEY_K, SW17 KEY_O, SW18 KEY_L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

Commit message: test keyboard
Parts:
- removed D10, D11, D12, D13, D14, D15, D16, D17, D18, D5, D6, D7, D8, D9: D, Diodes_SMD:D_0603, symbol D
- removed SW10: KEY_G, footprints:CHERRY_PCB_100H, symbol SWITCH_PUSH
- removed SW11: KEY_Y, footprints:CHERRY_PCB_100H, symbol SWITCH_PUSH
- removed SW12: KEY_H, footprints:CHERRY_PCB_100H, symbol SWITCH_PUSH
- removed SW13: KEY_U, footprints:CHERRY_PCB_100H, symbol SWITCH_PUSH
- removed SW14: KEY_J, footprints:CHERRY_PCB_100H, symbol SWITCH_PUSH
- removed SW15: KEY_I, footprints:CHERRY_PCB_100H, symbol SWITCH_PUSH
- removed SW16: KEY_K, footprints:CHERRY_PCB_100H, symbol SWITCH_PUSH
- removed SW17: KEY_O, footprints:CHERRY_PCB_100H, symbol SWITCH_PUSH
- removed SW18: KEY_L, footprints:CHERRY_PCB_100H, symbol SWITCH_PUSH
- removed SW5: KEY_E, footprints:CHERRY_PCB_100H, symbol SWITCH_PUSH
- removed SW6: KEY_D, footprints:CHERRY_PCB_100H, symbol SWITCH_PUSH
- removed SW7: KEY_R, footprints:CHERRY_PCB_100H, symbol SWITCH_PUSH
- removed SW8: KEY_F, footprints:CHERRY_PCB_100H, symbol SWITCH_PUSH
- removed SW9: KEY_T, footprints:CHERRY_PCB_100H, symbol SWITCH_PUSH
Connections:
- net labels removed: KEY_COL2, KEY_COL3, KEY_COL4, KEY_COL5, KEY_COL6, KEY_COL7, KEY_COL8
- wire segments 84 -> 20

Commit message: updates
Parts:
- removed D4: D, Diodes_SMD:D_0603, symbol D
- removed SW4: KEY_S, footprints:CHERRY_PCB_100H, symbol SWITCH_PUSH
- SW1, SW2, SW3: footprint footprints:CHERRY_PCB_100H -> footprints:CG6_CHERRY_PCB_100H
Connections:
- wire segments 20 -> 16
Changed lines of the file:
@@
 F 0 "SW1" H 2450 1710 50  0000 C CNN
 F 1 "KEY_Q" H 2300 1520 50  0000 C CNN
-F 2 "footprints:CHERRY_PCB_100H" H 2300 1600 60  0001 C CNN
+F 2 "footprints:CG6_CHERRY_PCB_100H" H 2300 1600 60  0001 C CNN
 F 3 "" H 2300 1600 60  0001 C CNN
 	1    2300 1600
@@
 F 0 "SW3" H 3200 1710 50  0000 C CNN
 F 1 "KEY_W" H 3050 1520 50  0000 C CNN
-F 2 "footprints:CHERRY_PCB_100H" H 3050 1600 60  0001 C CNN
+F 2 "footprints:CG6_CHERRY_PCB_100H" H 3050 1600 60  0001 C CNN
 F 3 "" H 3050 1600 60  0001 C CNN
 	1    3050 1600
@@
 F 0 "SW2" H 2450 2410 50  0000 C CNN
 F 1 "KEY_A" H 2300 2220 50  0000 C CNN
-F 2 "footprints:CHERRY_PCB_100H" H 2300 2300 60  0001 C CNN
+F 2 "footprints:CG6_CHERRY_PCB_100H" H 2300 2300 60  0001 C CNN
 F 3 "" H 2300 2300 60  0001 C CNN
 	1    2300 2300
@@
 	1    0    0    -1
 $EndComp
-$Comp
-L SWITCH_PUSH SW4
-U 1 1 58965EC9
-P 3050 2300
-F 0 "SW4" H 3200 2410 50  0000 C CNN
-F 1 "KEY_S" H 3050 2220 50  0000 C CNN
-F 2 "footprints:CHERRY_PCB_100H" H 3050 2300 60  0001 C CNN
-F 3 "" H 3050 2300 60  0001 C CNN
-	1    3050 2300
-	1    0    0    -1
-$EndComp
-$Comp
-L D D4
-U 1 1 58965ECF
-P 3050 2600
-F 0 "D4" H 3050 2700 50  0000 C CNN
-F 1 "D" H 3050 2500 50  0000 C CNN
-F 2 "Diodes_SMD:D_0603" H 3050 2600 50  0001 C CNN
-F 3 "" H 3050 2600 50  0000 C CNN
-	1    3050 2600
-	1    0    0    -1
-$EndComp
 Wire Wire Line
 	3350 1900 3200 1900
@@
 Wire Wire Line
 	1800 950  1800 4700
-Wire Wire Line
-	3350 2600 3200 2600
-Wire Wire Line
-	3350 2300 3350 2600
 Wire Wire Line
 	2600 2600 2450 2600
@@
 	2150 2600 1800 2600
 Connection ~ 1800 2600
-Wire Wire Line
-	2900 2600 2700 2600
 Connection ~ 2700 2600
 Wire Wire Line
@@
 	2000 2300 2000 2150
 Connection ~ 2000 2150
-Wire Wire Line
-	2750 2150 2750 2300
 Connection ~ 2750 2150
 Text HLabel 1350 2150 0    60   Input ~ 0

Commit message: messing around
Parts:
- added D4, D5, D6: D, Diodes_SMD:D_0603, symbol Keys-rescue:D
- added SW4, SW5, SW6: KEY_W, footprints:CG6_CHERRY_PCB_100H, symbol Keys-rescue:SWITCH_PUSH
- D1, D2, D3: symbol D -> Keys-rescue:D
- SW1, SW2, SW3: symbol SWITCH_PUSH -> Keys-rescue:SWITCH_PUSH
Connections:
- net labels added: KEY_ROW2
- wire segments 16 -> 42
Changed lines of the file:
@@
-EESchema Schematic File Version 2
-LIBS:power
-LIBS:device
-LIBS:switches
-LIBS:teensy
-LIBS:components
-LIBS:NXP-chgray
-LIBS:chgray-keyboard-cache
-EELAYER 25 0
+EESchema Schematic File Version 4
+EELAYER 30 0
 EELAYER END
 $Descr A4 11693 8268
 encoding utf-8
-Sheet 2 2
+Sheet 1 1
 Title ""
 Date ""
@@
 $EndDescr
 $Comp
-L SWITCH_PUSH SW1
+L Keys-rescue:SWITCH_PUSH SW1
 U 1 1 58964642
 P 2300 1600
@@
 $EndComp
 $Comp
-L D D1
+L Keys-rescue:D D1
 U 1 1 5896466F
 P 2300 1900
@@
 KEY_ROW0
 $Comp
-L SWITCH_PUSH SW3
+L Keys-rescue:SWITCH_PUSH SW3
 U 1 1 589655C0
 P 3050 1600
@@
 $EndComp
 $Comp
-L D D3
+L Keys-rescue:D D3
 U 1 1 589655C6
 P 3050 1900
@@
 $EndComp
 $Comp
-L SWITCH_PUSH SW2
+L Keys-rescue:SWITCH_PUSH SW2
 U 1 1 58965EBD
 P 2300 2300
@@
 $EndComp
 $Comp
-L D D2
+L Keys-rescue:D D2
 U 1 1 58965EC3
 P 2300 2600
@@
 	2600 1600 2600 1900
 Wire Wire Line
-	1800 950  1800 4700
+	1800 950  1800 1900
 Wire Wire Line
 	2600 2600 2450 2600
@@
 	2600 2300 2600 2600
 Wire Wire Line
-	2700 950  2700 4700
+	2700 950  2700 1900
 Wire Wire Line
 	2150 1900 1800 1900
@@
 	2150 2600 1800 2600
 Connection ~ 1800 2600
-Connection ~ 2700 2600
 Wire Wire Line
 	2900 1900 2700 1900
@@
 Wire Wire Line
 	2750 1300 2750 1600
-Connection ~ 2750 1300
 Wire Wire Line
 	2000 2300 2000 2150
 Connection ~ 2000 2150
-Connection ~ 2750 2150
 Text HLabel 1350 2150 0    60   Input ~ 0
 KEY_ROW1
@@
 KEY_COL1
 Wire Wire Line
-	1350 1300 2750 1300
-Wire Wire Line
-	1350 2150 2750 2150
+	1350 1300 2000 1300
+Wire Wire Line
+	1350 2150 2000 2150
+Wire Wire Line
+	1800 1900 1800 2600
+Wire Wire Line
+	2000 1300 2750 1300
+Wire Wire Line
+	2000 2150 2750 2150
+Wire Wire Line
+	2700 1900 2700 2600
+$Comp
+L Keys-rescue:SWITCH_PUSH SW4
+U 1 1 603DF303
+P 3050 2300
+F 0 "SW4" H 3200 2410 50  0000 C CNN
+F 1 "KEY_W" H 3050 2220 50  0000 C CNN
+F 2 "footprints:CG6_CHERRY_PCB_100H" H 3050 2300 60  0001 C CNN
+F 3 "" H 3050 2300 60  0001 C CNN
+	1    3050 2300
+	1    0    0    -1
+$EndComp
+Wire Wire Line
+	2750 2150 2750 2300
+Wire Wire Line
+	3000 1900 3100 1900
+$Comp
+L Keys-rescue:D D6
+U 1 1 603E2BDF
+P 3050 2600
+F 0 "D6" H 3050 2700 50  0000 C CNN
+F 1 "D" H 3050 2500 50  0000 C CNN
+F 2 "Diodes_SMD:D_0603" H 3050 2600 50  0001 C CNN
+F 3 "" H 3050 2600 50  0000 C CNN
+	1    3050 2600
+	1    0    0    -1
+$EndComp
+Wire Wire Line
+	3000 2600 3100 2600
+Wire Wire Line
+	3350 2300 3350 2600
+Wire Wire Line
+	3350 2600 3200 2600
+Wire Wire Line
+	2900 2600 2700 2600
+Connection ~ 2700 2600
+Wire Wire Line
+	2700 2600 2700 3550
+Wire Wire Line
+	1800 2600 1800 3550
+$Comp
+L Keys-rescue:SWITCH_PUSH SW5
+U 1 1 603E8C3D
+P 2250 3250
+F 0 "SW5" H 2400 3360 50  0000 C CNN
+F 1 "KEY_W" H 2250 3170 50  0000 C CNN
+F 2 "footprints:CG6_CHERRY_PCB_100H" H 2250 3250 60  0001 C CNN
+F 3 "" H 2250 3250 60  0001 C CNN
+	1    2250 3250
+	1    0    0    -1
+$EndComp
+$Comp
+L Keys-rescue:D D4
+U 1 1 603E8C43
+P 2250 3550
+F 0 "D4" H 2250 3650 50  0000 C CNN
+F 1 "D" H 2250 3450 50  0000 C CNN
+F 2 "Diodes_SMD:D_0603" H 2250 3550 50  0001 C CNN
+F 3 "" H 2250 3550 50  0000 C CNN
+	1    2250 3550
+	1    0    0    -1
+$EndComp
+Wire Wire Line
+	2200 3550 2300 3550
+Wire Wire Line
+	2550 3250 2550 3550
+Wire Wire Line
+	2550 3550 2400 3550
+Text HLabel 1350 3050 0    60   Input ~ 0
+KEY_ROW2
+Wire Wire Line
+	1950 3250 1950 3050
+Wire Wire Line
+	1950 3050 1350 3050
+Wire Wire Line
+	1800 3550 2100 3550
+Connection ~ 1800 3550
+Wire Wire Line
+	1800 3550 1800 4700
+$Comp
+L Keys-rescue:SWITCH_PUSH SW6
+U 1 1 603EBFA8
+P 3050 3250
+F 0 "SW6" H 3200 3360 50  0000 C CNN
+F 1 "KEY_W" H 3050 3170 50  0000 C CNN
+F 2 "footprints:CG6_CHERRY_PCB_100H" H 3050 3250 60  0001 C CNN
+F 3 "" H 3050 3250 60  0001 C CNN
+	1    3050 3250
+	1    0    0    -1
+$EndComp
+$Comp
+L Keys-rescue:D D5
+U 1 1 603EBFAE
+P 3050 3550
+F 0 "D5" H 3050 3650 50  0000 C CNN
+F 1 "D" H 3050 3450 50  0000 C CNN
+F 2 "Diodes_SMD:D_0603" H 3050 3550 50  0001 C CNN
+F 3 "" H 3050 3550 50  0000 C CNN
+	1    3050 3550
+	1    0    0    -1
+$EndComp
+Wire Wire Line
+	3000 3550 3100 3550
+Wire Wire Line
+	3350 3250 3350 3550
+Wire Wire Line
+	3350 3550 3200 3550
+Wire Wire Line
+	1950 3050 2750 3050
+Wire Wire Line
+	2750 3050 2750 3250
+Connection ~ 1950 3050
+Wire Wire Line
+	2700 3550 2900 3550
+Connection ~ 2700 3550
+Wire Wire Line
+	2700 3550 2700 4700
 $EndSCHEMATC

Commit message: docker file
Parts:
- D1, D2, D3, D4, D5, D6: symbol Keys-rescue:D -> chgray-keyboard-rescue:D-Keys-rescue
- SW1, SW4: footprint footprints:CG6_CHERRY_PCB_100H -> footprints:CHERRY_PCB_100H; symbol Keys-rescue:SWITCH_PUSH -> chgray-keyboard-rescue:SWITCH_PUSH-Keys-rescue
- SW2, SW3, SW5, SW6: symbol Keys-rescue:SWITCH_PUSH -> chgray-keyboard-rescue:SWITCH_PUSH-Keys-rescue
Changed lines of the file:
@@
 $Descr A4 11693 8268
 encoding utf-8
-Sheet 2 2
+Sheet 1 1
 Title ""
 Date ""
@@
 $EndDescr
 $Comp
-L Keys-rescue:SWITCH_PUSH SW1
+L chgray-keyboard-rescue:SWITCH_PUSH-Keys-rescue SW1
 U 1 1 58964642
 P 2300 1600
 F 0 "SW1" H 2450 1710 50  0000 C CNN
 F 1 "KEY_Q" H 2300 1520 50  0000 C CNN
-F 2 "footprints:CG6_CHERRY_PCB_100H" H 2300 1600 60  0001 C CNN
+F 2 "footprints:CHERRY_PCB_100H" H 2300 1600 60  0001 C CNN
 F 3 "" H 2300 1600 60  0001 C CNN
 	1    2300 1600
@@
 $EndComp
 $Comp
-L Keys-rescue:D D1
+L chgray-keyboard-rescue:D-Keys-rescue D1
 U 1 1 5896466F
 P 2300 1900
@@
 KEY_ROW0
 $Comp
-L Keys-rescue:SWITCH_PUSH SW3
+L chgray-keyboard-rescue:SWITCH_PUSH-Keys-rescue SW3
 U 1 1 589655C0
 P 3050 1600
@@
 $EndComp
 $Comp
-L Keys-rescue:D D3
+L chgray-keyboard-rescue:D-Keys-rescue D3
 U 1 1 589655C6
 P 3050 1900
@@
 $EndComp
 $Comp
-L Keys-rescue:SWITCH_PUSH SW2
+L chgray-keyboard-rescue:SWITCH_PUSH-Keys-rescue SW2
 U 1 1 58965EBD
 P 2300 2300
@@
 $EndComp
 $Comp
-L Keys-rescue:D D2
+L chgray-keyboard-rescue:D-Keys-rescue D2
 U 1 1 58965EC3
 P 2300 2600
@@
 	2700 1900 2700 2600
 $Comp
-L Keys-rescue:SWITCH_PUSH SW4
+L chgray-keyboard-rescue:SWITCH_PUSH-Keys-rescue SW4
 U 1 1 603DF303
 P 3050 2300
 F 0 "SW4" H 3200 2410 50  0000 C CNN
 F 1 "KEY_W" H 3050 2220 50  0000 C CNN
-F 2 "footprints:CG6_CHERRY_PCB_100H" H 3050 2300 60  0001 C CNN
+F 2 "footprints:CHERRY_PCB_100H" H 3050 2300 60  0001 C CNN
 F 3 "" H 3050 2300 60  0001 C CNN
 	1    3050 2300
@@
 	3000 1900 3100 1900
 $Comp
-L Keys-rescue:D D6
+L chgray-keyboard-rescue:D-Keys-rescue D6
 U 1 1 603E2BDF
 P 3050 2600
@@
 	1800 2600 1800 3550
 $Comp
-L Keys-rescue:SWITCH_PUSH SW5
+L chgray-keyboard-rescue:SWITCH_PUSH-Keys-rescue SW5
 U 1 1 603E8C3D
 P 2250 3250
@@
 $EndComp
 $Comp
-L Keys-rescue:D D4
+L chgray-keyboard-rescue:D-Keys-rescue D4
 U 1 1 603E8C43
 P 2250 3550
@@
 	1800 3550 1800 4700
 $Comp
-L Keys-rescue:SWITCH_PUSH SW6
+L chgray-keyboard-rescue:SWITCH_PUSH-Keys-rescue SW6
 U 1 1 603EBFA8
 P 3050 3250
@@
 $EndComp
 $Comp
-L Keys-rescue:D D5
+L chgray-keyboard-rescue:D-Keys-rescue D5
 U 1 1 603EBFAE
 P 3050 3550

Commit message: file
Parts:
- added D10: D9, Diode_SMD:D_0201_0603Metric, symbol chgray-keyboard-rescue:D-Keys-rescue-chgray-keyboard-rescue
- added D11: D11, Diode_SMD:D_0201_0603Metric, symbol chgray-keyboard-rescue:D-Keys-rescue-chgray-keyboard-rescue
- added D12: D13, Diode_SMD:D_0201_0603Metric, symbol chgray-keyboard-rescue:D-Keys-rescue-chgray-keyboard-rescue
- added D7: D8, Diode_SMD:D_0201_0603Metric, symbol chgray-keyboard-rescue:D-Keys-rescue-chgray-keyboard-rescue
- added D8: D10, Diode_SMD:D_0201_0603Metric, symbol chgray-keyboard-rescue:D-Keys-rescue-chgray-keyboard-rescue
- added D9: D12, Diode_SMD:D_0201_0603Metric, symbol chgray-keyboard-rescue:D-Keys-rescue-chgray-keyboard-rescue
- added SW10, SW11, SW12, SW7, SW8, SW9: KEY_W, footprints:CG6_CHERRY_PCB_100H, symbol chgray-keyboard-rescue:SWITCH_PUSH-Keys-rescue-chgray-keyboard-rescue
- D1, D2, D3, D4, D5, D6: footprint Diodes_SMD:D_0603 -> Diode_SMD:D_0201_0603Metric; symbol chgray-keyboard-rescue:D-Keys-rescue -> chgray-keyboard-rescue:D-Keys-rescue-chgray-keyboard-rescue
- SW1, SW2, SW3, SW4, SW5, SW6: symbol chgray-keyboard-rescue:SWITCH_PUSH-Keys-rescue -> chgray-keyboard-rescue:SWITCH_PUSH-Keys-rescue-chgray-keyboard-rescue
Connections:
- net labels added: KEY_ROW3, KEY_ROW4, KEY_ROW5
- wire segments 42 -> 84

Commit message: working
Parts:
- D?: renamed from D1; symbol chgray-keyboard-rescue:D-Keys-rescue-chgray-keyboard-rescue -> Keys-rescue:D-Keys-rescue-chgray-keyboard-rescue-chgray-keyboard-rescue
- D?: renamed from D3; symbol chgray-keyboard-rescue:D-Keys-rescue-chgray-keyboard-rescue -> Keys-rescue:D-Keys-rescue-chgray-keyboard-rescue-chgray-keyboard-rescue
- D?: renamed from D2; symbol chgray-keyboard-rescue:D-Keys-rescue-chgray-keyboard-rescue -> Keys-rescue:D-Keys-rescue-chgray-keyboard-rescue-chgray-keyboard-rescue
- D?: renamed from D6; symbol chgray-keyboard-rescue:D-Keys-rescue-chgray-keyboard-rescue -> Keys-rescue:D-Keys-rescue-chgray-keyboard-rescue-chgray-keyboard-rescue
- D?: renamed from D4; symbol chgray-keyboard-rescue:D-Keys-rescue-chgray-keyboard-rescue -> Keys-rescue:D-Keys-rescue-chgray-keyboard-rescue-chgray-keyboard-rescue
- D?: renamed from D5; symbol chgray-keyboard-rescue:D-Keys-rescue-chgray-keyboard-rescue -> Keys-rescue:D-Keys-rescue-chgray-keyboard-rescue-chgray-keyboard-rescue
- D?: renamed from D7; symbol chgray-keyboard-rescue:D-Keys-rescue-chgray-keyboard-rescue -> Keys-rescue:D-Keys-rescue-chgray-keyboard-rescue-chgray-keyboard-rescue
- D?: renamed from D10; symbol chgray-keyboard-rescue:D-Keys-rescue-chgray-keyboard-rescue -> Keys-rescue:D-Keys-rescue-chgray-keyboard-rescue-chgray-keyboard-rescue
- D?: renamed from D8; symbol chgray-keyboard-rescue:D-Keys-rescue-chgray-keyboard-rescue -> Keys-rescue:D-Keys-rescue-chgray-keyboard-rescue-chgray-keyboard-rescue
- D?: renamed from D11; symbol chgray-keyboard-rescue:D-Keys-rescue-chgray-keyboard-rescue -> Keys-rescue:D-Keys-rescue-chgray-keyboard-rescue-chgray-keyboard-rescue
- D?: renamed from D9; symbol chgray-keyboard-rescue:D-Keys-rescue-chgray-keyboard-rescue -> Keys-rescue:D-Keys-rescue-chgray-keyboard-rescue-chgray-keyboard-rescue
- D?: renamed from D12; symbol chgray-keyboard-rescue:D-Keys-rescue-chgray-keyboard-rescue -> Keys-rescue:D-Keys-rescue-chgray-keyboard-rescue-chgray-keyboard-rescue
- SW?: renamed from SW1; footprint footprints:CHERRY_PCB_100H -> CherryKeys:CHERRY_PCB_100H; symbol chgray-keyboard-rescue:SWITCH_PUSH-Keys-rescue-chgray-keyboard-rescue -> Keys-rescue:SWITCH_PUSH-Keys-rescue-chgray-keyboard-rescue-chgray-keyboard-rescue
- SW?: renamed from SW3; footprint footprints:CG6_CHERRY_PCB_100H -> CherryKeys:CHERRY_PCB_100H; symbol chgray-keyboard-rescue:SWITCH_PUSH-Keys-rescue-chgray-keyboard-rescue -> Keys-rescue:SWITCH_PUSH-Keys-rescue-chgray-keyboard-rescue-chgray-keyboard-rescue
- SW?: renamed from SW2; footprint footprints:CG6_CHERRY_PCB_100H -> CherryKeys:CHERRY_PCB_100H; symbol chgray-keyboard-rescue:SWITCH_PUSH-Keys-rescue-chgray-keyboard-rescue -> Keys-rescue:SWITCH_PUSH-Keys-rescue-chgray-keyboard-rescue-chgray-keyboard-rescue
- SW?: renamed from SW4; footprint footprints:CHERRY_PCB_100H -> CherryKeys:CHERRY_PCB_100H; symbol chgray-keyboard-rescue:SWITCH_PUSH-Keys-rescue-chgray-keyboard-rescue -> Keys-rescue:SWITCH_PUSH-Keys-rescue-chgray-keyboard-rescue-chgray-keyboard-rescue
- SW?: renamed from SW5; footprint footprints:CG6_CHERRY_PCB_100H -> CherryKeys:CHERRY_PCB_100H; symbol chgray-keyboard-rescue:SWITCH_PUSH-Keys-rescue-chgray-keyboard-rescue -> Keys-rescue:SWITCH_PUSH-Keys-rescue-chgray-keyboard-rescue-chgray-keyboard-rescue
- SW?: renamed from SW6; footprint footprints:CG6_CHERRY_PCB_100H -> CherryKeys:CHERRY_PCB_100H; symbol chgray-keyboard-rescue:SWITCH_PUSH-Keys-rescue-chgray-keyboard-rescue -> Keys-rescue:SWITCH_PUSH-Keys-rescue-chgray-keyboard-rescue-chgray-keyboard-rescue
- SW?: renamed from SW7; footprint footprints:CG6_CHERRY_PCB_100H -> CherryKeys:CHERRY_PCB_100H; symbol chgray-keyboard-rescue:SWITCH_PUSH-Keys-rescue-chgray-keyboard-rescue -> Keys-rescue:SWITCH_PUSH-Keys-rescue-chgray-keyboard-rescue-chgray-keyboard-rescue
- SW?: renamed from SW8; footprint footprints:CG6_CHERRY_PCB_100H -> CherryKeys:CHERRY_PCB_100H; symbol chgray-keyboard-rescue:SWITCH_PUSH-Keys-rescue-chgray-keyboard-rescue -> Keys-rescue:SWITCH_PUSH-Keys-rescue-chgray-keyboard-rescue-chgray-keyboard-rescue
- SW?: renamed from SW9; footprint footprints:CG6_CHERRY_PCB_100H -> CherryKeys:CHERRY_PCB_100H; symbol chgray-keyboard-rescue:SWITCH_PUSH-Keys-rescue-chgray-keyboard-rescue -> Keys-rescue:SWITCH_PUSH-Keys-rescue-chgray-keyboard-rescue-chgray-keyboard-rescue
- SW?: renamed from SW10; footprint footprints:CG6_CHERRY_PCB_100H -> CherryKeys:CHERRY_PCB_100H; symbol chgray-keyboard-rescue:SWITCH_PUSH-Keys-rescue-chgray-keyboard-rescue -> Keys-rescue:SWITCH_PUSH-Keys-rescue-chgray-keyboard-rescue-chgray-keyboard-rescue
- SW?: renamed from SW11; footprint footprints:CG6_CHERRY_PCB_100H -> CherryKeys:CHERRY_PCB_100H; symbol chgray-keyboard-rescue:SWITCH_PUSH-Keys-rescue-chgray-keyboard-rescue -> Keys-rescue:SWITCH_PUSH-Keys-rescue-chgray-keyboard-rescue-chgray-keyboard-rescue
- SW?: renamed from SW12; footprint footprints:CG6_CHERRY_PCB_100H -> CherryKeys:CHERRY_PCB_100H; symbol chgray-keyboard-rescue:SWITCH_PUSH-Keys-rescue-chgray-keyboard-rescue -> Keys-rescue:SWITCH_PUSH-Keys-rescue-chgray-keyboard-rescue-chgray-keyboard-rescue

Commit message: experiment
Parts:
- SW? (x2): symbol Keys-rescue:SWITCH_PUSH-Keys-rescue-chgray-keyboard-rescue-chgray-keyboard-rescue -> Cherry-Symbols:SWITCH_PUSH
