File: RGB-Circuit.sch (KiCad schematic (older format))
At the start: 6 parts

Commit message: rgb
Parts:
- removed D74, D75: DIODE, Diode_SMD:D_SOD-123, symbol LED:SK6812MINI
- added C10, C11, C12, C13, C14, C15, C16, C17, C18, C19, C20, C21, C22, C23, C24, C25, C26, C27, C28, C29, C30, C31, C32, C33, C34, C35, C36, C37, C38, C39, C4, C40, C41, C42, C43, C44, C45, C46, C47, C48, C49, C5, C50, C51, C52, C53, C54, C55, C56, C57, C58, C59, C6, C60, C61, C62, C63, C64, C65, C66, C67, C68, C69, C7, C70, C71, C72, C73, C74, C75, C76, C77, C78, C79, C8, C80, C81, C82, C83, C84, C85, C86, C87, C88, C89, C9, C90: C, Capacitor_SMD:C_0402_1005Metric, symbol Device:C
- added D100, D101, D102, D103, D104, D105, D106, D107, D108, D109, D110, D111, D112, D113, D114, D115, D116, D117, D118, D119, D120, D121, D122, D123, D124, D125, D126, D127, D128, D129, D130, D131, D132, D133, D134, D135, D136, D137, D138, D139, D140, D141, D142, D143, D144, D145, D146, D147, D148, D149, D150, D151, D152, D153, D154, D155, D156, D157, D158, D159, D160, D161, D162, D163, D164, D165, D166, D167, D168, D169, D170, D171, D172, D173, D174, D86, D87, D88, D89, D90, D91, D92, D93, D94, D95, D96, D97, D98, D99: LED, LED_SMD:LED_SK6812MINI_PLCC4_3.5x3.5mm_P1.75mm, symbol LED:SK6812MINI
- C1, C2, C3: footprint Capacitor_SMD:C_01005_0402Metric -> Capacitor_SMD:C_0402_1005Metric
- D85: renamed from D73; value DIODE -> LED; footprint Diode_SMD:D_SOD-123 -> LED_SMD:LED_SK6812MINI_PLCC4_3.5x3.5mm_P1.75mm
Connections:
- net labels added: 5V, INPUT, VDD
- wire segments 2 -> 10

Commit message: laying out keyboard, for final mfg
Parts:
- removed C10, C11, C12, C13, C14, C15, C16, C17, C18, C19, C2, C20, C21, C22, C23, C24, C25, C26, C27, C28, C29, C3, C30, C31, C32, C33, C34, C35, C36, C37, C38, C39, C40, C41, C42, C43, C44, C45, C46, C47, C48, C49, C5, C50, C51, C52, C53, C54, C55, C56, C57, C58, C59, C6, C60, C61, C62, C63, C64, C65, C66, C67, C68, C69, C70, C71, C72, C73, C74, C75, C76, C77, C78, C79, C8, C80, C81, C82, C83, C84, C85, C86, C87, C88, C89, C9, C90: C, Capacitor_SMD:C_0402_1005Metric, symbol Device:C
- removed D100, D101, D102, D103, D104, D105, D106, D107, D108, D109, D110, D111, D112, D113, D114, D115, D116, D117, D118, D119, D120, D121, D122, D123, D124, D125, D126, D127, D128, D129, D130, D131, D132, D133, D134, D135, D136, D137, D138, D139, D140, D141, D142, D143, D144, D145, D146, D147, D148, D149, D150, D151, D152, D153, D154, D155, D156, D157, D158, D159, D160, D161, D162, D163, D164, D165, D166, D167, D168, D169, D170, D171, D172, D173, D174, D86, D87, D89, D90, D92, D93, D94, D95, D96, D97, D98, D99: LED, LED_SMD:LED_SK6812MINI_PLCC4_3.5x3.5mm_P1.75mm, symbol LED:SK6812MINI
- D85, D88, D91: footprint LED_SMD:LED_SK6812MINI_PLCC4_3.5x3.5mm_P1.75mm -> daprice-keyswitches:LED_SK6812MINI_PLCC4_3.5x3.5mm_P1.75mm; symbol LED:SK6812MINI -> Cherry-Symbol:SK6812MINI
Connections:
- net labels removed: LED_INPUT
- wire segments 10 -> 7
- no-connect marks 0 -> 1
Other:
- moved on the sheet: C1, C4, C7

Commit message: placed LED's ..mostly
Parts:
- added C10, C11, C12, C13, C14, C15, C16, C17, C18, C19, C20, C21, C22, C23, C24, C25, C26, C27, C28, C29, C30, C31, C32, C33, C34, C35, C36, C37, C38, C39, C4, C40, C41, C42, C43, C44, C45, C46, C47, C48, C49, C5, C50, C51, C52, C53, C54, C55, C56, C57, C58, C59, C6, C60, C61, C62, C63, C64, C65, C66, C67, C68, C69, C7, C70, C71, C72, C73, C74, C75, C76, C77, C78, C79, C8, C80, C81, C82, C83, C9: C, Capacitor_SMD:C_0402_1005Metric, symbol Device:C
- added D100, D101, D102, D103, D104, D105, D106, D107, D108, D109, D110, D111, D112, D113, D114, D115, D116, D117, D118, D119, D120, D121, D122, D123, D124, D125, D126, D127, D128, D129, D130, D131, D132, D133, D134, D135, D136, D137, D138, D139, D140, D141, D142, D143, D144, D145, D146, D147, D148, D149, D150, D151, D152, D153, D154, D155, D156, D157, D158, D159, D160, D161, D162, D163, D164, D165, D166, D167, D88, D89, D90, D91, D92, D93, D94, D95, D96, D97, D98, D99: LED, daprice-keyswitches:LED_SK6812MINI_PLCC4_3.5x3.5mm_P1.75mm, symbol chgray-keyboard-rescue:SK6812MINI-Cherry-Symbol
- D85: symbol Cherry-Symbol:SK6812MINI -> chgray-keyboard-rescue:SK6812MINI-Cherry-Symbol
- D86: renamed from D88; symbol Cherry-Symbol:SK6812MINI -> chgray-keyboard-rescue:SK6812MINI-Cherry-Symbol
- D87: renamed from D91; symbol Cherry-Symbol:SK6812MINI -> chgray-keyboard-rescue:SK6812MINI-Cherry-Symbol
- renumbered C4 to C2, C7 to C3
Connections:
- wire segments 7 -> 185
Other:
- moved on the sheet: C2, C3

Commit message: placed LED's ..mostly
Parts:
- added C?: C, Capacitor_SMD:C_0402_1005Metric, symbol Device:C
- added D?: LED, daprice-keyswitches:LED_SK6812MINI_PLCC4_3.5x3.5mm_P1.75mm, symbol chgray-keyboard-rescue:SK6812MINI-Cherry-Symbol
Connections:
- net LED_VDD: now also D?.1 (VDD)
- net VCC_5V: now also C?.2
- net at D167.2 (DOUT): now also D?.4 (DIN)
- new net: C?.1, D?.3 (VSS)
Changed lines of the file:
@@
 Wire Wire Line
 	2100 10100 2300 10100
-NoConn ~ 3500 10100
+$Comp
+L chgray-keyboard-rescue:SK6812MINI-Cherry-Symbol D?
+U 1 1 60BC5CAF
+P 3800 10100
+AR Path="/60BC5CAF" Ref="D?"  Part="1"
+AR Path="/6096EA02/60BC5CAF" Ref="D?"  Part="1"
+F 0 "D?" H 4144 10146 50  0000 L CNN
+F 1 "LED" H 4144 10055 50  0000 L CNN
+F 2 "daprice-keyswitches:LED_SK6812MINI_PLCC4_3.5x3.5mm_P1.75mm" H 3850 9800 50  0000 L TNN
+F 3 "" H 3900 9725 50  0001 L TNN
+	1    3800 10100
+	1    0    0    -1
+$EndComp
+$Comp
+L Device:C C?
+U 1 1 60BC5CB5
+P 3800 10650
+F 0 "C?" H 3915 10696 50  0000 L CNN
+F 1 "C" H 3915 10605 50  0000 L CNN
+F 2 "Capacitor_SMD:C_0402_1005Metric" H 3838 10500 50  0001 C CNN
+F 3 "~" H 3800 10650 50  0001 C CNN
+	1    3800 10650
+	1    0    0    -1
+$EndComp
+Text GLabel 3800 9750 1    50   Input ~ 0
+LED_VDD
+Text GLabel 3800 10800 3    50   Input ~ 0
+VCC_5V
+Wire Wire Line
+	3800 9800 3800 9750
+Wire Wire Line
+	3800 10400 3800 10500
+NoConn ~ 4100 10100
 $EndSCHEMATC

Commit message: placed LED's ..mostly
Parts:
- gave numbers to parts that had none: 2
Changed lines of the file:
@@
 P 3800 10100
 AR Path="/60BC5CAF" Ref="D?"  Part="1"
-AR Path="/6096EA02/60BC5CAF" Ref="D?"  Part="1"
-F 0 "D?" H 4144 10146 50  0000 L CNN
+AR Path="/6096EA02/60BC5CAF" Ref="D168"  Part="1"
+F 0 "D168" H 4144 10146 50  0000 L CNN
 F 1 "LED" H 4144 10055 50  0000 L CNN
 F 2 "daprice-keyswitches:LED_SK6812MINI_PLCC4_3.5x3.5mm_P1.75mm" H 3850 9800 50  0000 L TNN
@@
 $EndComp
 $Comp
-L Device:C C?
+L Device:C C84
 U 1 1 60BC5CB5
 P 3800 10650
-F 0 "C?" H 3915 10696 50  0000 L CNN
+F 0 "C84" H 3915 10696 50  0000 L CNN
 F 1 "C" H 3915 10605 50  0000 L CNN
 F 2 "Capacitor_SMD:C_0402_1005Metric" H 3838 10500 50  0001 C CNN

Commit message: keyboard
Changed lines of the file:
@@
 Text GLabel 2600 3050 3    50   Input ~ 0
 VCC_5V
-Text GLabel 1300 950  2    50   Input ~ 0
-LED_VDD
-Text GLabel 1300 800  2    50   Input ~ 0
+Text GLabel 1600 950  2    50   Input ~ 0
+LED_VDD
+Text GLabel 1600 800  2    50   Input ~ 0
 VCC_5V
 Text HLabel 1300 800  0    50   Input ~ 0
@@
 	3800 10400 3800 10500
 NoConn ~ 4100 10100
+Wire Wire Line
+	1300 950  1600 950
+Wire Wire Line
+	1300 800  1600 800
 $EndSCHEMATC

Commit message: Logan signed off on board location
Parts:
- C1, C10, C11, C12, C13, C14, C15, C16, C17, C18, C19, C2, C20, C21, C22, C23, C24, C25, C26, C27, C28, C29, C3, C30, C31, C32, C33, C34, C35, C36, C37, C38, C39, C4, C40, C41, C42, C43, C44, C45, C46, C47, C48, C49, C5, C50, C51, C52, C53, C54, C55, C56, C57, C58, C59, C6, C60, C61, C62, C63, C64, C65, C66, C67, C68, C69, C7, C70, C71, C72, C73, C74, C75, C76, C77, C78, C79, C8, C80, C81, C82, C83, C84, C9: value C -> C104 0.1uF 100nF
Connections:
- net at D85.2 (DOUT): now also D86.4 (DIN)

Commit message: Logan signed off on board location
Parts:
- removed C12, C18, C6: C104 0.1uF 100nF, Capacitor_SMD:C_0402_1005Metric, symbol Device:C
- added C85, C86, C87: C104 0.1uF 100nF, Capacitor_SMD:C_0402_1005Metric, symbol Device:C
- renumbered D88 to D100, D109 to D101, D129 to D102, D149 to D103, D89 to D104, D110 to D105, D130 to D106, D150 to D107, D90 to D108, D111 to D109, D131 to D110, D151 to D111, D91 to D112, D112 to D113, D132 to D114, D152 to D115, D92 to D116, D113 to D117, D133 to D118, D153 to D119, D93 to D120, D114 to D121, D134 to D122, D154 to D123, D94 to D124, D115 to D125, D135 to D126, D155 to D127, D95 to D128, D116 to D129, D136 to D130, D156 to D131, D96 to D132, D117 to D133, D137 to D134, D157 to D135, D97 to D136, D118 to D137, D158 to D139, D98 to D140, D119 to D141, D139 to D142, D159 to D143, D99 to D144, D120 to D145, D140 to D146, D160 to D147, D100 to D148, D121 to D149, D141 to D150, D161 to D151, D101 to D152, D122 to D153, D142 to D154, D162 to D155, D102 to D156, D123 to D157, D143 to D158, D163 to D159, D103 to D160, D124 to D161, D144 to D162, D164 to D163, D104 to D164, D125 to D165, D145 to D166, D165 to D167, D105 to D168, D106 to D86, D126 to D87, D146 to D88, D166 to D89, D86 to D90, D107 to D91, D127 to D92, D147 to D93, D167 to D94, D87 to D95, D108 to D96, D128 to D97, D148 to D98, D168 to D99
Connections:
- net VCC_5V is gone; now on net LED_5V: C1.2, C10.2, C11.2, C13.2, C14.2, C15.2, C16.2, C17.2, C19.2, C2.2, C20.2, C21.2, C22.2, C23.2, C24.2, C25.2, C26.2, C27.2, C28.2, C29.2, C3.2, C30.2, C31.2, C32.2, C33.2, C34.2, C35.2, C36.2, C37.2, C38.2, C39.2, C4.2, C40.2, C41.2, C42.2, C43.2, C44.2, C45.2, C46.2, C47.2, C48.2, C49.2, C5.2, C50.2, C51.2, C52.2, C53.2, C54.2, C55.2, C56.2, C57.2, C58.2, C59.2, C60.2, C61.2, C62.2, C63.2, C64.2, C65.2, C66.2, C67.2, C68.2, C69.2, C7.2, C70.2, C71.2, C72.2, C73.2, C74.2, C75.2, C76.2, C77.2, C78.2, C79.2, C8.2, C80.2, C81.2, C82.2, C83.2, C84.2, C9.2
- net LED_GND: now reaches C1.1, D85.3 (VSS)
- net LED_GND: now also C10.1, C11.1, C13.1, C14.1, C15.1, C16.1, C17.1, C19.1, C2.1, C20.1, C21.1, C22.1, C23.1, C24.1, C25.1, C26.1, C27.1, C28.1, C29.1, C3.1, C30.1, C31.1, C32.1, C33.1, C34.1, C35.1, C36.1, C37.1, C38.1, C39.1, C4.1, C40.1, C41.1, C42.1, C43.1, C44.1, C45.1, C46.1, C47.1, C48.1, C49.1, C5.1, C50.1, C51.1, C52.1, C53.1, C54.1, C55.1, C56.1, C57.1, C58.1, C59.1, C60.1, C61.1, C62.1, C63.1, C64.1, C65.1, C66.1, C67.1, C68.1, C69.1, C7.1, C70.1, C71.1, C72.1, C73.1, C74.1, C75.1, C76.1, C77.1, C78.1, C79.1, C8.1, C80.1, C81.1, C82.1, C83.1, C84.1, C9.1, D100.3 (VSS), D101.3 (VSS), D102.3 (VSS), D103.3 (VSS), D104.3 (VSS), D105.3 (VSS), D106.3 (VSS), D107.3 (VSS), D108.3 (VSS), D109.3 (VSS), D110.3 (VSS), D111.3 (VSS), D112.3 (VSS), D113.3 (VSS), D114.3 (VSS), D115.3 (VSS), D116.3 (VSS), D117.3 (VSS), D118.3 (VSS), D119.3 (VSS), D120.3 (VSS), D121.3 (VSS), D122.3 (VSS), D123.3 (VSS), D124.3 (VSS), D125.3 (VSS), D126.3 (VSS), D127.3 (VSS), D128.3 (VSS), D129.3 (VSS), D130.3 (VSS), D131.3 (VSS), D132.3 (VSS), D133.3 (VSS), D134.3 (VSS), D135.3 (VSS), D136.3 (VSS), D137.3 (VSS), D138.3 (VSS), D139.3 (VSS), D140.3 (VSS), D141.3 (VSS), D142.3 (VSS), D143.3 (VSS), D144.3 (VSS), D145.3 (VSS), D146.3 (VSS), D147.3 (VSS), D148.3 (VSS), D149.3 (VSS), D150.3 (VSS), D151.3 (VSS), D152.3 (VSS), D153.3 (VSS), D154.3 (VSS), D155.3 (VSS), D156.3 (VSS), D157.3 (VSS), D158.3 (VSS), D159.3 (VSS), D160.3 (VSS), D161.3 (VSS), D162.3 (VSS), D163.3 (VSS), D164.3 (VSS), D165.3 (VSS), D166.3 (VSS), D167.3 (VSS), D168.3 (VSS), D86.3 (VSS), D87.3 (VSS), D88.3 (VSS), D89.3 (VSS), D90.3 (VSS), D91.3 (VSS), D92.3 (VSS), D93.3 (VSS), D94.3 (VSS), D95.3 (VSS), D96.3 (VSS), D97.3 (VSS), D98.3 (VSS), D99.3 (VSS), C85.1, C86.1, C87.1
- net LED_VDD renamed LED_5V
- net LED_5V: now also C85.2, C86.2, C87.2
Other:
- moved on the sheet: D85
