File: RGB-Circuit.sch (KiCad schematic (older format))
At the start: 168 parts

Commit message: working on the chip
Parts:
- renumbered C11 to C10, C13 to C11, C14 to C12, C15 to C13, C16 to C14, C17 to C15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

Commit message: RGB circuit rescue cleanup
Parts:
- D? (x84): symbol chgray-keyboard-rescue:SK6812MINI-Cherry-Symbol -> LED:SK6812MINI

Commit message: update keyboard
Parts:
- gave numbers to parts that had none: 84
