File: chgray-keyboard.kicad_pcb (KiCad board)
At the start: 2 copper layers, 377.4 x 105.5 mm, 338 parts, among them J1 Conn_01x01_Female, SW1 30, SW10 22, SW11 32, SW12 52, SW13 02, SW14 12, SW15 03, SW16 13, SW17 23, SW18 33, SW19 43, SW2 40, SW20 53, SW21 24, SW22 34, SW23 54, SW24 04, SW25 14, SW26 05, SW27 15, SW28 25, SW29 35, SW3 50, SW30 45, SW31 26, SW32 36, SW33 46, SW34 56, SW35 06, SW36 16, SW37 07, SW38 17, SW39 27, SW4 00, SW40 37, SW41 57, SW42 28, SW43 38, SW44 48, SW45 58, SW46 08, SW47 18, SW48 09, SW49 19, SW5 01, SW50 29, SW51 39, SW52 49, SW53 010, SW54 110, SW55 210, SW56 310, SW57 410, SW58 510, SW59 111, SW6 11, SW60 211, SW61 311, SW62 411, SW63 511, SW64 111, SW65 211, SW66 311, SW67 411, SW68 511, SW69 111, SW7 21, SW70 211, SW71 311, SW72 411, SW73 511, SW8 41, SW9 51, U1 Teensy2.0_(C)

Commit message: Logan signed off on board location
Routing:
- net LED_VDD: track 0.00 -> 2156.4 mm, vias 0 -> 21
- net /Keyboard Keys/KEY_ROW4: track 0.00 -> 597.6 mm, vias 0 -> 11
- net /Keyboard Keys/KEY_ROW0: track 0.00 -> 590.5 mm, vias 0 -> 9
- net /Keyboard Keys/KEY_ROW2: track 0.00 -> 562.1 mm, vias 0 -> 10
- net /Keyboard Keys/KEY_ROW3: track 0.00 -> 557.4 mm, vias 0 -> 13
- net /Keyboard Keys/KEY_COL0: track 0.00 -> 536.2 mm, vias 0 -> 8
- net /Keyboard Keys/KEY_ROW1: track 0.00 -> 491.2 mm, vias 0 -> 7
- net /Keyboard Keys/KEY_ROW5: track 0.00 -> 489.3 mm, vias 0 -> 13
- net /Keyboard Keys/KEY_COL2: track 0.00 -> 480.7 mm, vias 0 -> 10
- net /Keyboard Keys/KEY_COL13: track 0.00 -> 439.9 mm, vias 0 -> 5
- net Net-(C70-Pad1): track 0.00 -> 435.1 mm, vias 0 -> 4
- net Net-(D82-Pad1): track 0.00 -> 430.7 mm, vias 0 -> 6
- net /Keyboard Keys/KEY_COL3: track 0.00 -> 395.9 mm, vias 0 -> 8
- net Net-(C2-Pad1): track 0.00 -> 394.0 mm, vias 0 -> 4
- net /Keyboard Keys/KEY_COL1: track 0.00 -> 385.9 mm, vias 0 -> 4
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
Commit message: Logan signed off on board location
Parts:
- removed C12, C18, C6: C104 0.1uF 100nF, Capacitor_SMD:C_0402_1005Metric
- added C85: C104 0.1uF 100nF, Capacitor_SMD:C_0402_1005Metric, F.Cu at (306.1, 146.0)
- added C86: C104 0.1uF 100nF, Capacitor_SMD:C_0402_1005Metric, F.Cu at (298.2, 153.3)
- added C87: C104 0.1uF 100nF, Capacitor_SMD:C_0402_1005Metric, F.Cu at (302.0, 152.7)
- C1, C10, C11, C13, C14, C15, C16, C17, C19, C2, C20, C21, C22, C23, C24, C25, C26, C27, C28, C29, C3, C30, C31, C32, C33, C34, C35, C36, C37, C38, C39, C4, C40, C41, C42, C43, C44, C45, C46, C47, C48, C49, C5, C50, C51, C52, C53, C54, C55, C56, C57, C58, C59, C60, C61, C62, C63, C64, C65, C66, C67, C68, C69, C7, C70, C71, C72, C73, C74, C75, C76, C77, C78, C79, C8, C80, C81, C82, C83, C84, C9: moved to F.Cu
- moved D3 230.3 mm to (306.4, 160.6)
- moved D11 206.4 mm to (306.4, 163.7)
- moved D15 184.6 mm to (306.4, 151.4)
- moved D23 160.7 mm to (306.4, 154.5)
- moved D73 129.5 mm to (300.7, 170.2)
- moved D27 113.7 mm to (306.4, 157.5)
- moved D35 88.7 mm to (306.4, 166.8)
- moved D39 64.9 mm to (306.4, 169.8)
- moved C2 58.4 mm to (298.2, 114.6)
- moved C21 56.1 mm to (306.1, 118.3)
- moved C8 55.4 mm to (298.2, 117.7)
- moved C23 49.1 mm to (298.2, 122.3)
- moved C35 48.7 mm to (302.0, 117.8)
- moved C3 47.1 mm to (302.0, 113.0)
- moved C40 46.8 mm to (306.1, 122.9)
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- renumbered D88 to D100, D109 to D101, D129 to D102, D149 to D103, D89 to D104, D110 to D105, D130 to D106, D150 to D107, D90 to D108, D111 to D109, D131 to D110, D151 to D111, D91 to D112, D112 to D113, D132 to D114, D152 to D115, D92 to D116, D113 to D117, D133 to D118, D153 to D119, D93 to D120, D114 to D121, D134 to D122, D154 to D123, D94 to D124, D115 to D125, D135 to D126, D155 to D127, D95 to D128, D116 to D129, D136 to D130, D156 to D131, D96 to D132, D117 to D133, D137 to D134, D157 to D135, D97 to D136, D118 to D137, D158 to D139, D98 to D140, D119 to D141, D139 to D142, D159 to D143, D99 to D144, D120 to D145, D140 to D146, D160 to D147, D100 to D148, D121 to D149, D141 to D150, D161 to D151, D101 to D152, D122 to D153, D142 to D154, D162 to D155, D102 to D156, D123 to D157, D143 to D158, D163 to D159, D103 to D160, D124 to D161, D144 to D162, D164 to D163, D104 to D164, D125 to D165, D145 to D166, D165 to D167, D105 to D168, D106 to D86, D126 to D87, D146 to D88, D166 to D89, D86 to D90, D107 to D91, D127 to D92, D147 to D93, D167 to D94, D87 to D95, D108 to D96, D128 to D97, D148 to D98, D168 to D99
Connections:
- net GND renamed TEENSY_GND
- net Net-(J1-Pad13) renamed PWR_5V
- C1 pad 1: Net-(C1-Pad1) -> LED_GND
- C1 pad 2: VCC_5V -> LED_5V
- C10 pad 1: Net-(C10-Pad1) -> LED_GND
- C10 pad 2: VCC_5V -> LED_5V
- C11 pad 1: Net-(C11-Pad1) -> LED_GND
- C11 pad 2: VCC_5V -> LED_5V
- C13 pad 1: Net-(C13-Pad1) -> LED_GND
- C13 pad 2: VCC_5V -> LED_5V
- C14 pad 1: Net-(C14-Pad1) -> LED_GND
- C14 pad 2: VCC_5V -> LED_5V
- C15 pad 1: Net-(C15-Pad1) -> LED_GND
- C15 pad 2: VCC_5V -> LED_5V
- C16 pad 1: Net-(C16-Pad1) -> LED_GND
- C16 pad 2: VCC_5V -> LED_5V
- C17 pad 1: Net-(C17-Pad1) -> LED_GND
- C17 pad 2: VCC_5V -> LED_5V
- C19 pad 1: Net-(C19-Pad1) -> LED_GND
- C19 pad 2: VCC_5V -> LED_5V
- C2 pad 1: Net-(C2-Pad1) -> LED_GND
- C2 pad 2: VCC_5V -> LED_5V
- C20 pad 1: Net-(C20-Pad1) -> LED_GND
- C20 pad 2: VCC_5V -> LED_5V
- C21 pad 1: Net-(C21-Pad1) -> LED_GND
- C21 pad 2: VCC_5V -> LED_5V
- C22 pad 1: Net-(C22-Pad1) -> LED_GND
- C22 pad 2: VCC_5V -> LED_5V
- C23 pad 1: Net-(C23-Pad1) -> LED_GND
- C23 pad 2: VCC_5V -> LED_5V
- C24 pad 1: Net-(C24-Pad1) -> LED_GND
- C24 pad 2: VCC_5V -> LED_5V
- C25 pad 1: Net-(C25-Pad1) -> LED_GND
- C25 pad 2: VCC_5V -> LED_5V
- C26 pad 1: Net-(C26-Pad1) -> LED_GND
- C26 pad 2: VCC_5V -> LED_5V
- C27 pad 1: Net-(C27-Pad1) -> LED_GND
- C27 pad 2: VCC_5V -> LED_5V
- C28 pad 1: Net-(C28-Pad1) -> LED_GND
- C28 pad 2: VCC_5V -> LED_5V
- C29 pad 1: Net-(C29-Pad1) -> LED_GND
- C29 pad 2: VCC_5V -> LED_5V
- C3 pad 1: Net-(C3-Pad1) -> LED_GND
- C3 pad 2: VCC_5V -> LED_5V
- C30 pad 1: Net-(C30-Pad1) -> LED_GND
- C30 pad 2: VCC_5V -> LED_5V
- C31 pad 1: Net-(C31-Pad1) -> LED_GND
- C31 pad 2: VCC_5V -> LED_5V
- C32 pad 1: Net-(C32-Pad1) -> LED_GND
- C32 pad 2: VCC_5V -> LED_5V
- C33 pad 1: Net-(C33-Pad1) -> LED_GND
- C33 pad 2: VCC_5V -> LED_5V
- C34 pad 1: Net-(C34-Pad1) -> LED_GND
- C34 pad 2: VCC_5V -> LED_5V
- C35 pad 1: Net-(C35-Pad1) -> LED_GND
- C35 pad 2: VCC_5V -> LED_5V
- C36 pad 1: Net-(C36-Pad1) -> LED_GND
- C36 pad 2: VCC_5V -> LED_5V
- C37 pad 1: Net-(C37-Pad1) -> LED_GND
- C37 pad 2: VCC_5V -> LED_5V
- C38 pad 1: Net-(C38-Pad1) -> LED_GND
- C38 pad 2: VCC_5V -> LED_5V
- C39 pad 1: Net-(C39-Pad1) -> LED_GND
- C39 pad 2: VCC_5V -> LED_5V
- C4 pad 1: Net-(C4-Pad1) -> LED_GND
- C4 pad 2: VCC_5V -> LED_5V
- C40 pad 1: Net-(C40-Pad1) -> LED_GND
- C40 pad 2: VCC_5V -> LED_5V
- C41 pad 1: Net-(C41-Pad1) -> LED_GND
- C41 pad 2: VCC_5V -> LED_5V
- C42 pad 1: Net-(C42-Pad1) -> LED_GND
- C42 pad 2: VCC_5V -> LED_5V
- C43 pad 1: Net-(C43-Pad1) -> LED_GND
- C43 pad 2: VCC_5V -> LED_5V
- C44 pad 1: Net-(C44-Pad1) -> LED_GND
- C44 pad 2: VCC_5V -> LED_5V
- C45 pad 1: Net-(C45-Pad1) -> LED_GND
- C45 pad 2: VCC_5V -> LED_5V
- C46 pad 1: Net-(C46-Pad1) -> LED_GND
- C46 pad 2: VCC_5V -> LED_5V
- C47 pad 1: Net-(C47-Pad1) -> LED_GND
- C47 pad 2: VCC_5V -> LED_5V
- C48 pad 1: Net-(C48-Pad1) -> LED_GND
- C48 pad 2: VCC_5V -> LED_5V
- C49 pad 1: Net-(C49-Pad1) -> LED_GND
- C49 pad 2: VCC_5V -> LED_5V
- C5 pad 1: Net-(C5-Pad1) -> LED_GND
- C5 pad 2: VCC_5V -> LED_5V
- C50 pad 1: Net-(C50-Pad1) -> LED_GND
- C50 pad 2: VCC_5V -> LED_5V
- C51 pad 1: Net-(C51-Pad1) -> LED_GND
- C51 pad 2: VCC_5V -> LED_5V
- C52 pad 1: Net-(C52-Pad1) -> LED_GND
- C52 pad 2: VCC_5V -> LED_5V
- C53 pad 1: Net-(C53-Pad1) -> LED_GND
- C53 pad 2: VCC_5V -> LED_5V
- C54 pad 1: Net-(C54-Pad1) -> LED_GND
- C54 pad 2: VCC_5V -> LED_5V
- C55 pad 1: Net-(C55-Pad1) -> LED_GND
- C55 pad 2: VCC_5V -> LED_5V
- C56 pad 1: Net-(C56-Pad1) -> LED_GND
- C56 pad 2: VCC_5V -> LED_5V
- C57 pad 1: Net-(C57-Pad1) -> LED_GND
- C57 pad 2: VCC_5V -> LED_5V
- C58 pad 1: Net-(C58-Pad1) -> LED_GND
- C58 pad 2: VCC_5V -> LED_5V
- C59 pad 1: Net-(C59-Pad1) -> LED_GND
- C59 pad 2: VCC_5V -> LED_5V
- C60 pad 1: Net-(C60-Pad1) -> LED_GND
- C60 pad 2: VCC_5V -> LED_5V
- C61 pad 1: Net-(C61-Pad1) -> LED_GND
- C61 pad 2: VCC_5V -> LED_5V
- C62 pad 1: Net-(C62-Pad1) -> LED_GND
- C62 pad 2: VCC_5V -> LED_5V
- C63 pad 1: Net-(C63-Pad1) -> LED_GND
- C63 pad 2: VCC_5V -> LED_5V
- C64 pad 1: Net-(C64-Pad1) -> LED_GND
- C64 pad 2: VCC_5V -> LED_5V
- C65 pad 1: Net-(C65-Pad1) -> LED_GND
- C65 pad 2: VCC_5V -> LED_5V
- C66 pad 1: Net-(C66-Pad1) -> LED_GND
- C66 pad 2: VCC_5V -> LED_5V
- C67 pad 1: Net-(C67-Pad1) -> LED_GND
- C67 pad 2: VCC_5V -> LED_5V
- C68 pad 1: Net-(C68-Pad1) -> LED_GND
- C68 pad 2: VCC_5V -> LED_5V
- C69 pad 1: Net-(C69-Pad1) -> LED_GND
- C69 pad 2: VCC_5V -> LED_5V
- C7 pad 1: Net-(C7-Pad1) -> LED_GND
- C7 pad 2: VCC_5V -> LED_5V
- C70 pad 1: Net-(C70-Pad1) -> LED_GND
- C70 pad 2: VCC_5V -> LED_5V
- C71 pad 1: Net-(C71-Pad1) -> LED_GND
- C71 pad 2: VCC_5V -> LED_5V
- C72 pad 1: Net-(C72-Pad1) -> LED_GND
- C72 pad 2: VCC_5V -> LED_5V
- C73 pad 1: Net-(C73-Pad1) -> LED_GND
- C73 pad 2: VCC_5V -> LED_5V
- C74 pad 1: Net-(C74-Pad1) -> LED_GND
- C74 pad 2: VCC_5V -> LED_5V
- C75 pad 1: Net-(C75-Pad1) -> LED_GND
- C75 pad 2: VCC_5V -> LED_5V
- C76 pad 1: Net-(C76-Pad1) -> LED_GND
- C76 pad 2: VCC_5V -> LED_5V
- C77 pad 1: Net-(C77-Pad1) -> LED_GND
- C77 pad 2: VCC_5V -> LED_5V
- C78 pad 1: Net-(C78-Pad1) -> LED_GND
- C78 pad 2: VCC_5V -> LED_5V
- C79 pad 1: Net-(C79-Pad1) -> LED_GND
- C79 pad 2: VCC_5V -> LED_5V
- C8 pad 1: Net-(C8-Pad1) -> LED_GND
- C8 pad 2: VCC_5V -> LED_5V
- C80 pad 1: Net-(C80-Pad1) -> LED_GND
- C80 pad 2: VCC_5V -> LED_5V
- C81 pad 1: Net-(C81-Pad1) -> LED_GND
- C81 pad 2: VCC_5V -> LED_5V
- C82 pad 1: Net-(C82-Pad1) -> LED_GND
- C82 pad 2: VCC_5V -> LED_5V
- C83 pad 1: Net-(C83-Pad1) -> LED_GND
- C83 pad 2: VCC_5V -> LED_5V
- C84 pad 1: Net-(C84-Pad1) -> LED_GND
- C84 pad 2: VCC_5V -> LED_5V
- C9 pad 1: Net-(C9-Pad1) -> LED_GND
- C9 pad 2: VCC_5V -> LED_5V
- D100 pad 1: LED_VDD -> LED_5V
- D100 pad 3: Net-(C4-Pad1) -> LED_GND
- D101 pad 1: LED_VDD -> LED_5V
- D101 pad 3: Net-(C25-Pad1) -> LED_GND
- D102 pad 1: LED_VDD -> LED_5V
- D102 pad 3: Net-(C45-Pad1) -> LED_GND
- D103 pad 1: LED_VDD -> LED_5V
- D103 pad 3: Net-(C65-Pad1) -> LED_GND
- D104 pad 1: LED_VDD -> LED_5V
- D104 pad 3: Net-(C5-Pad1) -> LED_GND
- D105 pad 1: LED_VDD -> LED_5V
- D105 pad 3: Net-(C26-Pad1) -> LED_GND
- D106 pad 1: LED_VDD -> LED_5V
- D106 pad 3: Net-(C46-Pad1) -> LED_GND
- D107 pad 1: LED_VDD -> LED_5V
- D107 pad 3: Net-(C66-Pad1) -> LED_GND
- D108 pad 1: LED_VDD -> LED_5V
- D108 pad 3: Net-(C6-Pad1) -> LED_GND
- D109 pad 1: LED_VDD -> LED_5V
- D109 pad 3: Net-(C27-Pad1) -> LED_GND
- D110 pad 1: LED_VDD -> LED_5V
- D110 pad 3: Net-(C47-Pad1) -> LED_GND
- D111 pad 1: LED_VDD -> LED_5V
- D111 pad 3: Net-(C67-Pad1) -> LED_GND
- D112 pad 1: LED_VDD -> LED_5V
- D112 pad 3: Net-(C7-Pad1) -> LED_GND
- D113 pad 1: LED_VDD -> LED_5V
- D113 pad 3: Net-(C28-Pad1) -> LED_GND
- D114 pad 1: LED_VDD -> LED_5V
- D114 pad 3: Net-(C48-Pad1) -> LED_GND
- D115 pad 1: LED_VDD -> LED_5V
- D115 pad 3: Net-(C68-Pad1) -> LED_GND
- D116 pad 1: LED_VDD -> LED_5V
- D116 pad 3: Net-(C8-Pad1) -> LED_GND
- D117 pad 1: LED_VDD -> LED_5V
- D117 pad 3: Net-(C29-Pad1) -> LED_GND
- D118 pad 1: LED_VDD -> LED_5V
- D118 pad 3: Net-(C49-Pad1) -> LED_GND
- D119 pad 1: LED_VDD -> LED_5V
- D119 pad 3: Net-(C69-Pad1) -> LED_GND
- D120 pad 1: LED_VDD -> LED_5V
- D120 pad 3: Net-(C9-Pad1) -> LED_GND
- D121 pad 1: LED_VDD -> LED_5V
- D121 pad 3: Net-(C30-Pad1) -> LED_GND
- D122 pad 1: LED_VDD -> LED_5V
- D122 pad 3: Net-(C50-Pad1) -> LED_GND
- D123 pad 1: LED_VDD -> LED_5V
- D123 pad 3: Net-(C70-Pad1) -> LED_GND
- D124 pad 1: LED_VDD -> LED_5V
- D124 pad 3: Net-(C10-Pad1) -> LED_GND
- D125 pad 1: LED_VDD -> LED_5V
- D125 pad 3: Net-(C31-Pad1) -> LED_GND
- D126 pad 1: LED_VDD -> LED_5V
- D126 pad 3: Net-(C51-Pad1) -> LED_GND
- D127 pad 1: LED_VDD -> LED_5V
- D127 pad 3: Net-(C71-Pad1) -> LED_GND
- D128 pad 1: LED_VDD -> LED_5V
- D128 pad 3: Net-(C11-Pad1) -> LED_GND
- D129 pad 1: LED_VDD -> LED_5V
- D129 pad 3: Net-(C32-Pad1) -> LED_GND
- D130 pad 1: LED_VDD -> LED_5V
- D130 pad 3: Net-(C52-Pad1) -> LED_GND
- D131 pad 1: LED_VDD -> LED_5V
- D131 pad 3: Net-(C72-Pad1) -> LED_GND
- D132 pad 1: LED_VDD -> LED_5V
- D132 pad 3: Net-(C12-Pad1) -> LED_GND
- D133 pad 1: LED_VDD -> LED_5V
- D133 pad 3: Net-(C33-Pad1) -> LED_GND
- D134 pad 1: LED_VDD -> LED_5V
- D134 pad 3: Net-(C53-Pad1) -> LED_GND
- D135 pad 1: LED_VDD -> LED_5V
- D135 pad 3: Net-(C73-Pad1) -> LED_GND
- D136 pad 1: LED_VDD -> LED_5V
- D136 pad 3: Net-(C13-Pad1) -> LED_GND
- D137 pad 1: LED_VDD -> LED_5V
- D137 pad 3: Net-(C34-Pad1) -> LED_GND
- D138 pad 1: LED_VDD -> LED_5V
- D138 pad 3: Net-(C54-Pad1) -> LED_GND
- D139 pad 1: LED_VDD -> LED_5V
- D139 pad 3: Net-(C74-Pad1) -> LED_GND
- D140 pad 1: LED_VDD -> LED_5V
- D140 pad 3: Net-(C14-Pad1) -> LED_GND
- D141 pad 1: LED_VDD -> LED_5V
- D141 pad 3: Net-(C35-Pad1) -> LED_GND
- D142 pad 1: LED_VDD -> LED_5V
- D142 pad 3: Net-(C55-Pad1) -> LED_GND
- D143 pad 1: LED_VDD -> LED_5V
- D143 pad 3: Net-(C75-Pad1) -> LED_GND
- D144 pad 1: LED_VDD -> LED_5V
- D144 pad 3: Net-(C15-Pad1) -> LED_GND
- D145 pad 1: LED_VDD -> LED_5V
- D145 pad 3: Net-(C36-Pad1) -> LED_GND
- D146 pad 1: LED_VDD -> LED_5V
- D146 pad 3: Net-(C56-Pad1) -> LED_GND
- D147 pad 1: LED_VDD -> LED_5V
- D147 pad 3: Net-(C76-Pad1) -> LED_GND
- D148 pad 1: LED_VDD -> LED_5V
- D148 pad 3: Net-(C16-Pad1) -> LED_GND
- D149 pad 1: LED_VDD -> LED_5V
- D149 pad 3: Net-(C37-Pad1) -> LED_GND
- D150 pad 1: LED_VDD -> LED_5V
- D150 pad 3: Net-(C57-Pad1) -> LED_GND
- D151 pad 1: LED_VDD -> LED_5V
- D151 pad 3: Net-(C77-Pad1) -> LED_GND
- D152 pad 1: LED_VDD -> LED_5V
- D152 pad 3: Net-(C17-Pad1) -> LED_GND
- D153 pad 1: LED_VDD -> LED_5V
- D153 pad 3: Net-(C38-Pad1) -> LED_GND
- D154 pad 1: LED_VDD -> LED_5V
- D154 pad 3: Net-(C58-Pad1) -> LED_GND
- D155 pad 1: LED_VDD -> LED_5V
- D155 pad 3: Net-(C78-Pad1) -> LED_GND
- D156 pad 1: LED_VDD -> LED_5V
- D156 pad 3: Net-(C18-Pad1) -> LED_GND
- D157 pad 1: LED_VDD -> LED_5V
- D157 pad 3: Net-(C39-Pad1) -> LED_GND
- D158 pad 1: LED_VDD -> LED_5V
- D158 pad 3: Net-(C59-Pad1) -> LED_GND
- D159 pad 1: LED_VDD -> LED_5V
- D159 pad 3: Net-(C79-Pad1) -> LED_GND
- D160 pad 1: LED_VDD -> LED_5V
- D160 pad 3: Net-(C19-Pad1) -> LED_GND
- D161 pad 1: LED_VDD -> LED_5V
- D161 pad 3: Net-(C40-Pad1) -> LED_GND
- D162 pad 1: LED_VDD -> LED_5V
- D162 pad 3: Net-(C60-Pad1) -> LED_GND
- D163 pad 1: LED_VDD -> LED_5V
- D163 pad 3: Net-(C80-Pad1) -> LED_GND
- D164 pad 1: LED_VDD -> LED_5V
- D164 pad 3: Net-(C20-Pad1) -> LED_GND
- D165 pad 1: LED_VDD -> LED_5V
- D165 pad 3: Net-(C41-Pad1) -> LED_GND
- D166 pad 1: LED_VDD -> LED_5V
- D166 pad 3: Net-(C61-Pad1) -> LED_GND
- D167 pad 1: LED_VDD -> LED_5V
- D167 pad 3: Net-(C81-Pad1) -> LED_GND
- D168 pad 1: LED_VDD -> LED_5V
- D168 pad 3: Net-(C21-Pad1) -> LED_GND
- D85 pad 1: LED_VDD -> LED_5V
- D85 pad 3: Net-(C1-Pad1) -> LED_GND
- D86 pad 1: LED_VDD -> LED_5V
- D86 pad 3: Net-(C22-Pad1) -> LED_GND
- D87 pad 1: LED_VDD -> LED_5V
- D87 pad 3: Net-(C42-Pad1) -> LED_GND
- D88 pad 1: LED_VDD -> LED_5V
- D88 pad 3: Net-(C62-Pad1) -> LED_GND
- D89 pad 1: LED_VDD -> LED_5V
- D89 pad 3: Net-(C82-Pad1) -> LED_GND
- D90 pad 1: LED_VDD -> LED_5V
- D90 pad 3: Net-(C2-Pad1) -> LED_GND
- D91 pad 1: LED_VDD -> LED_5V
- D91 pad 3: Net-(C23-Pad1) -> LED_GND
- D92 pad 1: LED_VDD -> LED_5V
- D92 pad 3: Net-(C43-Pad1) -> LED_GND
- D93 pad 1: LED_VDD -> LED_5V
- D93 pad 3: Net-(C63-Pad1) -> LED_GND
- D94 pad 1: LED_VDD -> LED_5V
- D94 pad 3: Net-(C83-Pad1) -> LED_GND
- D95 pad 1: LED_VDD -> LED_5V
- D95 pad 3: Net-(C3-Pad1) -> LED_GND
- D96 pad 1: LED_VDD -> LED_5V
- D96 pad 3: Net-(C24-Pad1) -> LED_GND
- D97 pad 1: LED_VDD -> LED_5V
- D97 pad 3: Net-(C44-Pad1) -> LED_GND
- D98 pad 1: LED_VDD -> LED_5V
- D98 pad 3: Net-(C64-Pad1) -> LED_GND
- D99 pad 1: LED_VDD -> LED_5V
- D99 pad 3: Net-(C84-Pad1) -> LED_GND
- J1 pad 14: VCC_5V -> LED_GND
- J1 pad 2: LED_VDD -> LED_5V
Routing:
- net LED_VDD: track 2156.4 -> 0.00 mm, vias 21 -> 0
- net /Keyboard Keys/KEY_ROW4: track 597.6 -> 0.00 mm, vias 11 -> 0
- net /Keyboard Keys/KEY_ROW0: track 590.5 -> 0.00 mm, vias 9 -> 0
- net /Keyboard Keys/KEY_ROW2: track 562.1 -> 0.00 mm, vias 10 -> 0
- net /Keyboard Keys/KEY_ROW3: track 557.4 -> 0.00 mm, vias 13 -> 0
- net /Keyboard Keys/KEY_COL0: track 536.2 -> 0.00 mm, vias 8 -> 0
- net /Keyboard Keys/KEY_ROW1: track 491.2 -> 0.00 mm, vias 7 -> 0
- net /Keyboard Keys/KEY_ROW5: track 489.3 -> 0.00 mm, vias 13 -> 0
- net /Keyboard Keys/KEY_COL2: track 480.7 -> 0.00 mm, vias 10 -> 0
- net /Keyboard Keys/KEY_COL13: track 439.9 -> 0.00 mm, vias 5 -> 0
- net Net-(C70-Pad1): track 435.1 -> 0.00 mm, vias 4 -> 0
- net Net-(D82-Pad1): track 430.7 -> 0.00 mm, vias 6 -> 0
- net /Keyboard Keys/KEY_COL3: track 395.9 -> 0.00 mm, vias 8 -> 0
- net Net-(C2-Pad1): track 394.0 -> 0.00 mm, vias 4 -> 0
- net /Keyboard Keys/KEY_COL1: track 385.9 -> 0.00 mm, vias 4 -> 0
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
Commit message: Logan signed off on board location
Routing:
- net LED_GND: track 0.00 -> 2325.2 mm, vias 0 -> 18
- net LED_5V: track 0.00 -> 2264.1 mm, vias 0 -> 17
- net /Keyboard Keys/KEY_ROW4: track 0.00 -> 595.9 mm, vias 0 -> 4
- net /Keyboard Keys/KEY_ROW3: track 0.00 -> 567.4 mm, vias 0 -> 10
- net /Keyboard Keys/KEY_ROW0: track 0.00 -> 496.6 mm, vias 0 -> 3
- net /Keyboard Keys/KEY_ROW2: track 0.00 -> 468.6 mm, vias 0 -> 9
- net /Keyboard Keys/KEY_ROW1: track 0.00 -> 460.9 mm, vias 0 -> 10
- net /Keyboard Keys/KEY_ROW5: track 0.00 -> 447.5 mm, vias 0 -> 7
- net /Keyboard Keys/KEY_COL13: track 0.00 -> 430.3 mm, vias 0 -> 7
- net /Keyboard Keys/KEY_COL2: track 0.00 -> 378.9 mm, vias 0 -> 3
- net Net-(D2-Pad1): track 0.00 -> 375.3 mm, vias 0 -> 2
- net /Keyboard Keys/KEY_COL1: track 0.00 -> 372.5 mm, vias 0 -> 1
- net /Keyboard Keys/KEY_COL0: track 0.00 -> 372.4 mm, vias 0 -> 7
- net /Keyboard Keys/KEY_COL5: track 0.00 -> 369.9 mm, vias 0 -> 9
- net /Keyboard Keys/KEY_COL6: track 0.00 -> 364.6 mm, vias 0 -> 5
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
Commit message: n-1 to sendoff
Parts:
- C1, C10, C11, C13, C14, C15, C16, C17, C19, C2, C20, C21, C22, C23, C24, C25, C26, C27, C28, C29, C3, C30, C31, C32, C33, C34, C35, C36, C37, C38, C39, C4, C40, C41, C42, C43, C44, C45, C46, C47, C48, C49, C5, C50, C51, C52, C53, C54, C55, C56, C57, C58, C59, C60, C61, C62, C63, C64, C65, C66, C67, C68, C69, C7, C70, C71, C72, C73, C74, C75, C76, C77, C78, C79, C8, C80, C81, C82, C83, C84, C85, C86, C87, C9: moved to B.Cu
- moved D50 118.5 mm to (353.2, 143.3)
- moved D58 89.6 mm to (363.8, 143.3)
- moved D60 61.2 mm to (374.4, 143.3)
- moved C14 47.0 mm to (298.2, 160.0)
- moved C82 45.9 mm to (298.2, 113.6)
- moved C3 45.1 mm to (302.0, 158.1)
- moved C2 43.9 mm to (298.2, 158.5)
- moved C83 43.8 mm to (302.0, 113.7)
- moved C75 42.8 mm to (298.2, 115.1)
- moved C5 41.9 mm to (302.0, 156.5)
- moved C4 40.8 mm to (298.2, 156.9)
- moved C46 40.7 mm to (302.0, 115.2)
- moved D61 40.5 mm to (227.2, 104.9)
- moved D5 40.5 mm to (35.2, 104.9)
- moved D7 40.3 mm to (54.4, 104.9)
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Routing:
- net Net-(J1-Pad5): track 283.1 -> 90.5 mm, vias 2 -> 0
- net LED_GND: track 2325.2 -> 2187.8 mm, vias 18 -> 14
- net Net-(D50-Pad1): track 66.7 -> 179.3 mm, vias 0 -> 2
- net /Keyboard Keys/KEY_COL9: track 238.8 -> 344.4 mm, vias 4 -> 8
- net /Keyboard Keys/KEY_COL0: track 372.4 -> 458.7 mm, vias 7 -> 12
- net Net-(D58-Pad1): track 92.4 -> 171.0 mm
- net /Keyboard Keys/KEY_COL4: track 323.7 -> 402.0 mm, vias 6 -> 9
- net Net-(Backspace1-Pad2): track 58.5 -> 136.6 mm, vias 2 -> 4
- net /Keyboard Keys/KEY_COL3: track 316.2 -> 387.9 mm, vias 6 -> 10
- net /Keyboard Keys/KEY_COL1: track 372.5 -> 444.1 mm, vias 1 -> 10
- net Net-(D77-Pad1): track 112.5 -> 49.0 mm, vias 2 -> 0
- net /Keyboard Keys/KEY_ROW5: track 447.5 -> 394.2 mm, vias 7 -> 6
- net /Keyboard Keys/KEY_ROW0: track 496.6 -> 546.0 mm, vias 3 -> 5
- net /Keyboard Keys/KEY_COL6: track 364.6 -> 413.9 mm, vias 5 -> 12
- net Net-(D61-Pad1): track 61.6 -> 16.5 mm
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
Commit message: n-1 to sendoff
Parts:
- moved C14 58.8 mm to (309.0, 102.2)
- moved C17 58.8 mm to (309.0, 94.5)
- moved C19 58.8 mm to (312.8, 86.0)
- moved C2 58.8 mm to (309.0, 100.7)
- moved C20 58.8 mm to (312.8, 94.0)
- moved C21 58.8 mm to (316.3, 86.8)
- moved C23 58.8 mm to (309.0, 92.9)
- moved C24 58.8 mm to (312.8, 84.5)
- moved C25 58.8 mm to (309.0, 96.0)
- moved C28 58.8 mm to (316.3, 85.3)
- moved C3 58.8 mm to (312.8, 100.3)
- moved C33 58.8 mm to (316.3, 83.7)
- moved C36 58.8 mm to (312.8, 92.4)
- moved C38 58.8 mm to (312.8, 78.1)
- moved C4 58.8 mm to (309.0, 99.1)
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Other:
- board text added: "LOG0.Key.Yeet2 May 14, 2021"
- board text removed: "LOG0.Key.Yeet2"

Commit message: update keyboard
Parts:
- removed U1: Teensy2.0_(C), Teensy_Pretty:Teensy2.0
- added U2: ATmega32U4-AU, Package_QFP:TQFP-44_10x10mm_P0.8mm, F.Cu at (349.9, -55.1)
- renumbered C11 to C10, C13 to C11, C14 to C12, C15 to C13, C16 to C14, C17 to C15, C19 to C16, C20 to C17, C21 to C18, C22 to C19, C23 to C20, C24 to C21, C25 to C22, C26 to C23, C27 to C24, C28 to C25, C29 to C26, C30 to C27, C31 to C28, C32 to C29, C33 to C30, C34 to C31, C35 to C32, C36 to C33, C37 to C34, C38 to C35, C39 to C36, C40 to C37, C41 to C38, C42 to C39, C43 to C40, C44 to C41, C45 to C42, C46 to C43, C47 to C44, C48 to C45, C49 to C46, C50 to C47, C51 to C48, C52 to C49, C53 to C50, C54 to C51, C55 to C52, C56 to C53, C57 to C54, C58 to C55, C59 to C56, C60 to C57, C61 to C58, C62 to C59, C7 to C6, C63 to C60, C64 to C61, C65 to C62, C66 to C63, C67 to C64, C68 to C65, C69 to C66, C70 to C67, C71 to C68, C72 to C69, C8 to C7, C73 to C70, C74 to C71, C75 to C72, C76 to C73, C77 to C74, C78 to C75, C79 to C76, C80 to C77, C81 to C78, C82 to C79, C9 to C8, C83 to C80, C84 to C81, C85 to C82, C86 to C83, C87 to C84, C10 to C9
Connections:
- net /Keyboard Keys/KEY_COL0 renamed COL0
- net /Keyboard Keys/KEY_COL1 renamed COL1
- net /Keyboard Keys/KEY_COL10 renamed COL10
- net /Keyboard Keys/KEY_COL11 renamed COL11
- net /Keyboard Keys/KEY_COL12 renamed COL12
- net /Keyboard Keys/KEY_COL13 renamed COL13
- net /Keyboard Keys/KEY_COL2 renamed COL2
- net /Keyboard Keys/KEY_COL3 renamed COL3
- net /Keyboard Keys/KEY_COL4 renamed COL4
- net /Keyboard Keys/KEY_COL5 renamed COL5
- net /Keyboard Keys/KEY_COL6 renamed COL6
- net /Keyboard Keys/KEY_COL7 renamed COL7
- net /Keyboard Keys/KEY_COL8 renamed COL8
- net /Keyboard Keys/KEY_COL9 renamed COL9
- net /Keyboard Keys/KEY_ROW0 renamed ROW0
- net /Keyboard Keys/KEY_ROW1 renamed ROW1
- net /Keyboard Keys/KEY_ROW2 renamed ROW2
- net /Keyboard Keys/KEY_ROW3 renamed ROW3
- net /Keyboard Keys/KEY_ROW4 renamed ROW4
- net /Keyboard Keys/KEY_ROW5 renamed ROW5
- D100 pad 1: LED_5V -> Net-(D100-Pad1)
- D100 pad 2: Net-(D100-Pad2) -> LED_GND
- D100 pad 3: LED_GND -> Net-(D100-Pad3)
- D100 pad 4: Net-(D100-Pad4) -> LED_5V
- D101 pad 1: LED_5V -> Net-(D101-Pad1)
- D101 pad 2: Net-(D101-Pad2) -> LED_GND
- D101 pad 3: LED_GND -> Net-(D101-Pad3)
- D101 pad 4: Net-(D101-Pad4) -> LED_5V
- D102 pad 1: LED_5V -> Net-(D102-Pad1)
- D102 pad 2: Net-(D102-Pad2) -> LED_GND
- D102 pad 3: LED_GND -> Net-(D102-Pad3)
- D102 pad 4: Net-(D102-Pad4) -> LED_5V
- D103 pad 1: LED_5V -> Net-(D103-Pad1)
- D103 pad 2: Net-(D103-Pad2) -> LED_GND
- D103 pad 3: LED_GND -> Net-(D103-Pad3)
- D103 pad 4: Net-(D103-Pad4) -> LED_5V
- D104 pad 1: LED_5V -> Net-(D104-Pad1)
- D104 pad 2: Net-(D104-Pad2) -> LED_GND
- D104 pad 3: LED_GND -> Net-(D100-Pad1)
- D104 pad 4: Net-(D100-Pad2) -> LED_5V
- D105 pad 1: LED_5V -> Net-(D105-Pad1)
- D105 pad 2: Net-(D105-Pad2) -> LED_GND
- D105 pad 3: LED_GND -> Net-(D101-Pad1)
- D105 pad 4: Net-(D101-Pad2) -> LED_5V
- D106 pad 1: LED_5V -> Net-(D106-Pad1)
- D106 pad 2: Net-(D106-Pad2) -> LED_GND
- D106 pad 3: LED_GND -> Net-(D102-Pad1)
- D106 pad 4: Net-(D102-Pad2) -> LED_5V
- D107 pad 1: LED_5V -> Net-(D107-Pad1)
- D107 pad 2: Net-(D107-Pad2) -> LED_GND
- D107 pad 3: LED_GND -> Net-(D103-Pad1)
- D107 pad 4: Net-(D103-Pad2) -> LED_5V
- D108 pad 1: LED_5V -> Net-(D108-Pad1)
- D108 pad 2: Net-(D108-Pad2) -> LED_GND
- D108 pad 3: LED_GND -> Net-(D104-Pad1)
- D108 pad 4: Net-(D104-Pad2) -> LED_5V
- D109 pad 1: LED_5V -> Net-(D109-Pad1)
- D109 pad 2: Net-(D109-Pad2) -> LED_GND
- D109 pad 3: LED_GND -> Net-(D105-Pad1)
- D109 pad 4: Net-(D105-Pad2) -> LED_5V
- D110 pad 1: LED_5V -> Net-(D110-Pad1)
- D110 pad 2: Net-(D110-Pad2) -> LED_GND
- D110 pad 3: LED_GND -> Net-(D106-Pad1)
- D110 pad 4: Net-(D106-Pad2) -> LED_5V
- D111 pad 1: LED_5V -> Net-(D111-Pad1)
- D111 pad 2: Net-(D111-Pad2) -> LED_GND
- D111 pad 3: LED_GND -> Net-(D107-Pad1)
- D111 pad 4: Net-(D107-Pad2) -> LED_5V
- D112 pad 1: LED_5V -> Net-(D112-Pad1)
- D112 pad 2: Net-(D112-Pad2) -> LED_GND
- D112 pad 3: LED_GND -> Net-(D108-Pad1)
- D112 pad 4: Net-(D108-Pad2) -> LED_5V
- D113 pad 1: LED_5V -> Net-(D113-Pad1)
- D113 pad 2: Net-(D113-Pad2) -> LED_GND
- D113 pad 3: LED_GND -> Net-(D109-Pad1)
- D113 pad 4: Net-(D109-Pad2) -> LED_5V
- D114 pad 1: LED_5V -> Net-(D114-Pad1)
- D114 pad 2: Net-(D114-Pad2) -> LED_GND
- D114 pad 3: LED_GND -> Net-(D110-Pad1)
- D114 pad 4: Net-(D110-Pad2) -> LED_5V
- D115 pad 1: LED_5V -> Net-(D115-Pad1)
- D115 pad 2: Net-(D115-Pad2) -> LED_GND
- D115 pad 3: LED_GND -> Net-(D111-Pad1)
- D115 pad 4: Net-(D111-Pad2) -> LED_5V
- D116 pad 1: LED_5V -> Net-(D116-Pad1)
- D116 pad 2: Net-(D116-Pad2) -> LED_GND
- D116 pad 3: LED_GND -> Net-(D112-Pad1)
- D116 pad 4: Net-(D112-Pad2) -> LED_5V
- D117 pad 1: LED_5V -> Net-(D117-Pad1)
- D117 pad 2: Net-(D117-Pad2) -> LED_GND
- D117 pad 3: LED_GND -> Net-(D113-Pad1)
- D117 pad 4: Net-(D113-Pad2) -> LED_5V
- D118 pad 1: LED_5V -> Net-(D118-Pad1)
- D118 pad 2: Net-(D118-Pad2) -> LED_GND
- D118 pad 3: LED_GND -> Net-(D114-Pad1)
- D118 pad 4: Net-(D114-Pad2) -> LED_5V
- D119 pad 1: LED_5V -> Net-(D119-Pad1)
- D119 pad 2: Net-(D119-Pad2) -> LED_GND
- D119 pad 3: LED_GND -> Net-(D115-Pad1)
- D119 pad 4: Net-(D115-Pad2) -> LED_5V
- D120 pad 1: LED_5V -> Net-(D120-Pad1)
- D120 pad 2: Net-(D120-Pad2) -> LED_GND
- D120 pad 3: LED_GND -> Net-(D116-Pad1)
- D120 pad 4: Net-(D116-Pad2) -> LED_5V
- D121 pad 1: LED_5V -> Net-(D121-Pad1)
- D121 pad 2: Net-(D121-Pad2) -> LED_GND
- D121 pad 3: LED_GND -> Net-(D117-Pad1)
- D121 pad 4: Net-(D117-Pad2) -> LED_5V
- D122 pad 1: LED_5V -> Net-(D122-Pad1)
- D122 pad 2: Net-(D122-Pad2) -> LED_GND
- D122 pad 3: LED_GND -> Net-(D118-Pad1)
- D122 pad 4: Net-(D118-Pad2) -> LED_5V
- D123 pad 1: LED_5V -> Net-(D123-Pad1)
- D123 pad 2: Net-(D123-Pad2) -> LED_GND
- D123 pad 3: LED_GND -> Net-(D119-Pad1)
- D123 pad 4: Net-(D119-Pad2) -> LED_5V
- D124 pad 1: LED_5V -> Net-(D124-Pad1)
- D124 pad 2: Net-(D124-Pad2) -> LED_GND
- D124 pad 3: LED_GND -> Net-(D120-Pad1)
- D124 pad 4: Net-(D120-Pad2) -> LED_5V
- D125 pad 1: LED_5V -> Net-(D125-Pad1)
- D125 pad 2: Net-(D125-Pad2) -> LED_GND
- D125 pad 3: LED_GND -> Net-(D121-Pad1)
- D125 pad 4: Net-(D121-Pad2) -> LED_5V
- D126 pad 1: LED_5V -> Net-(D126-Pad1)
- D126 pad 2: Net-(D126-Pad2) -> LED_GND
- D126 pad 3: LED_GND -> Net-(D122-Pad1)
- D126 pad 4: Net-(D122-Pad2) -> LED_5V
- D127 pad 1: LED_5V -> Net-(D127-Pad1)
- D127 pad 2: Net-(D127-Pad2) -> LED_GND
- D127 pad 3: LED_GND -> Net-(D123-Pad1)
- D127 pad 4: Net-(D123-Pad2) -> LED_5V
- D128 pad 1: LED_5V -> Net-(D128-Pad1)
- D128 pad 2: Net-(D128-Pad2) -> LED_GND
- D128 pad 3: LED_GND -> Net-(D124-Pad1)
- D128 pad 4: Net-(D124-Pad2) -> LED_5V
- D129 pad 1: LED_5V -> Net-(D129-Pad1)
- D129 pad 2: Net-(D129-Pad2) -> LED_GND
- D129 pad 3: LED_GND -> Net-(D125-Pad1)
- D129 pad 4: Net-(D125-Pad2) -> LED_5V
- D130 pad 1: LED_5V -> Net-(D130-Pad1)
- D130 pad 2: Net-(D130-Pad2) -> LED_GND
- D130 pad 3: LED_GND -> Net-(D126-Pad1)
- D130 pad 4: Net-(D126-Pad2) -> LED_5V
- D131 pad 1: LED_5V -> Net-(D131-Pad1)
- D131 pad 2: Net-(D131-Pad2) -> LED_GND
- D131 pad 3: LED_GND -> Net-(D127-Pad1)
- D131 pad 4: Net-(D127-Pad2) -> LED_5V
- D132 pad 1: LED_5V -> Net-(D132-Pad1)
- D132 pad 2: Net-(D132-Pad2) -> LED_GND
- D132 pad 3: LED_GND -> Net-(D128-Pad1)
- D132 pad 4: Net-(D128-Pad2) -> LED_5V
- D133 pad 1: LED_5V -> Net-(D133-Pad1)
- D133 pad 2: Net-(D133-Pad2) -> LED_GND
- D133 pad 3: LED_GND -> Net-(D129-Pad1)
- D133 pad 4: Net-(D129-Pad2) -> LED_5V
- D134 pad 1: LED_5V -> Net-(D134-Pad1)
- D134 pad 2: Net-(D134-Pad2) -> LED_GND
- D134 pad 3: LED_GND -> Net-(D130-Pad1)
- D134 pad 4: Net-(D130-Pad2) -> LED_5V
- D135 pad 1: LED_5V -> Net-(D135-Pad1)
- D135 pad 2: Net-(D135-Pad2) -> LED_GND
- D135 pad 3: LED_GND -> Net-(D131-Pad1)
- D135 pad 4: Net-(D131-Pad2) -> LED_5V
- D136 pad 1: LED_5V -> Net-(D136-Pad1)
- D136 pad 2: Net-(D136-Pad2) -> LED_GND
- D136 pad 3: LED_GND -> Net-(D132-Pad1)
- D136 pad 4: Net-(D132-Pad2) -> LED_5V
- D137 pad 1: LED_5V -> Net-(D137-Pad1)
- D137 pad 2: Net-(D137-Pad2) -> LED_GND
- D137 pad 3: LED_GND -> Net-(D133-Pad1)
- D137 pad 4: Net-(D133-Pad2) -> LED_5V
- D138 pad 1: LED_5V -> Net-(D138-Pad1)
- D138 pad 2: Net-(D138-Pad2) -> LED_GND
- D138 pad 3: LED_GND -> Net-(D134-Pad1)
- D138 pad 4: Net-(D134-Pad2) -> LED_5V
- D139 pad 1: LED_5V -> Net-(D139-Pad1)
- D139 pad 2: Net-(D139-Pad2) -> LED_GND
- D139 pad 3: LED_GND -> Net-(D135-Pad1)
- D139 pad 4: Net-(D135-Pad2) -> LED_5V
- D140 pad 1: LED_5V -> Net-(D140-Pad1)
- D140 pad 2: Net-(D140-Pad2) -> LED_GND
- D140 pad 3: LED_GND -> Net-(D136-Pad1)
- D140 pad 4: Net-(D136-Pad2) -> LED_5V
- D141 pad 1: LED_5V -> Net-(D141-Pad1)
- D141 pad 2: Net-(D141-Pad2) -> LED_GND
- D141 pad 3: LED_GND -> Net-(D137-Pad1)
- D141 pad 4: Net-(D137-Pad2) -> LED_5V
- D142 pad 1: LED_5V -> Net-(D142-Pad1)
- D142 pad 2: Net-(D142-Pad2) -> LED_GND
- D142 pad 3: LED_GND -> Net-(D138-Pad1)
- D142 pad 4: Net-(D138-Pad2) -> LED_5V
- D143 pad 1: LED_5V -> Net-(D143-Pad1)
- D143 pad 2: Net-(D143-Pad2) -> LED_GND
- D143 pad 3: LED_GND -> Net-(D139-Pad1)
- D143 pad 4: Net-(D139-Pad2) -> LED_5V
- D144 pad 1: LED_5V -> Net-(D144-Pad1)
- D144 pad 2: Net-(D144-Pad2) -> LED_GND
- D144 pad 3: LED_GND -> Net-(D140-Pad1)
- D144 pad 4: Net-(D140-Pad2) -> LED_5V
- D145 pad 1: LED_5V -> Net-(D145-Pad1)
- D145 pad 2: Net-(D145-Pad2) -> LED_GND
- D145 pad 3: LED_GND -> Net-(D141-Pad1)
- D145 pad 4: Net-(D141-Pad2) -> LED_5V
- D146 pad 1: LED_5V -> Net-(D146-Pad1)
- D146 pad 2: Net-(D146-Pad2) -> LED_GND
- D146 pad 3: LED_GND -> Net-(D142-Pad1)
- D146 pad 4: Net-(D142-Pad2) -> LED_5V
- D147 pad 1: LED_5V -> Net-(D147-Pad1)
- D147 pad 2: Net-(D147-Pad2) -> LED_GND
- D147 pad 3: LED_GND -> Net-(D143-Pad1)
- D147 pad 4: Net-(D143-Pad2) -> LED_5V
- D148 pad 1: LED_5V -> Net-(D148-Pad1)
- D148 pad 2: Net-(D148-Pad2) -> LED_GND
- D148 pad 3: LED_GND -> Net-(D144-Pad1)
- D148 pad 4: Net-(D144-Pad2) -> LED_5V
- D149 pad 1: LED_5V -> Net-(D149-Pad1)
- D149 pad 2: Net-(D149-Pad2) -> LED_GND
- D149 pad 3: LED_GND -> Net-(D145-Pad1)
- D149 pad 4: Net-(D145-Pad2) -> LED_5V
- D150 pad 1: LED_5V -> Net-(D150-Pad1)
- D150 pad 2: Net-(D150-Pad2) -> LED_GND
- D150 pad 3: LED_GND -> Net-(D146-Pad1)
- D150 pad 4: Net-(D146-Pad2) -> LED_5V
- D151 pad 1: LED_5V -> Net-(D151-Pad1)
- D151 pad 2: Net-(D151-Pad2) -> LED_GND
- D151 pad 3: LED_GND -> Net-(D147-Pad1)
- D151 pad 4: Net-(D147-Pad2) -> LED_5V
- D152 pad 1: LED_5V -> Net-(D152-Pad1)
- D152 pad 2: Net-(D152-Pad2) -> LED_GND
- D152 pad 3: LED_GND -> Net-(D148-Pad1)
- D152 pad 4: Net-(D148-Pad2) -> LED_5V
- D153 pad 1: LED_5V -> Net-(D153-Pad1)
- D153 pad 2: Net-(D153-Pad2) -> LED_GND
- D153 pad 3: LED_GND -> Net-(D149-Pad1)
- D153 pad 4: Net-(D149-Pad2) -> LED_5V
- D154 pad 1: LED_5V -> Net-(D154-Pad1)
- D154 pad 2: Net-(D154-Pad2) -> LED_GND
- D154 pad 3: LED_GND -> Net-(D150-Pad1)
- D154 pad 4: Net-(D150-Pad2) -> LED_5V
- D155 pad 1: LED_5V -> Net-(D155-Pad1)
- D155 pad 2: Net-(D155-Pad2) -> LED_GND
- D155 pad 3: LED_GND -> Net-(D151-Pad1)
- D155 pad 4: Net-(D151-Pad2) -> LED_5V
- D156 pad 1: LED_5V -> Net-(D156-Pad1)
- D156 pad 2: Net-(D156-Pad2) -> LED_GND
- D156 pad 3: LED_GND -> Net-(D152-Pad1)
- D156 pad 4: Net-(D152-Pad2) -> LED_5V
- D157 pad 1: LED_5V -> Net-(D157-Pad1)
- D157 pad 2: Net-(D157-Pad2) -> LED_GND
- D157 pad 3: LED_GND -> Net-(D153-Pad1)
- D157 pad 4: Net-(D153-Pad2) -> LED_5V
- D158 pad 1: LED_5V -> Net-(D158-Pad1)
- D158 pad 2: Net-(D158-Pad2) -> LED_GND
- D158 pad 3: LED_GND -> Net-(D154-Pad1)
- D158 pad 4: Net-(D154-Pad2) -> LED_5V
- D159 pad 1: LED_5V -> Net-(D159-Pad1)
- D159 pad 2: Net-(D159-Pad2) -> LED_GND
- D159 pad 3: LED_GND -> Net-(D155-Pad1)
- D159 pad 4: Net-(D155-Pad2) -> LED_5V
- D160 pad 1: LED_5V -> Net-(D160-Pad1)
- D160 pad 2: Net-(D160-Pad2) -> LED_GND
- D160 pad 3: LED_GND -> Net-(D156-Pad1)
- D160 pad 4: Net-(D156-Pad2) -> LED_5V
- D161 pad 1: LED_5V -> Net-(D161-Pad1)
- D161 pad 2: Net-(D161-Pad2) -> LED_GND
- D161 pad 3: LED_GND -> Net-(D157-Pad1)
- D161 pad 4: Net-(D157-Pad2) -> LED_5V
- D162 pad 1: LED_5V -> Net-(D162-Pad1)
- D162 pad 2: Net-(D162-Pad2) -> LED_GND
- D162 pad 3: LED_GND -> Net-(D158-Pad1)
- D162 pad 4: Net-(D158-Pad2) -> LED_5V
- D163 pad 1: LED_5V -> Net-(D163-Pad1)
- D163 pad 2: Net-(D163-Pad2) -> LED_GND
- D163 pad 3: LED_GND -> Net-(D159-Pad1)
- D163 pad 4: Net-(D159-Pad2) -> LED_5V
- D164 pad 1: LED_5V -> Net-(D164-Pad1)
- D164 pad 2: Net-(D164-Pad2) -> LED_GND
- D164 pad 3: LED_GND -> Net-(D160-Pad1)
- D164 pad 4: Net-(D160-Pad2) -> LED_5V
- D165 pad 1: LED_5V -> Net-(D165-Pad1)
- D165 pad 2: Net-(D165-Pad2) -> LED_GND
- D165 pad 3: LED_GND -> Net-(D161-Pad1)
- D165 pad 4: Net-(D161-Pad2) -> LED_5V
- D166 pad 1: LED_5V -> Net-(D166-Pad1)
- D166 pad 2: Net-(D166-Pad2) -> LED_GND
- D166 pad 3: LED_GND -> Net-(D162-Pad1)
- D166 pad 4: Net-(D162-Pad2) -> LED_5V
- D167 pad 1: LED_5V -> Net-(D167-Pad1)
- D167 pad 2: Net-(D167-Pad2) -> LED_GND
- D167 pad 3: LED_GND -> Net-(D163-Pad1)
- D167 pad 4: Net-(D163-Pad2) -> LED_5V
- D168 pad 1: LED_5V -> Net-(D168-Pad1)
- D168 pad 2: Net-(D168-Pad2) -> LED_GND
- D168 pad 3: LED_GND -> Net-(D164-Pad1)
- D168 pad 4: Net-(D164-Pad2) -> LED_5V
- D85 pad 1: LED_5V -> Net-(D85-Pad1)
- D85 pad 2: Net-(D85-Pad2) -> LED_GND
- D85 pad 3: LED_GND -> /RGB/INPUT
- D85 pad 4: /Sheet6096EA01/INPUT -> LED_5V
- D86 pad 1: LED_5V -> Net-(D86-Pad1)
- D86 pad 2: Net-(D86-Pad2) -> LED_GND
- D86 pad 3: LED_GND -> Net-(D168-Pad1)
- D86 pad 4: Net-(D168-Pad2) -> LED_5V
- D87 pad 1: LED_5V -> Net-(D87-Pad1)
- D87 pad 2: Net-(D87-Pad2) -> LED_GND
- D87 pad 3: LED_GND -> Net-(D165-Pad1)
- D87 pad 4: Net-(D165-Pad2) -> LED_5V
- D88 pad 1: LED_5V -> Net-(D88-Pad1)
- D88 pad 2: Net-(D88-Pad2) -> LED_GND
- D88 pad 3: LED_GND -> Net-(D166-Pad1)
- D88 pad 4: Net-(D166-Pad2) -> LED_5V
- D89 pad 1: LED_5V -> Net-(D89-Pad1)
- D89 pad 2: Net-(D89-Pad2) -> LED_GND
- D89 pad 3: LED_GND -> Net-(D167-Pad1)
- D89 pad 4: Net-(D167-Pad2) -> LED_5V
- D90 pad 1: LED_5V -> Net-(D90-Pad1)
- D90 pad 2: Net-(D90-Pad2) -> LED_GND
- D90 pad 3: LED_GND -> Net-(D85-Pad1)
- D90 pad 4: Net-(D85-Pad2) -> LED_5V
- D91 pad 1: LED_5V -> Net-(D91-Pad1)
- D91 pad 2: Net-(D91-Pad2) -> LED_GND
- D91 pad 3: LED_GND -> Net-(D86-Pad1)
- D91 pad 4: Net-(D86-Pad2) -> LED_5V
- D92 pad 1: LED_5V -> Net-(D92-Pad1)
- D92 pad 2: Net-(D92-Pad2) -> LED_GND
- D92 pad 3: LED_GND -> Net-(D87-Pad1)
- D92 pad 4: Net-(D87-Pad2) -> LED_5V
- D93 pad 1: LED_5V -> Net-(D93-Pad1)
- D93 pad 2: Net-(D93-Pad2) -> LED_GND
- D93 pad 3: LED_GND -> Net-(D88-Pad1)
- D93 pad 4: Net-(D88-Pad2) -> LED_5V
- D94 pad 1: LED_5V -> Net-(D94-Pad1)
- D94 pad 2: Net-(D94-Pad2) -> LED_GND
- D94 pad 3: LED_GND -> Net-(D89-Pad1)
- D94 pad 4: Net-(D89-Pad2) -> LED_5V
- D95 pad 1: LED_5V -> Net-(D100-Pad3)
- D95 pad 2: Net-(D100-Pad4) -> LED_GND
- D95 pad 3: LED_GND -> Net-(D90-Pad1)
- D95 pad 4: Net-(D90-Pad2) -> LED_5V
- D96 pad 1: LED_5V -> Net-(D101-Pad3)
- D96 pad 2: Net-(D101-Pad4) -> LED_GND
- D96 pad 3: LED_GND -> Net-(D91-Pad1)
- D96 pad 4: Net-(D91-Pad2) -> LED_5V
- D97 pad 1: LED_5V -> Net-(D102-Pad3)
- D97 pad 2: Net-(D102-Pad4) -> LED_GND
- D97 pad 3: LED_GND -> Net-(D92-Pad1)
- D97 pad 4: Net-(D92-Pad2) -> LED_5V
- D98 pad 1: LED_5V -> Net-(D103-Pad3)
- D98 pad 2: Net-(D103-Pad4) -> LED_GND
- D98 pad 3: LED_GND -> Net-(D93-Pad1)
- D98 pad 4: Net-(D93-Pad2) -> LED_5V
- D99 pad 1: LED_5V -> (no net)
- D99 pad 2: (no net) -> LED_GND
- D99 pad 3: LED_GND -> Net-(D94-Pad1)
- D99 pad 4: Net-(D94-Pad2) -> LED_5V
- J1 pad 13: PWR_5V -> (no net)
- J1 pad 3: Net-(J1-Pad3) -> (no net)
- J1 pad 4: /Sheet6096EA01/INPUT -> /RGB/INPUT
- J1 pad 5: Net-(J1-Pad5) -> (no net)
- J1 pad 7: Net-(J1-Pad7) -> (no net)
Routing:
- net LED_5V: track 2287.3 -> 0.00 mm, vias 9 -> 0
- net LED_GND: track 2187.8 -> 0.00 mm, vias 14 -> 0
- net ROW4: track 613.1 -> 0.00 mm, vias 9 -> 0
- net ROW3: track 548.7 -> 0.00 mm, vias 10 -> 0
- net ROW0: track 546.0 -> 0.00 mm, vias 5 -> 0
- net ROW2: track 483.3 -> 0.00 mm, vias 11 -> 0
- net COL0: track 458.7 -> 0.00 mm, vias 12 -> 0
- net ROW1: track 454.9 -> 0.00 mm, vias 9 -> 0
- net COL1: track 444.1 -> 0.00 mm, vias 10 -> 0
- net COL13: track 414.4 -> 0.00 mm, vias 13 -> 0
- net COL6: track 413.9 -> 0.00 mm, vias 12 -> 0
- net COL4: track 402.0 -> 0.00 mm, vias 9 -> 0
- net ROW5: track 394.2 -> 0.00 mm, vias 6 -> 0
- net COL3: track 387.9 -> 0.00 mm, vias 10 -> 0
- net COL2: track 386.7 -> 0.00 mm, vias 4 -> 0
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
Commit message: updates to be nearly functional
Parts:
- added C85: 0.1u, Capacitor_SMD:C_0805_2012Metric, B.Cu at (309.2, 51.4)
- added C86: 0.1u, Capacitor_SMD:C_0805_2012Metric, B.Cu at (309.2, 48.4)
- added C87: 0.1u, Capacitor_SMD:C_0805_2012Metric, B.Cu at (313.7, 51.4)
- added C88: 0.1u, Capacitor_SMD:C_0805_2012Metric, B.Cu at (309.2, 45.4)
- added C89: 0.1u, Capacitor_SMD:C_0805_2012Metric, B.Cu at (313.7, 48.4)
- added C90: 22p, Capacitor_SMD:C_0805_2012Metric, B.Cu at (321.9, 45.7)
- added C91: 22p, Capacitor_SMD:C_0805_2012Metric, B.Cu at (318.1, 51.4)
- added C92: 1u, Capacitor_SMD:C_0805_2012Metric, B.Cu at (313.7, 45.4)
- added R1: 10k, Resistor_SMD:R_1206_3216Metric, B.Cu at (323.2, 42.5)
- added R2: 22R, Resistor_SMD:R_0805_2012Metric, B.Cu at (318.1, 48.5)
- added R3: 22R, Resistor_SMD:R_0805_2012Metric, B.Cu at (318.1, 45.5)
- added R4: R10K, Resistor_SMD:R_1206_3216Metric, B.Cu at (319.4, 54.0)
- added Y1: Crystal, Crystal:Crystal_SMD_5032-2Pin_5.0x3.2mm_HandSoldering, B.Cu at (323.9, 52.0)
- U1: renamed from U2; moved to B.Cu
- moved U1 97.4 mm to (316.2, 36.2)
Connections:
- J1 pad 3: (no net) -> LED_DATA
- U1 pad 1: (no net) -> LED_DATA
- U1 pad 13: (no net) -> Net-(R1-Pad2)
- U1 pad 16: (no net) -> Net-(C91-Pad1)
- U1 pad 17: (no net) -> Net-(C90-Pad1)
- U1 pad 3: (no net) -> Net-(R3-Pad1)
- U1 pad 33: (no net) -> Net-(R4-Pad2)
- U1 pad 4: (no net) -> Net-(R2-Pad1)
- U1 pad 6: (no net) -> Net-(C92-Pad2)

Commit message: moving parts around, trying to align to a standard keyboard keycap sizes
Parts:
- removed SW59: 111, daprice-keyswitches:Kailh_socket_MX
- added Slash1: 111, daprice-keyswitches:Stabilizer_MX_1.5u, F.Cu at (302.3, -57.5)
- Backspace1: footprint daprice-keyswitches:Stabilizer_MX_1.25u -> daprice-keyswitches:Stabilizer_MX_2u
- CAPS1: footprint daprice-keyswitches:Stabilizer_MX_1.5u -> daprice-keyswitches:Stabilizer_MX_1.75u
- ENTER1: footprint daprice-keyswitches:Stabilizer_MX_1.75u -> daprice-keyswitches:Stabilizer_MX_2.25u
- LEFT-SHIFT1: footprint daprice-keyswitches:Stabilizer_MX_2u -> daprice-keyswitches:Stabilizer_MX_2.25u
- LEFT_ALT1: renamed from SW19; footprint daprice-keyswitches:Kailh_socket_MX -> daprice-keyswitches:Stabilizer_MX_1.25u
- LEFT_CTRL1: renamed from SW2; footprint daprice-keyswitches:Kailh_socket_MX -> daprice-keyswitches:Stabilizer_MX_1.25u
- LEFT_FN1: renamed from SW8; footprint daprice-keyswitches:Kailh_socket_MX -> daprice-keyswitches:Stabilizer_MX_1.25u
- TAB1: footprint daprice-keyswitches:Stabilizer_MX_1.25u -> daprice-keyswitches:Stabilizer_MX_1.5u
- WinKey1: footprint daprice-keyswitches:Stabilizer_MX_1.5u -> daprice-keyswitches:Stabilizer_MX_1.25u
- moved D17 120.3 mm to (85.1, 167.4)
- moved D19 120.3 mm to (104.3, 167.4)
- moved D29 120.3 mm to (123.5, 167.4)
- moved D31 120.3 mm to (142.7, 167.4)
- moved D41 120.3 mm to (161.9, 167.4)
- moved D43 120.3 mm to (181.1, 167.4)
- moved D48 120.3 mm to (258.0, 167.4)
- moved D5 120.3 mm to (46.7, 167.4)
- moved D53 120.3 mm to (200.3, 167.4)
- moved D55 120.3 mm to (219.6, 167.4)
- moved D61 120.3 mm to (238.8, 167.4)
- moved D7 120.3 mm to (65.9, 167.4)
- moved SW4 114.3 mm to (40.2, -76.6)
- moved SW13 114.3 mm to (78.4, -76.6)
- moved SW15 114.3 mm to (97.4, -76.6)
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Other:
- board text added: "LOG0.Key.Yeet3"
- board text removed: "LOG0.Key.Yeet2 May 14, 2021"
