File: chgray-keyboard.kicad_pcb (KiCad board)
At the start: 2 copper layers, 377.4 x 105.5 mm, 351 parts, among them J1 Conn_01x01_Female, SW1 30, SW10 22, SW11 32, SW12 52, SW13 02, SW14 12, SW15 03, SW16 13, SW17 23, SW18 33, SW20 53, SW21 24, SW22 34, SW23 54, SW24 04, SW25 14, SW26 05, SW27 15, SW28 25, SW29 35, SW3 50, SW30 45, SW31 26, SW32 36, SW33 46, SW34 56, SW35 06, SW36 16, SW37 07, SW38 17, SW39 27, SW4 00, SW40 37, SW41 57, SW42 28, SW43 38, SW44 48, SW45 58, SW46 08, SW47 18, SW48 09, SW49 19, SW5 01, SW50 29, SW51 39, SW52 49, SW53 010, SW54 110, SW55 210, SW56 310, SW57 410, SW58 510, SW6 11, SW60 211, SW61 311, SW62 411, SW63 511, SW64 111, SW65 211, SW66 311, SW67 411, SW68 511, SW69 111, SW7 21, SW70 211, SW71 311, SW72 411, SW73 511, SW9 51, U1 ATmega32U4-AU, Y1 Crystal

Commit message: led work
Parts:
- D100, D101, D102, D103, D104, D105, D106, D107, D108, D109, D110, D111, D112, D113, D114, D115, D116, D117, D118, D119, D120, D121, D122, D123, D124, D125, D126, D127, D128, D129, D130, D131, D132, D133, D134, D135, D136, D137, D138, D139, D140, D141, D142, D143, D144, D145, D146, D147, D148, D149, D150, D151, D152, D153, D154, D155, D156, D157, D158, D159, D160, D161, D162, D163, D164, D165, D166, D167, D168, D85, D86, D87, D88, D89, D90, D91, D92, D93, D94, D95, D96, D97, D98, D99: footprint daprice-keyswitches:LED_SK6812MINI_PLCC4_3.5x3.5mm_P1.75mm -> CHGRAY_LED:LED_WS2812-2020
- moved D145 118.5 mm to (25.7, -35.9)
- moved D141 117.3 mm to (25.2, -53.8)
- moved D136 113.5 mm to (268.9, -71.1)
- moved D120 113.5 mm to (192.6, -71.1)
- moved D100 113.4 mm to (97.4, -71.0)
- moved D116 113.4 mm to (173.6, -71.1)
- moved D90 113.4 mm to (59.4, -71.1)
- moved D85 113.4 mm to (40.2, -71.0)
- moved D112 113.4 mm to (154.5, -71.0)
- moved D104 113.4 mm to (116.5, -71.0)
- moved D124 113.4 mm to (211.7, -71.0)
- moved D132 113.4 mm to (249.8, -71.0)
- moved D95 113.4 mm to (78.4, -71.0)
- moved D128 113.4 mm to (230.7, -71.0)
- moved D108 113.4 mm to (135.5, -71.0)
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Connections:
- D100 pad 1: Net-(D100-Pad1) -> LED_5V
- D100 pad 2: LED_GND -> Net-(D100-Pad2)
- D100 pad 3: Net-(D100-Pad3) -> LED_GND
- D100 pad 4: LED_5V -> Net-(D100-Pad4)
- D101 pad 1: Net-(D101-Pad1) -> LED_5V
- D101 pad 2: LED_GND -> Net-(D101-Pad2)
- D101 pad 3: Net-(D101-Pad3) -> LED_GND
- D101 pad 4: LED_5V -> Net-(D101-Pad4)
- D102 pad 1: Net-(D102-Pad1) -> LED_5V
- D102 pad 2: LED_GND -> Net-(D102-Pad2)
- D102 pad 3: Net-(D102-Pad3) -> LED_GND
- D102 pad 4: LED_5V -> Net-(D102-Pad4)
- D103 pad 1: Net-(D103-Pad1) -> LED_5V
- D103 pad 2: LED_GND -> Net-(D103-Pad2)
- D103 pad 3: Net-(D103-Pad3) -> LED_GND
- D103 pad 4: LED_5V -> Net-(D103-Pad4)
- D104 pad 1: Net-(D104-Pad1) -> LED_5V
- D104 pad 2: LED_GND -> Net-(D104-Pad2)
- D104 pad 3: Net-(D100-Pad1) -> LED_GND
- D104 pad 4: LED_5V -> Net-(D100-Pad2)
- D105 pad 1: Net-(D105-Pad1) -> LED_5V
- D105 pad 2: LED_GND -> Net-(D105-Pad2)
- D105 pad 3: Net-(D101-Pad1) -> LED_GND
- D105 pad 4: LED_5V -> Net-(D101-Pad2)
- D106 pad 1: Net-(D106-Pad1) -> LED_5V
- D106 pad 2: LED_GND -> Net-(D106-Pad2)
- D106 pad 3: Net-(D102-Pad1) -> LED_GND
- D106 pad 4: LED_5V -> Net-(D102-Pad2)
- D107 pad 1: Net-(D107-Pad1) -> LED_5V
- D107 pad 2: LED_GND -> Net-(D107-Pad2)
- D107 pad 3: Net-(D103-Pad1) -> LED_GND
- D107 pad 4: LED_5V -> Net-(D103-Pad2)
- D108 pad 1: Net-(D108-Pad1) -> LED_5V
- D108 pad 2: LED_GND -> Net-(D108-Pad2)
- D108 pad 3: Net-(D104-Pad1) -> LED_GND
- D108 pad 4: LED_5V -> Net-(D104-Pad2)
- D109 pad 1: Net-(D109-Pad1) -> LED_5V
- D109 pad 2: LED_GND -> Net-(D109-Pad2)
- D109 pad 3: Net-(D105-Pad1) -> LED_GND
- D109 pad 4: LED_5V -> Net-(D105-Pad2)
- D110 pad 1: Net-(D110-Pad1) -> LED_5V
- D110 pad 2: LED_GND -> Net-(D110-Pad2)
- D110 pad 3: Net-(D106-Pad1) -> LED_GND
- D110 pad 4: LED_5V -> Net-(D106-Pad2)
- D111 pad 1: Net-(D111-Pad1) -> LED_5V
- D111 pad 2: LED_GND -> Net-(D111-Pad2)
- D111 pad 3: Net-(D107-Pad1) -> LED_GND
- D111 pad 4: LED_5V -> Net-(D107-Pad2)
- D112 pad 1: Net-(D112-Pad1) -> LED_5V
- D112 pad 2: LED_GND -> Net-(D112-Pad2)
- D112 pad 3: Net-(D108-Pad1) -> LED_GND
- D112 pad 4: LED_5V -> Net-(D108-Pad2)
- D113 pad 1: Net-(D113-Pad1) -> LED_5V
- D113 pad 2: LED_GND -> Net-(D113-Pad2)
- D113 pad 3: Net-(D109-Pad1) -> LED_GND
- D113 pad 4: LED_5V -> Net-(D109-Pad2)
- D114 pad 1: Net-(D114-Pad1) -> LED_5V
- D114 pad 2: LED_GND -> Net-(D114-Pad2)
- D114 pad 3: Net-(D110-Pad1) -> LED_GND
- D114 pad 4: LED_5V -> Net-(D110-Pad2)
- D115 pad 1: Net-(D115-Pad1) -> LED_5V
- D115 pad 2: LED_GND -> Net-(D115-Pad2)
- D115 pad 3: Net-(D111-Pad1) -> LED_GND
- D115 pad 4: LED_5V -> Net-(D111-Pad2)
- D116 pad 1: Net-(D116-Pad1) -> LED_5V
- D116 pad 2: LED_GND -> Net-(D116-Pad2)
- D116 pad 3: Net-(D112-Pad1) -> LED_GND
- D116 pad 4: LED_5V -> Net-(D112-Pad2)
- D117 pad 1: Net-(D117-Pad1) -> LED_5V
- D117 pad 2: LED_GND -> Net-(D117-Pad2)
- D117 pad 3: Net-(D113-Pad1) -> LED_GND
- D117 pad 4: LED_5V -> Net-(D113-Pad2)
- D118 pad 1: Net-(D118-Pad1) -> LED_5V
- D118 pad 2: LED_GND -> Net-(D118-Pad2)
- D118 pad 3: Net-(D114-Pad1) -> LED_GND
- D118 pad 4: LED_5V -> Net-(D114-Pad2)
- D119 pad 1: Net-(D119-Pad1) -> LED_5V
- D119 pad 2: LED_GND -> Net-(D119-Pad2)
- D119 pad 3: Net-(D115-Pad1) -> LED_GND
- D119 pad 4: LED_5V -> Net-(D115-Pad2)
- D120 pad 1: Net-(D120-Pad1) -> LED_5V
- D120 pad 2: LED_GND -> Net-(D120-Pad2)
- D120 pad 3: Net-(D116-Pad1) -> LED_GND
- D120 pad 4: LED_5V -> Net-(D116-Pad2)
- D121 pad 1: Net-(D121-Pad1) -> LED_5V
- D121 pad 2: LED_GND -> Net-(D121-Pad2)
- D121 pad 3: Net-(D117-Pad1) -> LED_GND
- D121 pad 4: LED_5V -> Net-(D117-Pad2)
- D122 pad 1: Net-(D122-Pad1) -> LED_5V
- D122 pad 2: LED_GND -> Net-(D122-Pad2)
- D122 pad 3: Net-(D118-Pad1) -> LED_GND
- D122 pad 4: LED_5V -> Net-(D118-Pad2)
- D123 pad 1: Net-(D123-Pad1) -> LED_5V
- D123 pad 2: LED_GND -> Net-(D123-Pad2)
- D123 pad 3: Net-(D119-Pad1) -> LED_GND
- D123 pad 4: LED_5V -> Net-(D119-Pad2)
- D124 pad 1: Net-(D124-Pad1) -> LED_5V
- D124 pad 2: LED_GND -> Net-(D124-Pad2)
- D124 pad 3: Net-(D120-Pad1) -> LED_GND
- D124 pad 4: LED_5V -> Net-(D120-Pad2)
- D125 pad 1: Net-(D125-Pad1) -> LED_5V
- D125 pad 2: LED_GND -> Net-(D125-Pad2)
- D125 pad 3: Net-(D121-Pad1) -> LED_GND
- D125 pad 4: LED_5V -> Net-(D121-Pad2)
- D126 pad 1: Net-(D126-Pad1) -> LED_5V
- D126 pad 2: LED_GND -> Net-(D126-Pad2)
- D126 pad 3: Net-(D122-Pad1) -> LED_GND
- D126 pad 4: LED_5V -> Net-(D122-Pad2)
- D127 pad 1: Net-(D127-Pad1) -> LED_5V
- D127 pad 2: LED_GND -> Net-(D127-Pad2)
- D127 pad 3: Net-(D123-Pad1) -> LED_GND
- D127 pad 4: LED_5V -> Net-(D123-Pad2)
- D128 pad 1: Net-(D128-Pad1) -> LED_5V
- D128 pad 2: LED_GND -> Net-(D128-Pad2)
- D128 pad 3: Net-(D124-Pad1) -> LED_GND
- D128 pad 4: LED_5V -> Net-(D124-Pad2)
- D129 pad 1: Net-(D129-Pad1) -> LED_5V
- D129 pad 2: LED_GND -> Net-(D129-Pad2)
- D129 pad 3: Net-(D125-Pad1) -> LED_GND
- D129 pad 4: LED_5V -> Net-(D125-Pad2)
- D130 pad 1: Net-(D130-Pad1) -> LED_5V
- D130 pad 2: LED_GND -> Net-(D130-Pad2)
- D130 pad 3: Net-(D126-Pad1) -> LED_GND
- D130 pad 4: LED_5V -> Net-(D126-Pad2)
- D131 pad 1: Net-(D131-Pad1) -> LED_5V
- D131 pad 2: LED_GND -> Net-(D131-Pad2)
- D131 pad 3: Net-(D127-Pad1) -> LED_GND
- D131 pad 4: LED_5V -> Net-(D127-Pad2)
- D132 pad 1: Net-(D132-Pad1) -> LED_5V
- D132 pad 2: LED_GND -> Net-(D132-Pad2)
- D132 pad 3: Net-(D128-Pad1) -> LED_GND
- D132 pad 4: LED_5V -> Net-(D128-Pad2)
- D133 pad 1: Net-(D133-Pad1) -> LED_5V
- D133 pad 2: LED_GND -> Net-(D133-Pad2)
- D133 pad 3: Net-(D129-Pad1) -> LED_GND
- D133 pad 4: LED_5V -> Net-(D129-Pad2)
- D134 pad 1: Net-(D134-Pad1) -> LED_5V
- D134 pad 2: LED_GND -> Net-(D134-Pad2)
- D134 pad 3: Net-(D130-Pad1) -> LED_GND
- D134 pad 4: LED_5V -> Net-(D130-Pad2)
- D135 pad 1: Net-(D135-Pad1) -> LED_5V
- D135 pad 2: LED_GND -> Net-(D135-Pad2)
- D135 pad 3: Net-(D131-Pad1) -> LED_GND
- D135 pad 4: LED_5V -> Net-(D131-Pad2)
- D136 pad 1: Net-(D136-Pad1) -> LED_5V
- D136 pad 2: LED_GND -> Net-(D136-Pad2)
- D136 pad 3: Net-(D132-Pad1) -> LED_GND
- D136 pad 4: LED_5V -> Net-(D132-Pad2)
- D137 pad 1: Net-(D137-Pad1) -> LED_5V
- D137 pad 2: LED_GND -> Net-(D137-Pad2)
- D137 pad 3: Net-(D133-Pad1) -> LED_GND
- D137 pad 4: LED_5V -> Net-(D133-Pad2)
- D138 pad 1: Net-(D138-Pad1) -> LED_5V
- D138 pad 2: LED_GND -> Net-(D138-Pad2)
- D138 pad 3: Net-(D134-Pad1) -> LED_GND
- D138 pad 4: LED_5V -> Net-(D134-Pad2)
- D139 pad 1: Net-(D139-Pad1) -> LED_5V
- D139 pad 2: LED_GND -> Net-(D139-Pad2)
- D139 pad 3: Net-(D135-Pad1) -> LED_GND
- D139 pad 4: LED_5V -> Net-(D135-Pad2)
- D140 pad 1: Net-(D140-Pad1) -> LED_5V
- D140 pad 2: LED_GND -> Net-(D140-Pad2)
- D140 pad 3: Net-(D136-Pad1) -> LED_GND
- D140 pad 4: LED_5V -> Net-(D136-Pad2)
- D141 pad 1: Net-(D141-Pad1) -> LED_5V
- D141 pad 2: LED_GND -> Net-(D141-Pad2)
- D141 pad 3: Net-(D137-Pad1) -> LED_GND
- D141 pad 4: LED_5V -> Net-(D137-Pad2)
- D142 pad 1: Net-(D142-Pad1) -> LED_5V
- D142 pad 2: LED_GND -> Net-(D142-Pad2)
- D142 pad 3: Net-(D138-Pad1) -> LED_GND
- D142 pad 4: LED_5V -> Net-(D138-Pad2)
- D143 pad 1: Net-(D143-Pad1) -> LED_5V
- D143 pad 2: LED_GND -> Net-(D143-Pad2)
- D143 pad 3: Net-(D139-Pad1) -> LED_GND
- D143 pad 4: LED_5V -> Net-(D139-Pad2)
- D144 pad 1: Net-(D144-Pad1) -> LED_5V
- D144 pad 2: LED_GND -> Net-(D144-Pad2)
- D144 pad 3: Net-(D140-Pad1) -> LED_GND
- D144 pad 4: LED_5V -> Net-(D140-Pad2)
- D145 pad 1: Net-(D145-Pad1) -> LED_5V
- D145 pad 2: LED_GND -> Net-(D145-Pad2)
- D145 pad 3: Net-(D141-Pad1) -> LED_GND
- D145 pad 4: LED_5V -> Net-(D141-Pad2)
- D146 pad 1: Net-(D146-Pad1) -> LED_5V
- D146 pad 2: LED_GND -> Net-(D146-Pad2)
- D146 pad 3: Net-(D142-Pad1) -> LED_GND
- D146 pad 4: LED_5V -> Net-(D142-Pad2)
- D147 pad 1: Net-(D147-Pad1) -> LED_5V
- D147 pad 2: LED_GND -> Net-(D147-Pad2)
- D147 pad 3: Net-(D143-Pad1) -> LED_GND
- D147 pad 4: LED_5V -> Net-(D143-Pad2)
- D148 pad 1: Net-(D148-Pad1) -> LED_5V
- D148 pad 2: LED_GND -> Net-(D148-Pad2)
- D148 pad 3: Net-(D144-Pad1) -> LED_GND
- D148 pad 4: LED_5V -> Net-(D144-Pad2)
- D149 pad 1: Net-(D149-Pad1) -> LED_5V
- D149 pad 2: LED_GND -> Net-(D149-Pad2)
- D149 pad 3: Net-(D145-Pad1) -> LED_GND
- D149 pad 4: LED_5V -> Net-(D145-Pad2)
- D150 pad 1: Net-(D150-Pad1) -> LED_5V
- D150 pad 2: LED_GND -> Net-(D150-Pad2)
- D150 pad 3: Net-(D146-Pad1) -> LED_GND
- D150 pad 4: LED_5V -> Net-(D146-Pad2)
- D151 pad 1: Net-(D151-Pad1) -> LED_5V
- D151 pad 2: LED_GND -> Net-(D151-Pad2)
- D151 pad 3: Net-(D147-Pad1) -> LED_GND
- D151 pad 4: LED_5V -> Net-(D147-Pad2)
- D152 pad 1: Net-(D152-Pad1) -> LED_5V
- D152 pad 2: LED_GND -> Net-(D152-Pad2)
- D152 pad 3: Net-(D148-Pad1) -> LED_GND
- D152 pad 4: LED_5V -> Net-(D148-Pad2)
- D153 pad 1: Net-(D153-Pad1) -> LED_5V
- D153 pad 2: LED_GND -> Net-(D153-Pad2)
- D153 pad 3: Net-(D149-Pad1) -> LED_GND
- D153 pad 4: LED_5V -> Net-(D149-Pad2)
- D154 pad 1: Net-(D154-Pad1) -> LED_5V
- D154 pad 2: LED_GND -> Net-(D154-Pad2)
- D154 pad 3: Net-(D150-Pad1) -> LED_GND
- D154 pad 4: LED_5V -> Net-(D150-Pad2)
- D155 pad 1: Net-(D155-Pad1) -> LED_5V
- D155 pad 2: LED_GND -> Net-(D155-Pad2)
- D155 pad 3: Net-(D151-Pad1) -> LED_GND
- D155 pad 4: LED_5V -> Net-(D151-Pad2)
- D156 pad 1: Net-(D156-Pad1) -> LED_5V
- D156 pad 2: LED_GND -> Net-(D156-Pad2)
- D156 pad 3: Net-(D152-Pad1) -> LED_GND
- D156 pad 4: LED_5V -> Net-(D152-Pad2)
- D157 pad 1: Net-(D157-Pad1) -> LED_5V
- D157 pad 2: LED_GND -> Net-(D157-Pad2)
- D157 pad 3: Net-(D153-Pad1) -> LED_GND
- D157 pad 4: LED_5V -> Net-(D153-Pad2)
- D158 pad 1: Net-(D158-Pad1) -> LED_5V
- D158 pad 2: LED_GND -> Net-(D158-Pad2)
- D158 pad 3: Net-(D154-Pad1) -> LED_GND
- D158 pad 4: LED_5V -> Net-(D154-Pad2)
- D159 pad 1: Net-(D159-Pad1) -> LED_5V
- D159 pad 2: LED_GND -> Net-(D159-Pad2)
- D159 pad 3: Net-(D155-Pad1) -> LED_GND
- D159 pad 4: LED_5V -> Net-(D155-Pad2)
- D160 pad 1: Net-(D160-Pad1) -> LED_5V
- D160 pad 2: LED_GND -> Net-(D160-Pad2)
- D160 pad 3: Net-(D156-Pad1) -> LED_GND
- D160 pad 4: LED_5V -> Net-(D156-Pad2)
- D161 pad 1: Net-(D161-Pad1) -> LED_5V
- D161 pad 2: LED_GND -> Net-(D161-Pad2)
- D161 pad 3: Net-(D157-Pad1) -> LED_GND
- D161 pad 4: LED_5V -> Net-(D157-Pad2)
- D162 pad 1: Net-(D162-Pad1) -> LED_5V
- D162 pad 2: LED_GND -> Net-(D162-Pad2)
- D162 pad 3: Net-(D158-Pad1) -> LED_GND
- D162 pad 4: LED_5V -> Net-(D158-Pad2)
- D163 pad 1: Net-(D163-Pad1) -> LED_5V
- D163 pad 2: LED_GND -> Net-(D163-Pad2)
- D163 pad 3: Net-(D159-Pad1) -> LED_GND
- D163 pad 4: LED_5V -> Net-(D159-Pad2)
- D164 pad 1: Net-(D164-Pad1) -> LED_5V
- D164 pad 2: LED_GND -> Net-(D164-Pad2)
- D164 pad 3: Net-(D160-Pad1) -> LED_GND
- D164 pad 4: LED_5V -> Net-(D160-Pad2)
- D165 pad 1: Net-(D165-Pad1) -> LED_5V
- D165 pad 2: LED_GND -> Net-(D165-Pad2)
- D165 pad 3: Net-(D161-Pad1) -> LED_GND
- D165 pad 4: LED_5V -> Net-(D161-Pad2)
- D166 pad 1: Net-(D166-Pad1) -> LED_5V
- D166 pad 2: LED_GND -> Net-(D166-Pad2)
- D166 pad 3: Net-(D162-Pad1) -> LED_GND
- D166 pad 4: LED_5V -> Net-(D162-Pad2)
- D167 pad 1: Net-(D167-Pad1) -> LED_5V
- D167 pad 2: LED_GND -> Net-(D167-Pad2)
- D167 pad 3: Net-(D163-Pad1) -> LED_GND
- D167 pad 4: LED_5V -> Net-(D163-Pad2)
- D168 pad 1: Net-(D168-Pad1) -> LED_5V
- D168 pad 2: LED_GND -> Net-(D168-Pad2)
- D168 pad 3: Net-(D164-Pad1) -> LED_GND
- D168 pad 4: LED_5V -> Net-(D164-Pad2)
- D85 pad 1: Net-(D85-Pad1) -> LED_5V
- D85 pad 2: LED_GND -> Net-(D85-Pad2)
- D85 pad 3: /RGB/INPUT -> LED_GND
- D85 pad 4: LED_5V -> /RGB/INPUT
- D86 pad 1: Net-(D86-Pad1) -> LED_5V
- D86 pad 2: LED_GND -> Net-(D86-Pad2)
- D86 pad 3: Net-(D168-Pad1) -> LED_GND
- D86 pad 4: LED_5V -> Net-(D168-Pad2)
- D87 pad 1: Net-(D87-Pad1) -> LED_5V
- D87 pad 2: LED_GND -> Net-(D87-Pad2)
- D87 pad 3: Net-(D165-Pad1) -> LED_GND
- D87 pad 4: LED_5V -> Net-(D165-Pad2)
- D88 pad 1: Net-(D88-Pad1) -> LED_5V
- D88 pad 2: LED_GND -> Net-(D88-Pad2)
- D88 pad 3: Net-(D166-Pad1) -> LED_GND
- D88 pad 4: LED_5V -> Net-(D166-Pad2)
- D89 pad 1: Net-(D89-Pad1) -> LED_5V
- D89 pad 2: LED_GND -> Net-(D89-Pad2)
- D89 pad 3: Net-(D167-Pad1) -> LED_GND
- D89 pad 4: LED_5V -> Net-(D167-Pad2)
- D90 pad 1: Net-(D90-Pad1) -> LED_5V
- D90 pad 2: LED_GND -> Net-(D90-Pad2)
- D90 pad 3: Net-(D85-Pad1) -> LED_GND
- D90 pad 4: LED_5V -> Net-(D85-Pad2)
- D91 pad 1: Net-(D91-Pad1) -> LED_5V
- D91 pad 2: LED_GND -> Net-(D91-Pad2)
- D91 pad 3: Net-(D86-Pad1) -> LED_GND
- D91 pad 4: LED_5V -> Net-(D86-Pad2)
- D92 pad 1: Net-(D92-Pad1) -> LED_5V
- D92 pad 2: LED_GND -> Net-(D92-Pad2)
- D92 pad 3: Net-(D87-Pad1) -> LED_GND
- D92 pad 4: LED_5V -> Net-(D87-Pad2)
- D93 pad 1: Net-(D93-Pad1) -> LED_5V
- D93 pad 2: LED_GND -> Net-(D93-Pad2)
- D93 pad 3: Net-(D88-Pad1) -> LED_GND
- D93 pad 4: LED_5V -> Net-(D88-Pad2)
- D94 pad 1: Net-(D94-Pad1) -> LED_5V
- D94 pad 2: LED_GND -> Net-(D94-Pad2)
- D94 pad 3: Net-(D89-Pad1) -> LED_GND
- D94 pad 4: LED_5V -> Net-(D89-Pad2)
- D95 pad 1: Net-(D100-Pad3) -> LED_5V
- D95 pad 2: LED_GND -> Net-(D100-Pad4)
- D95 pad 3: Net-(D90-Pad1) -> LED_GND
- D95 pad 4: LED_5V -> Net-(D90-Pad2)
- D96 pad 1: Net-(D101-Pad3) -> LED_5V
- D96 pad 2: LED_GND -> Net-(D101-Pad4)
- D96 pad 3: Net-(D91-Pad1) -> LED_GND
- D96 pad 4: LED_5V -> Net-(D91-Pad2)
- D97 pad 1: Net-(D102-Pad3) -> LED_5V
- D97 pad 2: LED_GND -> Net-(D102-Pad4)
- D97 pad 3: Net-(D92-Pad1) -> LED_GND
- D97 pad 4: LED_5V -> Net-(D92-Pad2)
- D98 pad 1: Net-(D103-Pad3) -> LED_5V
- D98 pad 2: LED_GND -> Net-(D103-Pad4)
- D98 pad 3: Net-(D93-Pad1) -> LED_GND
- D98 pad 4: LED_5V -> Net-(D93-Pad2)
- D99 pad 1: (no net) -> LED_5V
- D99 pad 2: LED_GND -> (no net)
- D99 pad 3: Net-(D94-Pad1) -> LED_GND
- D99 pad 4: LED_5V -> Net-(D94-Pad2)

Commit message: working on led
Parts:
- moved D141 16.4 mm to (13.1, -64.9)

Commit message: working on the WS2812
Parts:
- RIGHT-SHIFT1: footprint daprice-keyswitches:Stabilizer_MX_2.25u -> daprice-keyswitches:Stabilizer_MX_2.75u
- RightMeta1: renamed from SW61; footprint daprice-keyswitches:Kailh_socket_MX -> daprice-keyswitches:Stabilizer_MX_1.25u
- moved D12 188.1 mm to (145.5, 66.3)
- moved D83 150.9 mm to (124.5, 66.3)
- moved D10 149.4 mm to (187.6, 66.3)
- moved D2 148.6 mm to (166.6, 66.3)
- moved D141 131.2 mm to (45.2, 62.4)
- moved D21 126.1 mm to (198.1, 66.3)
- moved D13 124.9 mm to (177.1, 66.3)
- moved D9 123.9 mm to (156.0, 66.3)
- moved D14 123.6 mm to (92.2, 85.2)
- moved D82 123.2 mm to (98.2, 66.3)
- moved D22 122.8 mm to (113.2, 85.2)
- moved D1 122.8 mm to (135.0, 66.3)
- moved D26 122.2 mm to (134.3, 85.2)
- moved D34 121.5 mm to (155.3, 85.2)
- moved D38 120.8 mm to (176.3, 85.2)
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
Commit message: working on layout
Parts:
- C1, C10, C11, C12, C13, C14, C15, C16, C17, C18, C19, C2, C20, C21, C22, C23, C24, C25, C26, C27, C28, C29, C3, C30, C31, C32, C33, C34, C35, C36, C37, C38, C39, C4, C40, C41, C42, C43, C44, C45, C46, C47, C48, C49, C5, C50, C51, C52, C53, C54, C55, C56, C57, C58, C59, C6, C60, C61, C62, C63, C64, C65, C66, C67, C68, C69, C7, C70, C71, C72, C73, C74, C75, C76, C77, C78, C79, C8, C80, C81, C82, C83, C84, C85, C86, C87, C88, C89, C9, C90, C91, C92, D1, D10, D11, D12, D13, D14, D15, D16, D17, D18, D19, D2, D20, D21, D22, D23, D24, D25, D26, D27, D28, D29, D3, D30, D31, D32, D33, D34, D35, D36, D37, D38, D39, D4, D40, D41, D42, D43, D44, D45, D46, D47, D48, D49, D5, D50, D51, D52, D53, D54, D55, D56, D57, D58, D59, D6, D60, D61, D62, D63, D64, D65, D66, D67, D68, D69, D7, D70, D71, D72, D73, D74, D75, D76, D77, D78, D79, D8, D80, D81, D82, D83, D84, D9, R1, R2, R3, R4, U1, Y1: moved to F.Cu
- moved D42 285.1 mm to (390.2, 125.4), turned to 90 degrees
- moved D14 284.1 mm to (373.4, 125.4), turned to 90 degrees
- moved D25 278.4 mm to (378.2, 125.4), turned to 90 degrees
- moved D22 277.5 mm to (387.8, 125.4), turned to 90 degrees
- moved D41 252.7 mm to (347.0, 125.4), turned to 90 degrees
- moved D28 250.5 mm to (371.0, 125.4), turned to 90 degrees
- moved D26 249.6 mm to (380.6, 125.4), turned to 90 degrees
- moved D54 245.9 mm to (392.6, 125.4), turned to 90 degrees
- moved D43 239.1 mm to (354.2, 125.4), turned to 90 degrees
- moved D32 231.9 mm to (318.7, 119.7)
- moved D82 230.9 mm to (324.3, 112.8)
- moved D37 225.5 mm to (361.4, 125.4), turned to 90 degrees
- moved D6 221.6 mm to (324.3, 117.4)
- moved D5 216.8 mm to (318.7, 91.9)
- moved D34 212.3 mm to (363.8, 125.4), turned to 90 degrees
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
Commit message: almost ready to send off
Parts:
- added J2: USB_B_Mini, Connector_USB:USB_Mini-B_Wuerth_65100516121_Horizontal, F.Cu at (323.1, 28.5)
- added SW_RESET1: SW_Push, CHGRAY_LED:SW_SPST_JLC_PCB_C520860, F.Cu at (323.8, 120.7)
- Y1-16hz1: renamed from Y1; footprint Crystal:Crystal_SMD_5032-2Pin_5.0x3.2mm_HandSoldering -> Crystal:Crystal_SMD_HC49-SD
- moved D75 317.6 mm to (73.4, 66.1), turned to 0 degrees
- moved D26 301.8 mm to (89.1, 47.0), turned to 0 degrees
- moved D24 294.8 mm to (98.8, 47.0), turned to 0 degrees
- moved D49 289.5 mm to (54.0, 66.1), turned to 0 degrees
- moved D54 286.6 mm to (112.2, 66.1), turned to 0 degrees
- moved D34 282.1 mm to (88.0, 66.1), turned to 0 degrees
- moved D37 278.3 mm to (86.0, 85.2), turned to 0 degrees
- moved D61 276.0 mm to (71.6, 85.2), turned to 0 degrees
- moved D43 275.9 mm to (81.2, 85.2), turned to 0 degrees
- moved D33 275.8 mm to (95.7, 85.2), turned to 0 degrees
- moved D78 273.3 mm to (124.7, 85.3), turned to 0 degrees
- moved D69 269.8 mm to (60.0, 47.0)
- moved D63 269.1 mm to (58.9, 66.1)
- moved D80 268.4 mm to (134.4, 85.3), turned to 0 degrees
- moved D62 265.5 mm to (107.4, 66.1), turned to 0 degrees
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Connections:
- C92 pad 1: (no net) -> Net-(C92-Pad1)
- R2 pad 2: (no net) -> Net-(J2-Pad3)
- R3 pad 2: (no net) -> Net-(J2-Pad2)
Other:
- board text added: "LOG0.Key.Yeet2.5"
- board text removed: "LOG0.Key.Yeet3"

Commit message: leds
Parts:
- moved D50 106.2 mm to (202.1, 85.3)
Routing:
- net LED_5V: track 0.00 -> 2062.5 mm, vias 0 -> 20
- net LED_GND: track 0.00 -> 2006.4 mm, vias 0 -> 16
- net ROW4: track 0.00 -> 605.3 mm, vias 0 -> 4
- net ROW0: track 0.00 -> 571.2 mm, vias 0 -> 3
- net ROW1: track 0.00 -> 521.2 mm, vias 0 -> 7
- net ROW3: track 0.00 -> 515.5 mm, vias 0 -> 6
- net ROW2: track 0.00 -> 431.1 mm, vias 0 -> 9
- net COL10: track 0.00 -> 426.0 mm, vias 0 -> 7
- net ROW5: track 0.00 -> 376.1 mm, vias 0 -> 1
- net /RGB/INPUT: track 0.00 -> 365.7 mm, vias 0 -> 4
- net Net-(D16-Pad1): track 0.00 -> 360.7 mm, vias 0 -> 3
- net COL4: track 0.00 -> 353.9 mm, vias 0 -> 8
- net COL13: track 0.00 -> 320.0 mm, vias 0 -> 7
- net Net-(D76-Pad1): track 0.00 -> 313.9 mm, vias 0 -> 5
- net COL8: track 0.00 -> 311.0 mm, vias 0 -> 6
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
Commit message: trying to clean up diodes
Parts:
- moved D69 337.0 mm to (392.1, 104.2)
- moved D82 306.5 mm to (382.4, 104.2)
- moved D59 291.8 mm to (371.2, 46.9)
- moved D16 286.9 mm to (361.5, 46.9)
- moved D60 283.8 mm to (376.0, 46.9)
- moved D68 282.1 mm to (351.8, 46.9)
- moved D83 277.8 mm to (387.3, 104.2)
- moved D75 277.7 mm to (348.5, 104.2)
- moved D62 274.1 mm to (380.9, 46.9)
- moved D64 250.0 mm to (366.3, 46.9)
- moved D78 239.1 mm to (363.0, 104.2)
- moved D79 239.1 mm to (367.9, 104.2)
- moved D80 239.1 mm to (372.7, 104.2)
- moved D76 234.3 mm to (353.3, 104.2)
- moved D71 230.3 mm to (395.4, 46.9)
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Connections:
- J1 pad 14: LED_GND -> LED_5V
- J1 pad 2: LED_5V -> LED_GND
Routing:
- net LED_5V: track 2062.5 -> 0.00 mm, vias 20 -> 0
- net LED_GND: track 2006.4 -> 0.00 mm, vias 16 -> 0
- net ROW4: track 605.3 -> 0.00 mm, vias 4 -> 0
- net ROW0: track 571.2 -> 0.00 mm, vias 3 -> 0
- net ROW1: track 521.2 -> 0.00 mm, vias 7 -> 0
- net ROW3: track 515.5 -> 0.00 mm, vias 6 -> 0
- net ROW2: track 431.1 -> 0.00 mm, vias 9 -> 0
- net COL10: track 426.0 -> 0.00 mm, vias 7 -> 0
- net ROW5: track 376.1 -> 0.00 mm, vias 1 -> 0
- net /RGB/INPUT: track 365.7 -> 0.00 mm, vias 4 -> 0
- net Net-(D16-Pad1): track 360.7 -> 0.00 mm, vias 3 -> 0
- net COL4: track 353.9 -> 0.00 mm, vias 8 -> 0
- net COL13: track 320.0 -> 0.00 mm, vias 7 -> 0
- net Net-(D76-Pad1): track 313.9 -> 0.00 mm, vias 5 -> 0
- net COL8: track 311.0 -> 0.00 mm, vias 6 -> 0
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
Commit message: about to send off
Routing:
- net LED_5V: track 0.00 -> 2088.8 mm, vias 0 -> 17
- net LED_GND: track 0.00 -> 2050.3 mm, vias 0 -> 20
- net ROW4: track 0.00 -> 594.0 mm, vias 0 -> 3
- net ROW3: track 0.00 -> 578.7 mm, vias 0 -> 7
- net ROW1: track 0.00 -> 492.7 mm, vias 0 -> 7
- net ROW0: track 0.00 -> 487.3 mm, vias 0 -> 3
- net COL0: track 0.00 -> 484.2 mm, vias 0 -> 7
- net ROW5: track 0.00 -> 476.9 mm, vias 0 -> 6
- net ROW2: track 0.00 -> 473.3 mm, vias 0 -> 10
- net COL11: track 0.00 -> 457.2 mm, vias 0 -> 7
- net COL4: track 0.00 -> 454.7 mm, vias 0 -> 5
- net COL2: track 0.00 -> 436.9 mm, vias 0 -> 5
- net COL5: track 0.00 -> 436.7 mm, vias 0 -> 7
- net COL1: track 0.00 -> 396.8 mm, vias 0 -> 9
- net COL7: track 0.00 -> 384.9 mm, vias 0 -> 5
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