File: microcontroller.sch (KiCad schematic (older format))
At the start: 11 parts, among them J2 USB_B_Mini, U2 ATmega32U4-AU, Y1 Crystal

Commit message: updates to be nearly functional
Parts:
- added C85, C87, C88, C89: 0.1u, Capacitor_SMD:C_0805_2012Metric, symbol Device:C
- added C91: 22p, Capacitor_SMD:C_0805_2012Metric, symbol Device:C
- C86: value C -> 0.1u; footprint (none) -> Capacitor_SMD:C_0805_2012Metric
- C90: renamed from C85; value C -> 22p; footprint (none) -> Capacitor_SMD:C_0805_2012Metric
- C92: renamed from C87; value C -> 1u; footprint (none) -> Capacitor_SMD:C_0805_2012Metric
- R1: value R -> 10k; footprint (none) -> Resistor_SMD:R_1206_3216Metric
- R2, R3: value R -> 22R; footprint (none) -> Resistor_SMD:R_0805_2012Metric
- R4: footprint (none) -> Resistor_SMD:R_1206_3216Metric
- Y1: footprint (none) -> Crystal:Crystal_SMD_5032-2Pin
- renumbered U2 to U1
Connections:
- wire segments 63 -> 71
Changed lines of the file:
@@
 P 6900 4350
 F 0 "R4" V 6693 4350 50  0000 C CNN
-F 1 "R10K" V 6800 4350 50  0000 C CNN
-F 2 "" V 6830 4350 50  0001 C CNN
-F 3 "~" H 6900 4350 50  0001 C CNN
+F 1 "R10K" V 6900 4350 50  0000 C CNN
+F 2 "Resistor_SMD:R_1206_3216Metric" V 6830 4350 50  0001 C CNN
+F 3 "1206W4F1002T5E " H 6900 4350 50  0001 C CNN
 	1    6900 4350
 	0    1    1    0
 $EndComp
 $Comp
-L power:GND #PWR013
+L power:GND #PWR015
 U 1 1 60A87FCE
 P 7050 4350
-F 0 "#PWR013" H 7050 4100 50  0001 C CNN
+F 0 "#PWR015" H 7050 4100 50  0001 C CNN
 F 1 "GND" V 7055 4222 50  0000 R CNN
 F 2 "" H 7050 4350 50  0001 C CNN
@@
 	6600 4350 6750 4350
 $Comp
-L power:GND #PWR09
+L power:GND #PWR011
 U 1 1 60A89E63
 P 5900 5550
-F 0 "#PWR09" H 5900 5300 50  0001 C CNN
+F 0 "#PWR011" H 5900 5300 50  0001 C CNN
 F 1 "GND" H 5905 5377 50  0000 C CNN
 F 2 "" H 5900 5550 50  0001 C CNN
@@
 $EndComp
 $Comp
-L power:GND #PWR011
+L power:GND #PWR013
 U 1 1 60A8ACF7
 P 6000 5550
-F 0 "#PWR011" H 6000 5300 50  0001 C CNN
+F 0 "#PWR013" H 6000 5300 50  0001 C CNN
 F 1 "GND" H 6005 5377 50  0000 C CNN
 F 2 "" H 6000 5550 50  0001 C CNN
@@
 $EndComp
 $Comp
-L power:VCC #PWR08
+L power:VCC #PWR010
 U 1 1 60A8BA34
 P 5900 1950
-F 0 "#PWR08" H 5900 1800 50  0001 C CNN
+F 0 "#PWR010" H 5900 1800 50  0001 C CNN
 F 1 "VCC" H 5915 2123 50  0000 C CNN
 F 2 "" H 5900 1950 50  0001 C CNN
@@
 $EndComp
 $Comp
-L power:VCC #PWR010
+L power:VCC #PWR012
 U 1 1 60A8C7C2
 P 6000 1950
-F 0 "#PWR010" H 6000 1800 50  0001 C CNN
+F 0 "#PWR012" H 6000 1800 50  0001 C CNN
 F 1 "VCC" H 6015 2123 50  0000 C CNN
 F 2 "" H 6000 1950 50  0001 C CNN
@@
 $EndComp
 $Comp
-L power:VCC #PWR012
+L power:VCC #PWR014
 U 1 1 60A8CCBE
 P 6100 1950
-F 0 "#PWR012" H 6100 1800 50  0001 C CNN
+F 0 "#PWR014" H 6100 1800 50  0001 C CNN
 F 1 "VCC" H 6115 2123 50  0000 C CNN
 F 2 "" H 6100 1950 50  0001 C CNN
@@
 F 0 "Y1" V 4554 2681 50  0000 L CNN
 F 1 "Crystal" V 4645 2681 50  0000 L CNN
-F 2 "" H 4600 2550 50  0001 C CNN
-F 3 "~" H 4600 2550 50  0001 C CNN
+F 2 "Crystal:Crystal_SMD_5032-2Pin" H 4600 2550 50  0001 C CNN
+F 3 "X1G004451000200 " H 4600 2550 50  0001 C CNN
 	1    4600 2550
 	0    1    1    0
 $EndComp
 $Comp
-L Device:C C85
+L Device:C C90
 U 1 1 60A8F4F8
 P 4050 2400
-F 0 "C85" V 3798 2400 50  0000 C CNN
-F 1 "C" V 3889 2400 50  0000 C CNN
-F 2 "" H 4088 2250 50  0001 C CNN
-F 3 "~" H 4050 2400 50  0001 C CNN
+F 0 "C90" V 3798 2400 50  0000 C CNN
+F 1 "22p" V 3889 2400 50  0000 C CNN
+F 2 "Capacitor_SMD:C_0805_2012Metric" H 4088 2250 50  0001 C CNN
+F 3 "CL21C220JBANNNC " H 4050 2400 50  0001 C CNN
 	1    4050 2400
-	0    1    1    0
-$EndComp
-$Comp
-L Device:C C86
-U 1 1 60A9094F
-P 4050 2700
-F 0 "C86" V 3798 2700 50  0000 C CNN
-F 1 "C" V 3889 2700 50  0000 C CNN
-F 2 "" H 4088 2550 50  0001 C CNN
-F 3 "~" H 4050 2700 50  0001 C CNN
-	1    4050 2700
 	0    1    1    0
 $EndComp
@@
 	3600 2700 3900 2700
 $Comp
-L power:GND #PWR03
+L power:GND #PWR05
 U 1 1 60A92E00
 P 3300 2550
-F 0 "#PWR03" H 3300 2300 50  0001 C CNN
+F 0 "#PWR05" H 3300 2300 50  0001 C CNN
 F 1 "GND" V 3305 2422 50  0000 R CNN
 F 2 "" H 3300 2550 50  0001 C CNN
@@
 P 3950 1200
 F 0 "R1" H 4020 1246 50  0000 L CNN
-F 1 "R" H 4020 1155 50  0000 L CNN
-F 2 "" V 3880 1200 50  0001 C CNN
-F 3 "~" H 3950 1200 50  0001 C CNN
+F 1 "10k" H 4020 1155 50  0000 L CNN
+F 2 "Resistor_SMD:R_1206_3216Metric" V 3880 1200 50  0001 C CNN
+F 3 "1206W4F1002T5E " H 3950 1200 50  0001 C CNN
 	1    3950 1200
 	1    0    0    -1
@@
 $EndComp
 $Comp
-L power:GND #PWR06
+L power:GND #PWR08
 U 1 1 60A95E1A
 P 4350 650
-F 0 "#PWR06" H 4350 400 50  0001 C CNN
+F 0 "#PWR08" H 4350 400 50  0001 C CNN
 F 1 "GND" H 4355 477 50  0000 C CNN
 F 2 "" H 4350 650 50  0001 C CNN
@@
 	4350 650  4350 1000
 $Comp
-L power:VCC #PWR04
+L power:VCC #PWR06
 U 1 1 60A972A5
 P 3950 1050
-F 0 "#PWR04" H 3950 900 50  0001 C CNN
+F 0 "#PWR06" H 3950 900 50  0001 C CNN
 F 1 "VCC" H 3965 1223 50  0000 C CNN
 F 2 "" H 3950 1050 50  0001 C CNN
@@
 P 4450 4350
 F 0 "R2" V 4243 4350 50  0000 C CNN
-F 1 "R" V 4334 4350 50  0000 C CNN
-F 2 "" V 4380 4350 50  0001 C CNN
-F 3 "~" H 4450 4350 50  0001 C CNN
+F 1 "22R" V 4450 4350 50  0000 C CNN
+F 2 "Resistor_SMD:R_0805_2012Metric" V 4380 4350 50  0001 C CNN
+F 3 "0805W8F220JT5E " H 4450 4350 50  0001 C CNN
 	1    4450 4350
 	0    1    1    0
 $EndComp
-$Comp
-L Device:R R3
-U 1 1 60A9D28A
-P 4450 4550
-F 0 "R3" V 4243 4550 50  0000 C CNN
-F 1 "R" V 4334 4550 50  0000 C CNN
-F 2 "" V 4380 4550 50  0001 C CNN
-F 3 "~" H 4450 4550 50  0001 C CNN
-	1    4450 4550
-	0    1    1    0
-$EndComp
 Wire Wire Line
 	4050 4500 4300 4500
@@
 	5200 4550 4600 4550
 $Comp
-L power:VCC #PWR05
+L power:VCC #PWR07
 U 1 1 60AA0262
 P 4250 4050
-F 0 "#PWR05" H 4250 3900 50  0001 C CNN
+F 0 "#PWR07" H 4250 3900 50  0001 C CNN
 F 1 "VCC" H 4265 4223 50  0000 C CNN
 F 2 "" H 4250 4050 50  0001 C CNN
@@
 NoConn ~ 4050 4600
 $Comp
-L Device:C C87
+L Device:C C92
 U 1 1 60AA1797
 P 4400 5050
-F 0 "C87" V 4652 5050 50  0000 C CNN
-F 1 "C" V 4561 5050 50  0000 C CNN
-F 2 "" H 4438 4900 50  0001 C CNN
-F 3 "~" H 4400 5050 50  0001 C CNN
+F 0 "C92" V 4652 5050 50  0000 C CNN
+F 1 "1u" V 4561 5050 50  0000 C CNN
+F 2 "Capacitor_SMD:C_0805_2012Metric" H 4438 4900 50  0001 C CNN
+F 3 "CL21B105KBFNNNE " H 4400 5050 50  0001 C CNN
 	1    4400 5050
 	0    -1   -1   0
@@
 	6600 2250 6800 2250
 $Comp
-L power:VCC #PWR07
+L power:VCC #PWR09
 U 1 1 60AAA3DE
 P 4900 3050
-F 0 "#PWR07" H 4900 2900 50  0001 C CNN
+F 0 "#PWR09" H 4900 2900 50  0001 C CNN
 F 1 "VCC" V 4915 3177 50  0000 L CNN
 F 2 "" H 4900 3050 50  0001 C CNN
@@
 	6600 5150 6800 5150
 $Comp
-L MCU_Microchip_ATmega:ATmega32U4-AU U2
+L MCU_Microchip_ATmega:ATmega32U4-AU U1
 U 1 1 60A82FF7
 P 6000 3750
-F 0 "U2" H 6000 1861 50  0000 C CNN
+F 0 "U1" H 6000 1861 50  0000 C CNN
 F 1 "ATmega32U4-AU" H 6000 1770 50  0000 C CNN
 F 2 "Package_QFP:TQFP-44_10x10mm_P0.8mm" H 6000 3750 50  0001 C CIN
@@
 	6600 3250 6800 3250
 NoConn ~ 5400 2850
+$Comp
+L Device:C C85
+U 1 1 60BB0957
+P 2200 6100
+F 0 "C85" H 2315 6146 50  0000 L CNN
+F 1 "0.1u" H 2315 6055 50  0000 L CNN
+F 2 "Capacitor_SMD:C_0805_2012Metric" H 2238 5950 50  0001 C CNN
+F 3 "C0805C104J5RACAUTO" H 2200 6100 50  0001 C CNN
+	1    2200 6100
+	1    0    0    -1
+$EndComp
+$Comp
+L Device:C C88
+U 1 1 60BB15A4
+P 3450 6100
+F 0 "C88" H 3565 6146 50  0000 L CNN
+F 1 "0.1u" H 3565 6055 50  0000 L CNN
+F 2 "Capacitor_SMD:C_0805_2012Metric" H 3488 5950 50  0001 C CNN
+F 3 "C0805C104J5RACAUTO" H 3450 6100 50  0001 C CNN
+	1    3450 6100
+	1    0    0    -1
+$EndComp
+$Comp
+L Device:C C86
+U 1 1 60BB2F1B
+P 2650 6100
+F 0 "C86" H 2765 6146 50  0000 L CNN
+F 1 "0.1u" H 2765 6055 50  0000 L CNN
+F 2 "Capacitor_SMD:C_0805_2012Metric" H 2688 5950 50  0001 C CNN
+F 3 "C0805C104J5RACAUTO" H 2650 6100 50  0001 C CNN
+	1    2650 6100
+	1    0    0    -1
+$EndComp
+$Comp
+L Device:C C87
+U 1 1 60BB46FD
+P 3050 6100
+F 0 "C87" H 3165 6146 50  0000 L CNN
+F 1 "0.1u" H 3165 6055 50  0000 L CNN
+F 2 "Capacitor_SMD:C_0805_2012Metric" H 3088 5950 50  0001 C CNN
+F 3 "C0805C104J5RACAUTO" H 3050 6100 50  0001 C CNN
+	1    3050 6100
+	1    0    0    -1
+$EndComp
+Wire Wire Line
+	2200 5950 2650 5950
+Wire Wire Line
+	3050 5950 3450 5950
+Wire Wire Line
+	2650 5950 3050 5950
+Connection ~ 2650 5950
+Connection ~ 3050 5950
+Wire Wire Line
+	2200 6250 2650 6250
+Wire Wire Line
+	3050 6250 2650 6250
+Connection ~ 2650 6250
+Wire Wire Line
+	3050 6250 3450 6250
+Connection ~ 3050 6250
+$Comp
+L Device:C C89
+U 1 1 60BBF39F
+P 3850 6100
+F 0 "C89" H 3965 6146 50  0000 L CNN
+F 1 "0.1u" H 3965 6055 50  0000 L CNN
+F 2 "Capacitor_SMD:C_0805_2012Metric" H 3888 5950 50  0001 C CNN
+F 3 "C0805C104J5RACAUTO" H 3850 6100 50  0001 C CNN
+	1    3850 6100
+	1    0    0    -1
+$EndComp
+Wire Wire Line
+	3450 5950 3850 5950
+Connection ~ 3450 5950
+Wire Wire Line
+	3450 6250 3850 6250
+Connection ~ 3450 6250
+$Comp
+L power:VCC #PWR03
+U 1 1 60BC98D5
+P 2200 5950
+F 0 "#PWR03" H 2200 5800 50  0001 C CNN
+F 1 "VCC" H 2215 6123 50  0000 C CNN
+F 2 "" H 2200 5950 50  0001 C CNN
+F 3 "" H 2200 5950 50  0001 C CNN
+	1    2200 5950
+	1    0    0    -1
+$EndComp
+$Comp
+L power:GND #PWR04
+U 1 1 60BCBB0F
+P 2200 6250
+F 0 "#PWR04" H 2200 6000 50  0001 C CNN
+F 1 "GND" H 2205 6077 50  0000 C CNN
+F 2 "" H 2200 6250 50  0001 C CNN
+F 3 "" H 2200 6250 50  0001 C CNN
+	1    2200 6250
+	1    0    0    -1
+$EndComp
+Connection ~ 2200 6250
+Connection ~ 2200 5950
+$Comp
+L Device:C C91
+U 1 1 60BD615F
+P 4050 2700
+F 0 "C91" V 3798 2700 50  0000 C CNN
+F 1 "22p" V 3889 2700 50  0000 C CNN
+F 2 "Capacitor_SMD:C_0805_2012Metric" H 4088 2550 50  0001 C CNN
+F 3 "CL21C220JBANNNC " H 4050 2700 50  0001 C CNN
+	1    4050 2700
+	0    1    1    0
+$EndComp
+$Comp
+L Device:R R3
+U 1 1 60BDEC5A
+P 4450 4550
+F 0 "R3" V 4243 4550 50  0000 C CNN
+F 1 "22R" V 4450 4550 50  0000 C CNN
+F 2 "Resistor_SMD:R_0805_2012Metric" V 4380 4550 50  0001 C CNN
+F 3 "0805W8F220JT5E " H 4450 4550 50  0001 C CNN
+	1    4450 4550
+	0    1    1    0
+$EndComp
 $EndSCHEMATC

Commit message: almost ready to send off
Parts:
- J2: footprint (none) -> Connector_USB:USB_Mini-B_Wuerth_65100516121_Horizontal
- SW_RESET1: footprint (none) -> CHGRAY_LED:SW_SPST_JLC_PCB_C520860
- Y1-16hz1: renamed from Y1; footprint Crystal:Crystal_SMD_5032-2Pin -> Crystal:Crystal_SMD_HC49-SD
Changed lines of the file:
@@
 $Descr A4 11693 8268
 encoding utf-8
-Sheet 4 4
+Sheet 3 4
 Title ""
 Date ""
@@
 $EndComp
 $Comp
-L Device:Crystal Y1
+L Device:Crystal Y1-16hz1
 U 1 1 60A8D8F1
 P 4600 2550
-F 0 "Y1" V 4554 2681 50  0000 L CNN
+F 0 "Y1-16hz1" V 4554 2681 50  0000 L CNN
 F 1 "Crystal" V 4645 2681 50  0000 L CNN
-F 2 "Crystal:Crystal_SMD_5032-2Pin" H 4600 2550 50  0001 C CNN
-F 3 "X1G004451000200 " H 4600 2550 50  0001 C CNN
+F 2 "Crystal:Crystal_SMD_HC49-SD" H 4600 2550 50  0001 C CNN
+F 3 "X49SM16MSD2SC " H 4600 2550 50  0000 C CNN
 	1    4600 2550
 	0    1    1    0
@@
 F 0 "SW_RESET1" V 4304 1348 50  0000 L CNN
 F 1 "SW_Push" V 4395 1348 50  0000 L CNN
-F 2 "" H 4350 1400 50  0001 C CNN
-F 3 "~" H 4350 1400 50  0001 C CNN
+F 2 "CHGRAY_LED:SW_SPST_JLC_PCB_C520860" H 4350 1400 50  0000 C CNN
+F 3 "C520860" H 4350 1400 50  0001 C CNN
 	1    4350 1200
 	0    1    1    0
@@
 F 0 "J2" H 3807 4867 50  0000 C CNN
 F 1 "USB_B_Mini" H 3807 4776 50  0000 C CNN
-F 2 "" H 3900 4350 50  0001 C CNN
-F 3 "~" H 3900 4350 50  0001 C CNN
+F 2 "Connector_USB:USB_Mini-B_Wuerth_65100516121_Horizontal" H 3900 4350 50  0001 C CNN
+F 3 "920-462A2021S10100" H 3900 4350 50  0001 C CNN
 	1    3750 4400
 	1    0    0    -1

Commit message: almost done
Parts:
- R1: value 10k -> R10k
- R4: value R10K -> R10k
Changed lines of the file:
@@
 P 6900 4350
 F 0 "R4" V 6693 4350 50  0000 C CNN
-F 1 "R10K" V 6900 4350 50  0000 C CNN
+F 1 "R10k" V 6900 4350 50  0000 C CNN
 F 2 "Resistor_SMD:R_1206_3216Metric" V 6830 4350 50  0001 C CNN
-F 3 "1206W4F1002T5E " H 6900 4350 50  0001 C CNN
+F 3 "C17902" H 6900 4350 50  0001 C CNN
 	1    6900 4350
 	0    1    1    0
@@
 F 1 "Crystal" V 4645 2681 50  0000 L CNN
 F 2 "Crystal:Crystal_SMD_HC49-SD" H 4600 2550 50  0001 C CNN
-F 3 "X49SM16MSD2SC " H 4600 2550 50  0000 C CNN
+F 3 "C12676" H 4600 2550 50  0000 C CNN
 	1    4600 2550
 	0    1    1    0
@@
 F 1 "22p" V 3889 2400 50  0000 C CNN
 F 2 "Capacitor_SMD:C_0805_2012Metric" H 4088 2250 50  0001 C CNN
-F 3 "CL21C220JBANNNC " H 4050 2400 50  0001 C CNN
+F 3 "C1804" H 4050 2400 50  0001 C CNN
 	1    4050 2400
 	0    1    1    0
@@
 P 3950 1200
 F 0 "R1" H 4020 1246 50  0000 L CNN
-F 1 "10k" H 4020 1155 50  0000 L CNN
+F 1 "R10k" H 4020 1155 50  0000 L CNN
 F 2 "Resistor_SMD:R_1206_3216Metric" V 3880 1200 50  0001 C CNN
-F 3 "1206W4F1002T5E " H 3950 1200 50  0001 C CNN
+F 3 "C17902" H 3950 1200 50  0001 C CNN
 	1    3950 1200
 	1    0    0    -1
@@
 F 1 "USB_B_Mini" H 3807 4776 50  0000 C CNN
 F 2 "Connector_USB:USB_Mini-B_Wuerth_65100516121_Horizontal" H 3900 4350 50  0001 C CNN
-F 3 "920-462A2021S10100" H 3900 4350 50  0001 C CNN
+F 3 "C69074" H 3900 4350 50  0001 C CNN
 	1    3750 4400
 	1    0    0    -1
@@
 F 1 "22R" V 4450 4350 50  0000 C CNN
 F 2 "Resistor_SMD:R_0805_2012Metric" V 4380 4350 50  0001 C CNN
-F 3 "0805W8F220JT5E " H 4450 4350 50  0001 C CNN
+F 3 "C17561" H 4450 4350 50  0001 C CNN
 	1    4450 4350
 	0    1    1    0
@@
 F 1 "1u" V 4561 5050 50  0000 C CNN
 F 2 "Capacitor_SMD:C_0805_2012Metric" H 4438 4900 50  0001 C CNN
-F 3 "CL21B105KBFNNNE " H 4400 5050 50  0001 C CNN
+F 3 "C28323" H 4400 5050 50  0001 C CNN
 	1    4400 5050
 	0    -1   -1   0
@@
 F 1 "ATmega32U4-AU" H 6000 1770 50  0000 C CNN
 F 2 "Package_QFP:TQFP-44_10x10mm_P0.8mm" H 6000 3750 50  0001 C CIN
-F 3 "http://ww1.microchip.com/downloads/en/DeviceDoc/Atmel-7766-8-bit-AVR-ATmega16U4-32U4_Datasheet.pdf" H 6000 3750 50  0001 C CNN
+F 3 "C44854" H 6000 3750 50  0001 C CNN
 	1    6000 3750
 	1    0    0    -1
@@
 F 1 "0.1u" H 2315 6055 50  0000 L CNN
 F 2 "Capacitor_SMD:C_0805_2012Metric" H 2238 5950 50  0001 C CNN
-F 3 "C0805C104J5RACAUTO" H 2200 6100 50  0001 C CNN
+F 3 "C696366" H 2200 6100 50  0001 C CNN
 	1    2200 6100
 	1    0    0    -1
@@
 F 1 "0.1u" H 3565 6055 50  0000 L CNN
 F 2 "Capacitor_SMD:C_0805_2012Metric" H 3488 5950 50  0001 C CNN
-F 3 "C0805C104J5RACAUTO" H 3450 6100 50  0001 C CNN
+F 3 "C696366" H 3450 6100 50  0001 C CNN
 	1    3450 6100
 	1    0    0    -1
@@
 F 1 "0.1u" H 2765 6055 50  0000 L CNN
 F 2 "Capacitor_SMD:C_0805_2012Metric" H 2688 5950 50  0001 C CNN
-F 3 "C0805C104J5RACAUTO" H 2650 6100 50  0001 C CNN
+F 3 "C696366" H 2650 6100 50  0001 C CNN
 	1    2650 6100
 	1    0    0    -1
@@
 F 1 "0.1u" H 3165 6055 50  0000 L CNN
 F 2 "Capacitor_SMD:C_0805_2012Metric" H 3088 5950 50  0001 C CNN
-F 3 "C0805C104J5RACAUTO" H 3050 6100 50  0001 C CNN
+F 3 "C696366" H 3050 6100 50  0001 C CNN
 	1    3050 6100
 	1    0    0    -1
@@
 F 1 "0.1u" H 3965 6055 50  0000 L CNN
 F 2 "Capacitor_SMD:C_0805_2012Metric" H 3888 5950 50  0001 C CNN
-F 3 "C0805C104J5RACAUTO" H 3850 6100 50  0001 C CNN
+F 3 "C696366" H 3850 6100 50  0001 C CNN
 	1    3850 6100
 	1    0    0    -1
@@
 F 1 "22p" V 3889 2700 50  0000 C CNN
 F 2 "Capacitor_SMD:C_0805_2012Metric" H 4088 2550 50  0001 C CNN
-F 3 "CL21C220JBANNNC " H 4050 2700 50  0001 C CNN
+F 3 "C1804" H 4050 2700 50  0001 C CNN
 	1    4050 2700
 	0    1    1    0
@@
 F 1 "22R" V 4450 4550 50  0000 C CNN
 F 2 "Resistor_SMD:R_0805_2012Metric" V 4380 4550 50  0001 C CNN
-F 3 "0805W8F220JT5E " H 4450 4550 50  0001 C CNN
+F 3 "C17561" H 4450 4550 50  0001 C CNN
 	1    4450 4550
 	0    1    1    0
