File: microcontroller.sch (KiCad schematic (older format))
At the start: 16 parts, among them J2 USB_B_Mini, U1 ATmega32U4-AU, Y1-16hz1 Crystal

Commit message: final
Parts:
- renumbered C85 to C102, C86 to C103, C87 to C104, C88 to C105, C89 to C106, C90 to C107, C91 to C108, C92 to C109
Connections:
- net labels added: TEENSY_GND
Changed lines of the file:
@@
 $EndComp
 $Comp
-L Device:C C90
+L Device:C C107
 U 1 1 60A8F4F8
 P 4050 2400
-F 0 "C90" V 3798 2400 50  0000 C CNN
+F 0 "C107" V 3798 2400 50  0000 C CNN
 F 1 "22p" V 3889 2400 50  0000 C CNN
 F 2 "Capacitor_SMD:C_0805_2012Metric" H 4088 2250 50  0001 C CNN
@@
 NoConn ~ 4050 4600
 $Comp
-L Device:C C92
+L Device:C C109
 U 1 1 60AA1797
 P 4400 5050
-F 0 "C92" V 4652 5050 50  0000 C CNN
+F 0 "C109" V 4652 5050 50  0000 C CNN
 F 1 "1u" V 4561 5050 50  0000 C CNN
 F 2 "Capacitor_SMD:C_0805_2012Metric" H 4438 4900 50  0001 C CNN
@@
 NoConn ~ 5400 2850
 $Comp
-L Device:C C85
+L Device:C C102
 U 1 1 60BB0957
 P 2200 6100
-F 0 "C85" H 2315 6146 50  0000 L CNN
+F 0 "C102" H 2315 6146 50  0000 L CNN
 F 1 "0.1u" H 2315 6055 50  0000 L CNN
 F 2 "Capacitor_SMD:C_0805_2012Metric" H 2238 5950 50  0001 C CNN
@@
 $EndComp
 $Comp
-L Device:C C88
+L Device:C C105
 U 1 1 60BB15A4
 P 3450 6100
-F 0 "C88" H 3565 6146 50  0000 L CNN
+F 0 "C105" H 3565 6146 50  0000 L CNN
 F 1 "0.1u" H 3565 6055 50  0000 L CNN
 F 2 "Capacitor_SMD:C_0805_2012Metric" H 3488 5950 50  0001 C CNN
@@
 $EndComp
 $Comp
-L Device:C C86
+L Device:C C103
 U 1 1 60BB2F1B
 P 2650 6100
-F 0 "C86" H 2765 6146 50  0000 L CNN
+F 0 "C103" H 2765 6146 50  0000 L CNN
 F 1 "0.1u" H 2765 6055 50  0000 L CNN
 F 2 "Capacitor_SMD:C_0805_2012Metric" H 2688 5950 50  0001 C CNN
@@
 $EndComp
 $Comp
-L Device:C C87
+L Device:C C104
 U 1 1 60BB46FD
 P 3050 6100
-F 0 "C87" H 3165 6146 50  0000 L CNN
+F 0 "C104" H 3165 6146 50  0000 L CNN
 F 1 "0.1u" H 3165 6055 50  0000 L CNN
 F 2 "Capacitor_SMD:C_0805_2012Metric" H 3088 5950 50  0001 C CNN
@@
 Connection ~ 3050 6250
 $Comp
-L Device:C C89
+L Device:C C106
 U 1 1 60BBF39F
 P 3850 6100
-F 0 "C89" H 3965 6146 50  0000 L CNN
+F 0 "C106" H 3965 6146 50  0000 L CNN
 F 1 "0.1u" H 3965 6055 50  0000 L CNN
 F 2 "Capacitor_SMD:C_0805_2012Metric" H 3888 5950 50  0001 C CNN
@@
 Connection ~ 2200 5950
 $Comp
-L Device:C C91
+L Device:C C108
 U 1 1 60BD615F
 P 4050 2700
-F 0 "C91" V 3798 2700 50  0000 C CNN
+F 0 "C108" V 3798 2700 50  0000 C CNN
 F 1 "22p" V 3889 2700 50  0000 C CNN
 F 2 "Capacitor_SMD:C_0805_2012Metric" H 4088 2550 50  0001 C CNN
@@
 	1    0    0    -1
 $EndComp
+$Comp
+L power:GND #PWR016
+U 1 1 613A6263
+P 8450 4550
+F 0 "#PWR016" H 8450 4300 50  0001 C CNN
+F 1 "GND" H 8455 4377 50  0000 C CNN
+F 2 "" H 8450 4550 50  0001 C CNN
+F 3 "" H 8450 4550 50  0001 C CNN
+	1    8450 4550
+	1    0    0    -1
+$EndComp
+Text HLabel 8450 4550 1    50   Input ~ 0
+TEENSY_GND
 $EndSCHEMATC

Commit message: swapping out controller with a different one
Parts:
- removed U1: ATmega32U4-AU, Package_QFP:TQFP-44_10x10mm_P0.8mm, symbol MCU_Microchip_ATmega:ATmega32U4-AU
- added U1: ATmega32U4-MU, Package_DFN_QFN:QFN-44-1EP_7x7mm_P0.5mm_EP5.2x5.2mm, symbol MCU_Microchip_ATmega:ATmega32U4-MU
Connections:
- net labels added: ATMEL_VCC, RESET
- wire segments 71 -> 74
Changed lines of the file:
@@
 $Descr A4 11693 8268
 encoding utf-8
-Sheet 3 4
+Sheet 4 4
 Title ""
 Date ""
@@
 U 1 1 60A86D65
 P 6900 4350
-F 0 "R4" V 6693 4350 50  0000 C CNN
+F 0 "R4" V 6900 4500 50  0000 C CNN
 F 1 "R10k" V 6900 4350 50  0000 C CNN
 F 2 "Resistor_SMD:R_1206_3216Metric" V 6830 4350 50  0001 C CNN
@@
 F 1 "Crystal" V 4645 2681 50  0000 L CNN
 F 2 "Crystal:Crystal_SMD_HC49-SD" H 4600 2550 50  0001 C CNN
-F 3 "C12676" H 4600 2550 50  0000 C CNN
+F 3 "C718667" H 4600 2550 50  0000 C CNN
 	1    4600 2550
 	0    1    1    0
@@
 F 1 "0.1u" H 2315 6055 50  0000 L CNN
 F 2 "Capacitor_SMD:C_0805_2012Metric" H 2238 5950 50  0001 C CNN
-F 3 "C696366;  used C696367 as alt due to inventory shortage" H 2200 6100 50  0001 C CNN
+F 3 "C696367" H 2200 6100 50  0001 C CNN
 	1    2200 6100
 	1    0    0    -1
@@
 F 1 "0.1u" H 3565 6055 50  0000 L CNN
 F 2 "Capacitor_SMD:C_0805_2012Metric" H 3488 5950 50  0001 C CNN
-F 3 "C696366;  used C696367 as alt due to inventory shortage" H 3450 6100 50  0001 C CNN
+F 3 "C696367" H 3450 6100 50  0001 C CNN
 	1    3450 6100
 	1    0    0    -1
@@
 F 1 "0.1u" H 2765 6055 50  0000 L CNN
 F 2 "Capacitor_SMD:C_0805_2012Metric" H 2688 5950 50  0001 C CNN
-F 3 "C696366;  used C696367 as alt due to inventory shortage" H 2650 6100 50  0001 C CNN
+F 3 "C696367" H 2650 6100 50  0001 C CNN
 	1    2650 6100
 	1    0    0    -1
@@
 F 1 "0.1u" H 3165 6055 50  0000 L CNN
 F 2 "Capacitor_SMD:C_0805_2012Metric" H 3088 5950 50  0001 C CNN
-F 3 "C696366;  used C696367 as alt due to inventory shortage" H 3050 6100 50  0001 C CNN
+F 3 "C696367" H 3050 6100 50  0001 C CNN
 	1    3050 6100
 	1    0    0    -1
@@
 F 1 "0.1u" H 3965 6055 50  0000 L CNN
 F 2 "Capacitor_SMD:C_0805_2012Metric" H 3888 5950 50  0001 C CNN
-F 3 "C696366;  used C696367 as alt due to inventory shortage" H 3850 6100 50  0001 C CNN
+F 3 "C696367" H 3850 6100 50  0001 C CNN
 	1    3850 6100
 	1    0    0    -1
@@
 	0    1    1    0
 $EndComp
-$Comp
-L MCU_Microchip_ATmega:ATmega32U4-AU U1
-U 1 1 60A82FF7
+Text HLabel 3600 2850 0    50   Input ~ 0
+TEENSY_GND
+Wire Wire Line
+	3600 2700 3600 2850
+Connection ~ 3600 2700
+Wire Wire Line
+	6100 1850 6500 1850
+Wire Wire Line
+	6500 1850 6500 1400
+Text HLabel 6500 1400 0    50   Output ~ 0
+ATMEL_VCC
+$Comp
+L MCU_Microchip_ATmega:ATmega32U4-MU U1
+U 1 1 6161C1B1
 P 6000 3750
 F 0 "U1" H 6000 1861 50  0000 C CNN
-F 1 "ATmega32U4-AU" H 6400 1450 50  0000 C CNN
-F 2 "Package_QFP:TQFP-44_10x10mm_P0.8mm" H 6000 3750 50  0001 C CIN
-F 3 "C44854" H 6000 3750 50  0001 C CNN
+F 1 "ATmega32U4-MU" H 5900 1550 50  0000 C CNN
+F 2 "Package_DFN_QFN:QFN-44-1EP_7x7mm_P0.5mm_EP5.2x5.2mm" H 6000 3750 50  0001 C CIN
+F 3 "C112161" H 6000 3750 50  0001 C CNN
 	1    6000 3750
 	1    0    0    -1
 $EndComp
-$Comp
-L power:GND #PWR016
-U 1 1 613A6263
-P 8450 4550
-F 0 "#PWR016" H 8450 4300 50  0001 C CNN
-F 1 "GND" H 8455 4377 50  0000 C CNN
-F 2 "" H 8450 4550 50  0001 C CNN
-F 3 "" H 8450 4550 50  0001 C CNN
-	1    8450 4550
-	1    0    0    -1
-$EndComp
-Text HLabel 8450 4550 1    50   Input ~ 0
-TEENSY_GND
+Text HLabel 5400 1400 2    50   Input ~ 0
+RESET
 $EndSCHEMATC

Commit message: almost done with the 3.3
Parts:
- C106: value 0.1u -> 10u
- Y1-16hz1: footprint Crystal:Crystal_SMD_HC49-SD -> CHGRAY-Keyboard:JLC_PCB_C718667
Connections:
- wire segments 74 -> 76
Other:
- moved on the sheet: C102, C103, C104, C105, C106
Changed lines of the file:
@@
 L Device:Crystal Y1-16hz1
 U 1 1 60A8D8F1
-P 4600 2550
-F 0 "Y1-16hz1" V 4554 2681 50  0000 L CNN
-F 1 "Crystal" V 4645 2681 50  0000 L CNN
-F 2 "Crystal:Crystal_SMD_HC49-SD" H 4600 2550 50  0001 C CNN
-F 3 "C718667" H 4600 2550 50  0000 C CNN
-	1    4600 2550
+P 4500 2550
+F 0 "Y1-16hz1" V 4454 2681 50  0000 L CNN
+F 1 "Crystal" V 4545 2681 50  0000 L CNN
+F 2 "CHGRAY-Keyboard:JLC_PCB_C718667" H 4500 2200 50  0000 C CNN
+F 3 "C718667" H 4550 2400 50  0000 C CNN
+	1    4500 2550
 	0    1    1    0
 $EndComp
@@
 $EndComp
 Wire Wire Line
-	4600 2400 5150 2400
-Wire Wire Line
 	5150 2400 5150 2450
 Wire Wire Line
 	5150 2450 5400 2450
 Wire Wire Line
-	4600 2700 5150 2700
-Wire Wire Line
 	5150 2700 5150 2650
 Wire Wire Line
 	5150 2650 5400 2650
-Wire Wire Line
-	4200 2400 4600 2400
-Connection ~ 4600 2400
-Wire Wire Line
-	4200 2700 4600 2700
-Connection ~ 4600 2700
 Wire Wire Line
 	3900 2400 3600 2400
@@
 	5400 3350 5200 3350
 Wire Wire Line
-	5200 3350 5200 4550
+	5200 3350 5200 4350
 Wire Wire Line
 	5200 4550 4600 4550
@@
 	4550 5050 5300 5050
 Wire Wire Line
-	5300 5050 5300 3550
+	5300 5050 5300 4350
 Wire Wire Line
 	5300 3550 5400 3550
@@
 L Device:C C102
 U 1 1 60BB0957
-P 2200 6100
-F 0 "C102" H 2315 6146 50  0000 L CNN
-F 1 "0.1u" H 2315 6055 50  0000 L CNN
-F 2 "Capacitor_SMD:C_0805_2012Metric" H 2238 5950 50  0001 C CNN
-F 3 "C696367" H 2200 6100 50  0001 C CNN
-	1    2200 6100
+P 3350 5750
+F 0 "C102" H 3465 5796 50  0000 L CNN
+F 1 "0.1u" H 3465 5705 50  0000 L CNN
+F 2 "Capacitor_SMD:C_0805_2012Metric" H 3388 5600 50  0001 C CNN
+F 3 "C696367" H 3350 5750 50  0001 C CNN
+	1    3350 5750
 	1    0    0    -1
 $EndComp
@@
 L Device:C C105
 U 1 1 60BB15A4
-P 3450 6100
-F 0 "C105" H 3565 6146 50  0000 L CNN
-F 1 "0.1u" H 3565 6055 50  0000 L CNN
-F 2 "Capacitor_SMD:C_0805_2012Metric" H 3488 5950 50  0001 C CNN
-F 3 "C696367" H 3450 6100 50  0001 C CNN
-	1    3450 6100
+P 4600 5750
+F 0 "C105" H 4715 5796 50  0000 L CNN
+F 1 "0.1u" H 4715 5705 50  0000 L CNN
+F 2 "Capacitor_SMD:C_0805_2012Metric" H 4638 5600 50  0001 C CNN
+F 3 "C696367" H 4600 5750 50  0001 C CNN
+	1    4600 5750
 	1    0    0    -1
 $EndComp
@@
 L Device:C C103
 U 1 1 60BB2F1B
-P 2650 6100
-F 0 "C103" H 2765 6146 50  0000 L CNN
-F 1 "0.1u" H 2765 6055 50  0000 L CNN
-F 2 "Capacitor_SMD:C_0805_2012Metric" H 2688 5950 50  0001 C CNN
-F 3 "C696367" H 2650 6100 50  0001 C CNN
-	1    2650 6100
+P 3800 5750
+F 0 "C103" H 3915 5796 50  0000 L CNN
+F 1 "0.1u" H 3915 5705 50  0000 L CNN
+F 2 "Capacitor_SMD:C_0805_2012Metric" H 3838 5600 50  0001 C CNN
+F 3 "C696367" H 3800 5750 50  0001 C CNN
+	1    3800 5750
 	1    0    0    -1
 $EndComp
@@
 L Device:C C104
 U 1 1 60BB46FD
-P 3050 6100
-F 0 "C104" H 3165 6146 50  0000 L CNN
-F 1 "0.1u" H 3165 6055 50  0000 L CNN
-F 2 "Capacitor_SMD:C_0805_2012Metric" H 3088 5950 50  0001 C CNN
-F 3 "C696367" H 3050 6100 50  0001 C CNN
-	1    3050 6100
-	1    0    0    -1
-$EndComp
-Wire Wire Line
-	2200 5950 2650 5950
-Wire Wire Line
-	3050 5950 3450 5950
-Wire Wire Line
-	2650 5950 3050 5950
-Connection ~ 2650 5950
-Connection ~ 3050 5950
-Wire Wire Line
-	2200 6250 2650 6250
-Wire Wire Line
-	3050 6250 2650 6250
-Connection ~ 2650 6250
-Wire Wire Line
-	3050 6250 3450 6250
-Connection ~ 3050 6250
+P 4200 5750
+F 0 "C104" H 4315 5796 50  0000 L CNN
+F 1 "0.1u" H 4315 5705 50  0000 L CNN
+F 2 "Capacitor_SMD:C_0805_2012Metric" H 4238 5600 50  0001 C CNN
+F 3 "C696367" H 4200 5750 50  0001 C CNN
+	1    4200 5750
+	1    0    0    -1
+$EndComp
+Wire Wire Line
+	3350 5600 3800 5600
+Wire Wire Line
+	4200 5600 4600 5600
+Wire Wire Line
+	3800 5600 4200 5600
+Connection ~ 3800 5600
+Connection ~ 4200 5600
+Wire Wire Line
+	3350 5900 3800 5900
+Wire Wire Line
+	4200 5900 3800 5900
+Connection ~ 3800 5900
+Wire Wire Line
+	4200 5900 4600 5900
+Connection ~ 4200 5900
 $Comp
 L Device:C C106
 U 1 1 60BBF39F
-P 3850 6100
-F 0 "C106" H 3965 6146 50  0000 L CNN
-F 1 "0.1u" H 3965 6055 50  0000 L CNN
-F 2 "Capacitor_SMD:C_0805_2012Metric" H 3888 5950 50  0001 C CNN
-F 3 "C696367" H 3850 6100 50  0001 C CNN
-	1    3850 6100
-	1    0    0    -1
-$EndComp
-Wire Wire Line
-	3450 5950 3850 5950
-Connection ~ 3450 5950
-Wire Wire Line
-	3450 6250 3850 6250
-Connection ~ 3450 6250
+P 5000 5750
+F 0 "C106" H 5115 5796 50  0000 L CNN
+F 1 "10u" H 5115 5705 50  0000 L CNN
+F 2 "Capacitor_SMD:C_0805_2012Metric" H 5038 5600 50  0001 C CNN
+F 3 "C15850" H 5000 5750 50  0001 C CNN
+	1    5000 5750
+	1    0    0    -1
+$EndComp
+Wire Wire Line
+	4600 5600 5000 5600
+Connection ~ 4600 5600
+Wire Wire Line
+	4600 5900 5000 5900
+Connection ~ 4600 5900
 $Comp
 L power:VCC #PWR03
 U 1 1 60BC98D5
-P 2200 5950
-F 0 "#PWR03" H 2200 5800 50  0001 C CNN
-F 1 "VCC" H 2215 6123 50  0000 C CNN
-F 2 "" H 2200 5950 50  0001 C CNN
-F 3 "" H 2200 5950 50  0001 C CNN
-	1    2200 5950
-	1    0    0    -1
-$EndComp
-$Comp
-L power:GND #PWR04
-U 1 1 60BCBB0F
-P 2200 6250
-F 0 "#PWR04" H 2200 6000 50  0001 C CNN
-F 1 "GND" H 2205 6077 50  0000 C CNN
-F 2 "" H 2200 6250 50  0001 C CNN
-F 3 "" H 2200 6250 50  0001 C CNN
-	1    2200 6250
-	1    0    0    -1
-$EndComp
-Connection ~ 2200 6250
-Connection ~ 2200 5950
+P 3350 5600
+F 0 "#PWR03" H 3350 5450 50  0001 C CNN
+F 1 "VCC" H 3365 5773 50  0000 C CNN
+F 2 "" H 3350 5600 50  0001 C CNN
+F 3 "" H 3350 5600 50  0001 C CNN
+	1    3350 5600
+	1    0    0    -1
+$EndComp
+Connection ~ 3350 5600
 $Comp
 L Device:C C108
@@
 L MCU_Microchip_ATmega:ATmega32U4-MU U1
 U 1 1 6161C1B1
-P 6000 3750
-F 0 "U1" H 6000 1861 50  0000 C CNN
-F 1 "ATmega32U4-MU" H 5900 1550 50  0000 C CNN
-F 2 "Package_DFN_QFN:QFN-44-1EP_7x7mm_P0.5mm_EP5.2x5.2mm" H 6000 3750 50  0001 C CIN
-F 3 "C112161" H 6000 3750 50  0001 C CNN
-	1    6000 3750
+P 5300 2550
+F 0 "U1" H 5300 661 50  0000 C CNN
+F 1 "ATmega32U4-MU" H 5200 350 50  0000 C CNN
+F 2 "Package_DFN_QFN:QFN-44-1EP_7x7mm_P0.5mm_EP5.2x5.2mm" H 5300 2550 50  0001 C CIN
+F 3 "C112161" H 5300 2550 50  0001 C CNN
+	1    5300 2550
 	1    0    0    -1
 $EndComp
 Text HLabel 5400 1400 2    50   Input ~ 0
 RESET
+$Comp
+L power:GND #PWR0103
+U 1 1 6190D24A
+P 3350 5900
+F 0 "#PWR0103" H 3350 5650 50  0001 C CNN
+F 1 "GND" H 3355 5727 50  0000 C CNN
+F 2 "" H 3350 5900 50  0001 C CNN
+F 3 "" H 3350 5900 50  0001 C CNN
+	1    3350 5900
+	1    0    0    -1
+$EndComp
+Connection ~ 3350 5900
+Wire Wire Line
+	4200 2400 4500 2400
+Wire Wire Line
+	4200 2700 4500 2700
+Connection ~ 4500 2400
+Wire Wire Line
+	4500 2400 5150 2400
+Connection ~ 4500 2700
+Wire Wire Line
+	4500 2700 5150 2700
+Connection ~ 5300 4350
+Wire Wire Line
+	5300 4350 5300 3550
+Connection ~ 5200 4350
+Wire Wire Line
+	5200 4350 5200 4550
 $EndSCHEMATC

Commit message: working on 6.3
Connections:
- wire segments 76 -> 73
Changed lines of the file:
@@
 	5400 3350 5200 3350
-Wire Wire Line
-	5200 3350 5200 4350
 Wire Wire Line
 	5200 4550 4600 4550
@@
 	4550 5050 5300 5050
 Wire Wire Line
-	5300 5050 5300 4350
-Wire Wire Line
 	5300 3550 5400 3550
 Wire Wire Line
@@
 	0    1    1    0
 $EndComp
-Text HLabel 3600 2850 0    50   Input ~ 0
+Text HLabel 3750 5050 0    50   Input ~ 0
 TEENSY_GND
-Wire Wire Line
-	3600 2700 3600 2850
-Connection ~ 3600 2700
 Wire Wire Line
 	6100 1850 6500 1850
@@
 L MCU_Microchip_ATmega:ATmega32U4-MU U1
 U 1 1 6161C1B1
-P 5300 2550
-F 0 "U1" H 5300 661 50  0000 C CNN
-F 1 "ATmega32U4-MU" H 5200 350 50  0000 C CNN
-F 2 "Package_DFN_QFN:QFN-44-1EP_7x7mm_P0.5mm_EP5.2x5.2mm" H 5300 2550 50  0001 C CIN
-F 3 "C112161" H 5300 2550 50  0001 C CNN
-	1    5300 2550
+P 6000 3750
+F 0 "U1" H 6000 1861 50  0000 C CNN
+F 1 "ATmega32U4-MU" H 5900 1550 50  0000 C CNN
+F 2 "Package_DFN_QFN:QFN-44-1EP_7x7mm_P0.5mm_EP5.2x5.2mm" H 6000 3750 50  0001 C CIN
+F 3 "C112161" H 6000 3750 50  0001 C CNN
+	1    6000 3750
 	1    0    0    -1
 $EndComp
@@
 Wire Wire Line
 	4500 2700 5150 2700
-Connection ~ 5300 4350
-Wire Wire Line
-	5300 4350 5300 3550
-Connection ~ 5200 4350
-Wire Wire Line
-	5200 4350 5200 4550
+Wire Wire Line
+	5200 3350 5200 4550
+Wire Wire Line
+	5300 3550 5300 5050
 $EndSCHEMATC
