File: microcontroller.sch (KiCad schematic (older format))
At the start: 16 parts, among them J2 USB_B_Mini, U1 ATmega32U4-MU, Y1-16hz1 Crystal

Commit message: 3.3-AU
Parts:
- removed U1: ATmega32U4-MU, Package_DFN_QFN:QFN-44-1EP_7x7mm_P0.5mm_EP5.2x5.2mm, symbol MCU_Microchip_ATmega:ATmega32U4-MU
- added U1: ATmega32U4-AU, Package_QFP:TQFP-44_10x10mm_P0.8mm, symbol MCU_Microchip_ATmega:ATmega32U4-AU
Changed lines of the file:
@@
 Text HLabel 6500 1400 0    50   Output ~ 0
 ATMEL_VCC
-$Comp
-L MCU_Microchip_ATmega:ATmega32U4-MU U1
-U 1 1 6161C1B1
-P 6000 3750
-F 0 "U1" H 6000 1861 50  0000 C CNN
-F 1 "ATmega32U4-MU" H 5900 1550 50  0000 C CNN
-F 2 "Package_DFN_QFN:QFN-44-1EP_7x7mm_P0.5mm_EP5.2x5.2mm" H 6000 3750 50  0001 C CIN
-F 3 "C112161" H 6000 3750 50  0001 C CNN
-	1    6000 3750
-	1    0    0    -1
-$EndComp
 Text HLabel 5400 1400 2    50   Input ~ 0
 RESET
@@
 Wire Wire Line
 	5300 3550 5300 5050
+$Comp
+L MCU_Microchip_ATmega:ATmega32U4-AU U1
+U 1 1 618DD3F7
+P 6000 3750
+F 0 "U1" H 6000 1861 50  0000 C CNN
+F 1 "ATmega32U4-AU" H 6000 1770 50  0000 C CNN
+F 2 "Package_QFP:TQFP-44_10x10mm_P0.8mm" H 6000 3750 50  0001 C CIN
+F 3 "http://ww1.microchip.com/downloads/en/DeviceDoc/Atmel-7766-8-bit-AVR-ATmega16U4-32U4_Datasheet.pdf" H 6000 3750 50  0001 C CNN
+	1    6000 3750
+	1    0    0    -1
+$EndComp
 $EndSCHEMATC

Commit message: update to new keyboard sizes
Parts:
- removed U1: ATmega32U4-AU, Package_QFP:TQFP-44_10x10mm_P0.8mm, symbol MCU_Microchip_ATmega:ATmega32U4-AU
- added U1: ATmega32U4RC-AU, Package_QFP:TQFP-44_10x10mm_P0.8mm, symbol MCU_Microchip_ATmega:ATmega32U4RC-AU
Changed lines of the file:
@@
 P 6000 5550
 F 0 "#PWR013" H 6000 5300 50  0001 C CNN
-F 1 "GND" H 6005 5377 50  0000 C CNN
+F 1 "GND" H 6250 5400 50  0000 C CNN
 F 2 "" H 6000 5550 50  0001 C CNN
 F 3 "" H 6000 5550 50  0001 C CNN
@@
 P 5900 1950
 F 0 "#PWR010" H 5900 1800 50  0001 C CNN
-F 1 "VCC" H 5915 2123 50  0000 C CNN
+F 1 "VCC" H 5700 2150 50  0000 C CNN
 F 2 "" H 5900 1950 50  0001 C CNN
 F 3 "" H 5900 1950 50  0001 C CNN
@@
 P 6000 1950
 F 0 "#PWR012" H 6000 1800 50  0001 C CNN
-F 1 "VCC" H 6015 2123 50  0000 C CNN
+F 1 "VCC" H 5850 2250 50  0000 C CNN
 F 2 "" H 6000 1950 50  0001 C CNN
 F 3 "" H 6000 1950 50  0001 C CNN
@@
 	5300 3550 5300 5050
 $Comp
-L MCU_Microchip_ATmega:ATmega32U4-AU U1
-U 1 1 618DD3F7
+L MCU_Microchip_ATmega:ATmega32U4RC-AU U1
+U 1 1 6193204F
 P 6000 3750
 F 0 "U1" H 6000 1861 50  0000 C CNN
-F 1 "ATmega32U4-AU" H 6000 1770 50  0000 C CNN
+F 1 "ATmega32U4RC-AU" H 6000 1600 50  0000 C CNN
 F 2 "Package_QFP:TQFP-44_10x10mm_P0.8mm" H 6000 3750 50  0001 C CIN
 F 3 "http://ww1.microchip.com/downloads/en/DeviceDoc/Atmel-7766-8-bit-AVR-ATmega16U4-32U4_Datasheet.pdf" H 6000 3750 50  0001 C CNN

Commit message: attempting 3.3-AU
Parts:
- J2: footprint Connector_USB:USB_Mini-B_Wuerth_65100516121_Horizontal -> CHGRAY-Keyboard:USB_Mini-B_Wuerth_65100516121_Horizontal
Changed lines of the file:
@@
 F 0 "J2" H 3807 4867 50  0000 C CNN
 F 1 "USB_B_Mini" H 3807 4776 50  0000 C CNN
-F 2 "Connector_USB:USB_Mini-B_Wuerth_65100516121_Horizontal" H 3900 4350 50  0001 C CNN
+F 2 "CHGRAY-Keyboard:USB_Mini-B_Wuerth_65100516121_Horizontal" H 3900 4350 50  0001 C CNN
 F 3 "C69074" H 3900 4350 50  0001 C CNN
 	1    3750 4400

Commit message: working on Yeet3.4;  changed microcontroller, added screw hole, and I think fixed the 5V LED issue (needs to be verified)
Parts:
- removed U1: ATmega32U4RC-AU, Package_QFP:TQFP-44_10x10mm_P0.8mm, symbol MCU_Microchip_ATmega:ATmega32U4RC-AU
- added U1: ATmega32U4-MU, Package_DFN_QFN:QFN-44-1EP_7x7mm_P0.5mm_EP5.2x5.2mm, symbol MCU_Microchip_ATmega:ATmega32U4-MU
Connections:
- wire segments 73 -> 71
Changed lines of the file:
@@
 P 5900 1950
 F 0 "#PWR010" H 5900 1800 50  0001 C CNN
-F 1 "VCC" H 5700 2150 50  0000 C CNN
+F 1 "VCC" H 5800 2000 50  0000 C CNN
 F 2 "" H 5900 1950 50  0001 C CNN
 F 3 "" H 5900 1950 50  0001 C CNN
@@
 F 1 "Crystal" V 4545 2681 50  0000 L CNN
 F 2 "CHGRAY-Keyboard:JLC_PCB_C718667" H 4500 2200 50  0000 C CNN
-F 3 "C718667" H 4550 2400 50  0000 C CNN
+F 3 "C111377" H 4550 2400 50  0000 C CNN
 	1    4500 2550
 	0    1    1    0
@@
 	5400 2250 5400 1400
 Wire Wire Line
-	5400 1400 4350 1400
-Wire Wire Line
 	4350 1400 3950 1400
 Wire Wire Line
@@
 Text HLabel 3750 5050 0    50   Input ~ 0
 TEENSY_GND
-Wire Wire Line
-	6100 1850 6500 1850
-Wire Wire Line
-	6500 1850 6500 1400
-Text HLabel 6500 1400 0    50   Output ~ 0
+Text HLabel 5900 1850 1    50   Output ~ 0
 ATMEL_VCC
 Text HLabel 5400 1400 2    50   Input ~ 0
@@
 Wire Wire Line
 	5300 3550 5300 5050
-$Comp
-L MCU_Microchip_ATmega:ATmega32U4RC-AU U1
-U 1 1 6193204F
+Text HLabel 6100 1850 1    50   Output ~ 0
+ATMEL_VCC
+Text HLabel 7050 -250 1    50   Output ~ 0
+ATMEL_VCC
+Wire Wire Line
+	4350 1400 5400 1400
+Text HLabel 7350 -100 1    50   Output ~ 0
+ATMEL_VCC
+Text HLabel 6000 1850 1    50   Output ~ 0
+ATMEL_VCC
+Text HLabel 4950 3050 3    50   Output ~ 0
+ATMEL_VCC
+$Comp
+L MCU_Microchip_ATmega:ATmega32U4-MU U1
+U 1 1 61AF3258
 P 6000 3750
 F 0 "U1" H 6000 1861 50  0000 C CNN
-F 1 "ATmega32U4RC-AU" H 6000 1600 50  0000 C CNN
-F 2 "Package_QFP:TQFP-44_10x10mm_P0.8mm" H 6000 3750 50  0001 C CIN
+F 1 "ATmega32U4-MU" H 6000 1770 50  0000 C CNN
+F 2 "Package_DFN_QFN:QFN-44-1EP_7x7mm_P0.5mm_EP5.2x5.2mm" H 6000 3750 50  0001 C CIN
 F 3 "http://ww1.microchip.com/downloads/en/DeviceDoc/Atmel-7766-8-bit-AVR-ATmega16U4-32U4_Datasheet.pdf" H 6000 3750 50  0001 C CNN
 	1    6000 3750

Commit message: updates
Parts:
- Y1-16hz1: footprint CHGRAY-Keyboard:JLC_PCB_C718667 -> CHGRAY-Keyboard:JLC_PCB_C111377
Changed lines of the file:
@@
 F 0 "Y1-16hz1" V 4454 2681 50  0000 L CNN
 F 1 "Crystal" V 4545 2681 50  0000 L CNN
-F 2 "CHGRAY-Keyboard:JLC_PCB_C718667" H 4500 2200 50  0000 C CNN
+F 2 "CHGRAY-Keyboard:JLC_PCB_C111377" H 4500 2200 50  0000 C CNN
 F 3 "C111377" H 4550 2400 50  0000 C CNN
 	1    4500 2550

Commit message: Yeet; possibly final!!
Parts:
- renumbered Y1-16hz1 to Y1
Changed lines of the file:
@@
 $Descr A4 11693 8268
 encoding utf-8
-Sheet 4 4
+Sheet 3 4
 Title ""
 Date ""
@@
 $EndComp
 $Comp
-L Device:Crystal Y1-16hz1
+L Device:Crystal Y1
 U 1 1 60A8D8F1
 P 4500 2550
-F 0 "Y1-16hz1" V 4454 2681 50  0000 L CNN
+F 0 "Y1" V 4454 2681 50  0000 L CNN
 F 1 "Crystal" V 4545 2681 50  0000 L CNN
 F 2 "CHGRAY-Keyboard:JLC_PCB_C111377" H 4500 2200 50  0000 C CNN

Commit message: copy the ATMega32U4-AU into our private library
Parts:
- U1: symbol MCU_Microchip_ATmega:ATmega32U4-MU -> Cherry-Symbol:ATmega32U4-AU
Changed lines of the file:
@@
 ATMEL_VCC
 $Comp
-L MCU_Microchip_ATmega:ATmega32U4-MU U1
+L Cherry-Symbol:ATmega32U4-AU U1
 U 1 1 61AF3258
 P 6000 3750
