File: WS2812-LEDs.sch (KiCad schematic (older format))
At the start: 168 parts

Commit message: flip to WS2812
Parts:
- renumbered C72 to C?, C76 to C?, C80 to C?, C60 to C?, C64 to C?, C68 to C?, C48 to C?, C52 to C?, C56 to C?, C36 to C?, C40 to C?, C44 to C?, C24 to C?, C28 to C?, C32 to C?, C11 to C?, C16 to C?, C20 to C?, C1 to C?, C6 to C?, C84 to C?, C73 to C?, C77 to C?, C81 to C?, C61 to C?, C65 to C?, C69 to C?, C49 to C?, C53 to C?, C57 to C?, C37 to C?, C41 to C?, C45 to C?, C25 to C?, C29 to C?, C33 to C?, C12 to C?, C17 to C?, C21 to C?, C2 to C?, C7 to C?, C74 to C?, C78 to C?, C82 to C?, C62 to C?, C66 to C?, C70 to C?, C50 to C?, C54 to C?, C58 to C?, C38 to C?, C42 to C?, C46 to C?, C26 to C?, C30 to C?, C34 to C?, C13 to C?, C18 to C?, C22 to C?, C3 to C?, C8 to C?, C75 to C?, C79 to C?, C83 to C?, C63 to C?, C67 to C?, C71 to C?, C51 to C?, C55 to C?, C59 to C?, C39 to C?, C43 to C?, C47 to C?, C27 to C?, C31 to C?, C35 to C?, C14 to C?, C19 to C?, C23 to C?, C4 to C?, C9 to C?, C15 to C?, C5 to C?, C10 to C?

Commit message: led work
Parts:
- D100, D101, D102, D103, D104, D105, D106, D107, D108, D109, D110, D111, D112, D113, D114, D115, D116, D117, D118, D119, D120, D121, D122, D123, D124, D125, D126, D127, D128, D129, D130, D131, D132, D133, D134, D135, D136, D137, D138, D139, D140, D141, D142, D143, D144, D145, D146, D147, D148, D149, D150, D151, D152, D153, D154, D155, D156, D157, D158, D159, D160, D161, D162, D163, D164, D165, D166, D167, D168, D85, D86, D87, D88, D89, D90, D91, D92, D93, D94, D95, D96, D97, D98, D99: footprint daprice-keyswitches:LED_SK6812MINI_PLCC4_3.5x3.5mm_P1.75mm -> CHGRAY_LED:LED_WS2812-2020; symbol LED:SK6812MINI -> LED:WS2812B
- gave numbers to parts that had none: 84

Commit message: leds
Changed lines of the file:
@@
 	1    0    0    -1
 $EndComp
-Text GLabel 1600 950  2    50   Input ~ 0
+Text GLabel 1600 800  2    50   Input ~ 0
 LED_5V
 Text HLabel 1300 800  0    50   Input ~ 0
@@
 Wire Wire Line
 	1300 800  1600 800
-Text GLabel 1600 800  2    50   Input ~ 0
+Text GLabel 1600 950  2    50   Input ~ 0
 LED_GND
 $Comp

Commit message: final
Parts:
- added C20, C25, C30, C35, C40, C45, C50, C55, C60, C65, C70, C75, C80, C85: C104 0.1uF 100nF, Capacitor_SMD:C_0402_1005Metric, symbol Device:C
- added D114, D119, D124, D129, D134, D139, D144, D149, D154, D159, D164, D169, D174, D179: LED, CHGRAY_LED:LED_WS2812-2020, symbol LED:WS2812B
- renumbered C84 to C101, C20 to C21, C21 to C22, C22 to C23, C23 to C24, C24 to C26, C25 to C27, C26 to C28, C27 to C29, C28 to C31, C29 to C32, C30 to C33, C31 to C34, C32 to C36, C33 to C37, C34 to C38, C35 to C39, C36 to C41, C37 to C42, C38 to C43, C39 to C44, C40 to C46, C41 to C47, C42 to C48, C43 to C49, C44 to C51, C45 to C52, C46 to C53, C47 to C54, C48 to C56, C49 to C57, C50 to C58, C51 to C59, C52 to C61, C53 to C62, C54 to C63, C55 to C64, C56 to C66, C57 to C67, C58 to C68, C59 to C69, C60 to C71, C61 to C72, C62 to C73, C63 to C74, C64 to C76, C65 to C77, C66 to C78, C67 to C79, C68 to C81, C69 to C82, C70 to C83, C71 to C84, C72 to C86, C73 to C87, C74 to C88, C75 to C89, C76 to C91, C77 to C92, C78 to C93, C79 to C94, C80 to C96, C81 to C97, C82 to C98, C83 to C99, D90 to D100, D91 to D101, D92 to D102, D93 to D103, D94 to D104, D95 to D105, D96 to D106, D97 to D107, D98 to D108, D99 to D109, D100 to D110, D101 to D111, D102 to D112, D103 to D113, D104 to D115, D105 to D116, D106 to D117, D107 to D118, D108 to D120, D109 to D121, D110 to D122, D111 to D123, D112 to D125, D113 to D126, D114 to D127, D115 to D128, D116 to D130, D117 to D131, D118 to D132, D119 to D133, D120 to D135, D121 to D136, D122 to D137, D123 to D138, D124 to D140, D125 to D141, D126 to D142, D127 to D143, D128 to D145, D129 to D146, D130 to D147, D131 to D148, D132 to D150, D133 to D151, D134 to D152, D135 to D153, D136 to D155, D137 to D156, D138 to D157, D139 to D158, D140 to D160, D141 to D161, D142 to D162, D143 to D163, D144 to D165, D145 to D166, D146 to D167, D147 to D168, D148 to D170, D149 to D171, D150 to D172, D151 to D173, D152 to D175, D153 to D176, D154 to D177, D155 to D178, D156 to D180, D157 to D181, D158 to D182, D159 to D183, D160 to D185, D161 to D186, D162 to D187, D163 to D188, D164 to D190, D165 to D191, D166 to D192, D167 to D193, D168 to D195, D85 to D95, D86 to D96, D87 to D97, D88 to D98, D89 to D99
Connections:
- wire segments 105 -> 119
